File: hardware/Ziess-Microsope-Controller_Main_board/X_Driver.kicad_sch (KiCad schematic)
At the start: 38 parts, among them J2 B4B-XH-AM, U5 TMC2209-LA

Commit message: m
Parts:
- R38: now left out of the parts list
Changed lines of the file:
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@@
 		(body_style 1)
 		(exclude_from_sim no)
-		(in_bom yes)
-		(on_board no)
+		(in_bom no)
+		(on_board yes)
 		(in_pos_files yes)
 		(dnp yes)

Commit message: init
Parts:
- J2: value B4B-XH-AM -> 43045-0418
Changed lines of the file:
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@@
 			)
 		)
-		(property "Value" "B4B-XH-AM"
+		(property "Value" "43045-0418"
 			(at 234.95 101.6 0)
 			(show_name no)

Commit message: m
Parts:
- renumbered C25 to C64, C26 to C65, C27 to C66, C28 to C67, C29 to C68, C30 to C69, C31 to C70, C32 to C71, C33 to C72, C34 to C73, C35 to C74, C36 to C75, C37 to C76, C38 to C77, C39 to C78, C40 to C79, C41 to C80, C42 to C81, D4 to D6, J2 to J6, R22 to R60, R23 to R61, R24 to R62, R25 to R63, R26 to R64, R27 to R65, R28 to R66, R29 to R67, R30 to R68, R31 to R69, R32 to R70, R33 to R71, R34 to R72, R35 to R73, R36 to R74, R37 to R75, R38 to R76, U5 to U10
