File: hardware/Ziess-Microsope-Controller_Main_board/MCU.kicad_sch (KiCad schematic)
At the start: 48 parts, among them J17 B10B-XH-AM, J18 B4B-XH-AM, SW2 SW_Push, SW3 CJS1201A, U17 STM32F446VETx, Y1 X322516MMB4SI

Commit message: m
Parts:
- added U18: STM32F765VGTx, Package_QFP:LQFP-100_14x14mm_P0.5mm, symbol MCU_ST_STM32F7:STM32F765VGTx
Connections:
- new net: U18.10 (VSS), U18.26 (VSS), U18.49 (VSS), U18.74 (VSS), U18.99 (VSS)
