File: hardware/Ziess-Microsope-Controller_Main_board/MCU.kicad_sch (KiCad schematic)
At the start: 49 parts, among them J17 B10B-XH-AM, J18 B4B-XH-AM, SW2 SW_Push, SW3 CJS1201A, U17 STM32F446VETx, U18 STM32F765VGTx, Y1 X322516MMB4SI

Commit message: m
Parts:
- removed C106: 100nF, Capacitor_SMD:C_0603_1608Metric, symbol Device:C_Small
- removed J18: B4B-XH-AM, Library:BM04BGHSTBTLFSN, symbol Connector_Generic:Conn_01x04
- removed R136: 10k, Resistor_SMD:R_0603_1608Metric, symbol Device:R_Small
- removed U17: STM32F446VETx, Package_QFP:LQFP-100_14x14mm_P0.5mm, symbol MCU_ST_STM32F4:STM32F446VETx
- removed Y1: X322516MMB4SI, Library:X322516MMB4SI, symbol Device:Crystal_GND24
- added C122: 100nF, Capacitor_SMD:C_0603_1608Metric, symbol Device:C_Small
- added Y1: Crystal_Small, Library:XTAL_NX3225GD-8MHZ-STD-CRA-3_NDK, symbol Device:Crystal_Small
- C117, C118: footprint Capacitor_SMD:C_0603_1608Metric -> Capacitor_SMD:C_0402_1005Metric
- J17: value B10B-XH-AM -> Conn_01x10; footprint Library:B10BXHAMLFSN -> Library:BM10BGHSTBT
Connections:
- net +3.3V: now also U18.100 (VDD), U18.11 (VDD), U18.27 (VDD), U18.50 (VDD), U18.6 (VBAT), U18.75 (VDD)
- net EXP_GPIO_1: now also R134.1
- net EXP_GPIO_6: no longer R134.1
- net GND: now also U18.10 (VSS), U18.19 (VSSA), U18.26 (VSS), U18.49 (VSS), U18.74 (VSS), U18.99 (VSS), C122.1
- net MCU_RESET: now also U18.14 (NRST)
- net SWCLK: now also U18.76 (PA14)
- net SWDIO: now also U18.72 (PA13)
- net USB_N: now also U18.71 (PA12)
- net USB_P: now also U18.70 (PA11)
- net USB_VBUS: now also U18.68 (PA9), C122.2
- net VDDA: now also U18.20 (VREF+), U18.21 (VDDA)
- net at C118.2: now also U18.13 (PH1), Y1.2
- net at C119.2: now also U18.48 (VCAP_1)
- net at C117.2: now also U18.12 (PH0), Y1.1
- net at C120.2: now also U18.73 (VCAP_2)
- net at R135.2: now also U18.94 (BOOT0)
- no-connect marks 73 -> 75
Other:
- moved on the sheet: C100, C101, C102, C103, C104, C105, U18

Commit message: init
Parts:
- added J16: TC2030, Connector:Tag-Connect_TC2030-IDC-NL_2x03_P1.27mm_Vertical, symbol Connector:TC2030
- C119, C120: footprint Capacitor_SMD:C_1206_3216Metric -> Capacitor_SMD:C_0805_2012Metric
- R123, R124, R125, R126, R127, R128: value 0 -> 330
Connections:
- net +3.3V: now also J16.1
- net GND: now also J16.5
- net MCU_RESET: now also J16.3
- net SWCLK: now also J16.4
- net SWDIO: now also J16.2
- net SWO: now reaches U18.89 (PB3)
- net SWO: now also J16.6
- no-connect marks 75 -> 74

Commit message: m
Parts:
- removed C100: 4.7uF, Capacitor_SMD:C_0805_2012Metric, symbol Device:C_Small
- removed C101, C102, C103, C104, C105, C107, C109, C116, C122: 100nF, Capacitor_SMD:C_0603_1608Metric, symbol Device:C_Small
- removed C108: 1uF, Capacitor_SMD:C_0603_1608Metric, symbol Device:C_Small
- removed C117, C118: 10pf, Capacitor_SMD:C_0402_1005Metric, symbol Device:C_Small
- removed C119, C120: 2.2uF, Capacitor_SMD:C_0805_2012Metric, symbol Device:C_Small
- removed R135: 10k, Resistor_SMD:R_0603_1608Metric, symbol Device:R_Small
- removed U18: STM32F765VGTx, Package_QFP:LQFP-100_14x14mm_P0.5mm, symbol MCU_ST_STM32F7:STM32F765VGTx
- added C28, C29: 4.7uF, Capacitor_SMD:C_0805_2012Metric, symbol Device:C_Small
- added C30, C31, C32, C33, C34, C35, C36, C37, C38, C39, C40, C42, C43, C44, C51, C52: 100nF, Capacitor_SMD:C_0603_1608Metric, symbol Device:C_Small
- added C41: 1uF, Capacitor_SMD:C_0603_1608Metric, symbol Device:C_Small
- added C53, C54: 10pf, Capacitor_SMD:C_0402_1005Metric, symbol Device:C_Small
- added C55, C56: 2.2uF, Capacitor_SMD:C_0805_2012Metric, symbol Device:C_Small
- added R45: 10k, Resistor_SMD:R_0603_1608Metric, symbol Device:R_Small
- added U5: STM32F765ZGTx, Package_QFP:LQFP-144_20x20mm_P0.5mm, symbol MCU_ST_STM32F7:STM32F765ZGTx
- renumbered C110 to C45, C111 to C46, C112 to C47, C113 to C48, C114 to C49, C115 to C50, J17 to J2, J16 to J3, R117 to R27, R118 to R28, R119 to R29, R120 to R30, R121 to R31, R122 to R32, R123 to R33, R124 to R34, R125 to R35, R126 to R36, R127 to R37, R128 to R38, R129 to R39, R130 to R40, R131 to R41, R132 to R42, R133 to R43, R134 to R44
Connections:
- net +3.3V: now also C28.2, C29.2, C30.2, C31.2, C32.2, C33.2, C34.2, C35.2, C36.2, C37.2, C38.2, C39.2, C42.2, C43.2, C44.2, C51.2, U5.108 (VDD), U5.121 (VDDSDMMC), U5.131 (VDD), U5.143 (PDR_ON), U5.144 (VDD), U5.17 (VDD), U5.30 (VDD), U5.39 (VDD), U5.52 (VDD), U5.6 (VBAT), U5.62 (VDD), U5.72 (VDD), U5.84 (VDD), U5.95 (VDDUSB)
- net GND: now also C28.1, C29.1, C30.1, C31.1, C32.1, C33.1, C34.1, C35.1, C36.1, C37.1, C38.1, C39.1, C40.1, C41.1, C42.1, C43.1, C44.1, C51.1, C52.1, C53.1, C54.1, C55.1, C56.1, U5.107 (VSS), U5.120 (VSS), U5.130 (VSS), U5.16 (VSS), U5.31 (VSSA), U5.38 (VSS), U5.51 (VSS), U5.61 (VSS), U5.83 (VSS), U5.94 (VSS)
- net MCU_RESET: now also C52.2, U5.25 (NRST)
- net SWCLK: now also U5.109 (PA14)
- net SWDIO: now also U5.105 (PA13)
- net SWO: now also U5.133 (PB3)
- net USB_N: now also U5.103 (PA11)
- net USB_P: now also U5.104 (PA12)
- net VDDA: now also C40.2, C41.2, U5.32 (VREF+), U5.33 (VDDA)
- net at Y1.2: now also C54.2, U5.24 (PH1)
- net at Y1.1: now also C53.2, U5.23 (PH0)
- net at SW3.2 (B): now also R45.1
- new net: C56.2, U5.106 (VCAP_2)
- new net: R45.2, U5.138 (BOOT0)
- new net: C55.2, U5.71 (VCAP_1)
- no-connect marks 74 -> 0
