File: hardware/Ziess-Microsope-Controller_Main_board/Ziess-Microsope-Controller_Main_board.kicad_sch (KiCad schematic)
At the start: 0 parts

Commit message: m
Parts:
- added J1: 670689000, Library:670689000, symbol Connector:USB_B
- added J10, J14, J20, J7: Conn_01x03, Library:B3BXHAMLFSN, symbol Connector_Generic:Conn_01x03
- added J11, J15, J18, J8: Conn_01x04, Library:B4BXHAM, symbol Connector_Generic:Conn_01x04
- added J12, J9: Conn_01x06, Library:B6BXHAMLFSN, symbol Connector_Generic:Conn_01x06
- added J13, J16, J17, J19: Conn_01x02, Library:B2BXHAMLFSN, symbol Connector_Generic:Conn_01x02
- added J2: 23117633, Library:23117633, symbol Connector:DE15_Socket_HighDensity
- added J21: Conn_01x10, Library:B10BXHAMLFSN, symbol Connector_Generic:Conn_01x10
- added J3, J4: 57478404, Library:57478404, symbol Connector:DE9_Pins
- added J5: 0039301040, Library:0039301040, symbol Connector_Generic:Conn_01x04
- added J6: Conn_Coaxial, symbol Library:Conn_Coaxial
- added U1: TPS24751RUVR, RUV(R-PVQFN-N36), symbol Library:TPS24751RUVR
Connections:
- new net: J6.2 (Ext), J6.3 (Ext)

Commit message: m
Parts:
- removed J11: Conn_01x04, Library:B4BXHAM, symbol Connector_Generic:Conn_01x04
- removed J12: Conn_01x06, Library:B6BXHAMLFSN, symbol Connector_Generic:Conn_01x06
- added C1, C17: 22uF, symbol Device:C_Small
- added C10: 120pF, symbol Device:C_Small
- added C11, C15, C16, C19, C2, C22, C26, C28, C29, C30, C31, C32, C37, C38, C39, C4, C41, C43, C44, C45, C46, C47, C49, C51, C53, C55, C63, C64: 100nF, symbol Device:C_Small
- added C12: 10nF, symbol Device:C_Small
- added C13, C14: 47uF, symbol Device:C_Small
- added C18, C24, C25, C50, C52, C7, C8: 10uF, symbol Device:C_Small
- added C20, C48, C65: 22nF, symbol Device:C_Small
- added C21, C56: 4.7uF, symbol Device:C_Small
- added C23, C27, C54, C58: 100uF, Capacitor_SMD:CP_Elec_8x10, symbol Device:C_Polarized_Small
- added C3: 33nF, symbol Device:C_Small
- added C33, C34, C35, C36, C57, C59, C60, C61: 470pF, symbol Device:C_Small
- added C40, C42: 1uF, symbol Device:C_Small
- added C5, C6, C62: 220uF, Capacitor_SMD:CP_Elec_8x10, symbol Device:C_Polarized_Small
- added C9: 12nF, symbol Device:C_Small
- added D1: GREEN, LED_SMD:LED_0805_2012Metric, symbol Device:LED
- added D2: SMAJ15A, Diode_SMD:D_SMA, symbol Diode:SMAJ15A
- added D3, D5, D6: RED, LED_SMD:LED_0805_2012Metric, symbol Device:LED
- added D4: MBRS340, Diode_SMD:D_SMC, symbol Diode:MBRS340
- added J11: B6B-XH-AM, Library:B6BXHAMLFSN, symbol Connector_Generic:Conn_01x06
- added J12: B4B-XH-AM, Library:B4BXHAM, symbol Connector_Generic:Conn_01x04
- added L1: 15uH, Library:XAL6060153MEC, symbol Device:L_Iron
- added R1: 15k, Resistor_SMD:R_0603_1608Metric, symbol Device:R_Small
- added R10: 0.002, Resistor_SMD:R_2512_6332Metric, symbol Device:R_Small
- added R11, R5: ~, Resistor_SMD:R_0603_1608Metric, symbol Device:R_Small
- added R12, R14, R52, R53: 0.1, Resistor_SMD:R_0603_1608Metric, symbol Device:R_Small
- added R13: 3.74k, Resistor_SMD:R_0603_1608Metric, symbol Device:R_Small
- added R15, R7: 51.1, Resistor_SMD:R_0603_1608Metric, symbol Device:R_Small
- added R16, R28, R43: 100k, Resistor_SMD:R_0603_1608Metric, symbol Device:R_Small
- added R17: 19.1k, Resistor_SMD:R_0603_1608Metric, symbol Device:R_Small
- added R18, R19, R20, R21, R22, R23, R25, R35, R36, R37, R38, R39, R40, R44: 0, Resistor_SMD:R_0603_1608Metric, symbol Device:R_Small
- added R2, R33, R34, R49, R51, R54: 10k, Resistor_SMD:R_0603_1608Metric, symbol Device:R_Small
- added R24, R41: 20k, Resistor_SMD:R_0603_1608Metric, symbol Device:R_Small
- added R26, R30, R47, R50: 10K, Resistor_SMD:R_0603_1608Metric, symbol Device:R_Small
- added R27, R42: 1k, Resistor_SMD:R_0603_1608Metric, symbol Device:R_Small
- added R29, R45: 1K, Resistor_SMD:R_0603_1608Metric, symbol Device:R_Small
- added R3: 130k, Resistor_SMD:R_0603_1608Metric, symbol Device:R_Small
- added R31, R32, R46, R48: 33, Resistor_SMD:R_0603_1608Metric, symbol Device:R_Small
- added R4: 64.9k, Resistor_SMD:R_0603_1608Metric, symbol Device:R_Small
- added R6: 1.58k, Resistor_SMD:R_0603_1608Metric, symbol Device:R_Small
- added R8, R9: 2k, Resistor_SMD:R_0603_1608Metric, symbol Device:R_Small
- added SW1: RESET, symbol Switch:SW_Push
- added U2: TPS54336ADDA, Package_SO:TI_SO-PowerPAD-8_ThermalVias, symbol Regulator_Switching:TPS54336ADDA
- added U3: AMS1117-3.3, Package_TO_SOT_SMD:SOT-223-3_TabPin2, symbol Regulator_Linear:AMS1117-3.3
- added U4, U5: TMC2209-LA, Package_DFN_QFN:VQFN-28-1EP_5x5mm_P0.5mm_EP3.7x3.7mm_ThermalVias, symbol Driver_Motor:TMC2209-LA
- added U6: DRV8876PWPR, SOP65P640X120-17N, symbol Library:DRV8876PWPR
- J10, J7: value Conn_01x03 -> B3B-XH-AM
- J13: value Conn_01x02 -> B2B-XH-AM
- J8: value Conn_01x04 -> B4B-XH-AM
- J9: value Conn_01x06 -> B6B-XH-AM
- U1: footprint RUV(R-PVQFN-N36) -> Library:TPS24751RUVR
Connections:
- net at U1.1 (OV): now also R2.2, R3.1
- net at U1.10 (OUT_5): now also U1.11 (OUT_6), U1.12 (OUT_7), U1.13 (OUT_8), U1.19 (OUT_9), U1.20 (OUT_10), U1.21 (OUT_11), U1.22 (OUT_12), U1.23 (OUT_13), U1.24 (OUT_14), U1.6 (OUT_1), U1.7 (OUT_2), U1.8 (OUT_3), U1.9 (OUT_4)
- net +12V: now reaches U1.14 (DRAIN_2)
- net +12V: now also U1.15 (DRAIN_3), U1.16 (DRAIN_4), U1.17 (DRAIN_5), U1.18 (DRAIN_6), U1.26 (SENSE), U1.38 (DRAIN_8), C15.1, C22.1, C23.1, C24.1, C25.1, C26.1, C27.1, C4.1, C45.1, C47.1, C5.1, C50.1, C52.1, C54.1, C58.1, C6.1, C62.1, C63.1, C64.2, C7.1, C8.1, D4.1 (K), R10.1, R5.1, U2.2 (VIN), U4.22 (VS), U4.28 (VS), U5.22 (VS), U5.28 (VS), U6.11 (VM)
- net INPUT_IMON: now reaches U1.2 (IMON)
- net INPUT_IMON: now also R6.1
- net GND: now reaches U1.28 (GND_2)
- net GND: now also J10.3 (Pin_3), J5.1 (Pin_1), J5.2 (Pin_2), J7.3 (Pin_3), J9.5 (Pin_5), U1.32 (GND_3), U1.36 (GND_4), U1.37 (GND_5), U1.4 (GND_1), C1.2, C10.2, C12.2, C13.2, C14.2, C15.2, C16.2, C17.2, C18.2, C19.2, C2.2, C21.2, C23.2, C24.2, C25.2, C26.2, C27.2, C28.2, C29.1, C3.2, C30.1, C31.1, C32.1, C33.2, C34.2, C35.2, C36.2, C37.1, C38.1, C39.1, C4.2, C40.1, C41.2, C42.1, C43.1, C44.1, C46.1, C47.2, C49.1, C5.2, C50.2, C51.1, C52.2, C53.1, C54.2, C55.1, C56.2, C57.2, C58.2, C59.2, C6.2, C60.2, C61.2, C62.2, C63.2, C7.2, C8.2, C9.2, D2.2 (A2), D4.2 (A), D5.1 (K), D6.1 (K), J11.5 (Pin_5), R11.2, R12.2, R14.2, R17.2, R18.2, R21.2, R23.2, R24.2, R28.2, R3.2, R36.2, R38.2, R4.2, R40.2, R41.2, R43.2, R52.2, R53.2, R6.2, SW1.1, U2.4 (GND), U2.9 (ETPAD), U3.1 (GND), U4.13 (CLK), U4.18 (GND), U4.25 (NC), U4.29 (GND), U4.3 (GND), U5.13 (CLK), U5.18 (GND), U5.25 (NC), U5.29 (GND), U5.3 (GND), U6.15 (GND), U6.16 (PMODE), U6.17 (EP), U6.7 (IMODE), U6.9 (PGND)
- net VIN: now reaches U1.29 (VCC)
- net VIN: now also J5.3 (Pin_3), J5.4 (Pin_4), C1.1, C2.1, D2.1 (A1), R1.1, R10.2, R7.2, R8.1, R9.1
- net at U1.3 (SET): now also R7.1
- net at U1.30 (FLTB): now also D3.1 (K)
- net at U1.31 (PGB): now also D1.1 (K)
- net at U1.33 (EN): now also R1.2, R2.1, SW1.2
- net at U1.34 (PROG): now also R4.1
- net at U1.35 (TIMER): now also C3.1
- net at J8.1 (Pin_1): now also C36.1, U5.24 (OA1)
- net at J8.2 (Pin_2): now also C35.1, U5.21 (OA2)
- net at J8.3 (Pin_3): now also C34.1, U5.26 (OB1)
- net at J8.4 (Pin_4): now also C33.1, U5.1 (OB2)
- net X_lLIM_1: now reaches J7.1 (Pin_1)
- net X_lLIM_1: now also C38.2, R26.1
- net X_lLIM_2: now reaches J7.2 (Pin_2)
- net X_lLIM_2: now also C37.2, R30.1
- net at J13.1 (Pin_1): now also U6.10 (OUT2)
- net at J13.2 (Pin_2): now also U6.8 (OUT1)
- net X_ENC_INDEX: now reaches J9.1 (Pin_1)
- net X_ENC_INDEX: now also R34.2
- net X_ENC_CS: now reaches J9.2 (Pin_2)
- net X_ENC_CS: now also R33.2
- net at J9.3 (Pin_3): now also R32.1
- net at J9.4 (Pin_4): now also R31.1
- net +3.3V: now reaches J9.6 (Pin_6)
- net +3.3V: now also C17.1, C19.1, C28.1, C39.2, C40.2, C41.1, C42.2, C43.2, J11.6 (Pin_6), R19.1, R20.1, R22.1, R26.2, R30.2, R33.1, R34.1, R35.1, R37.1, R39.1, R47.2, R49.1, R50.2, R51.1, R54.1, U3.2 (VO), U4.15 (VCC_IO), U5.15 (VCC_IO)
- net Y_lLIM_1: now reaches J10.1 (Pin_1)
- net Y_lLIM_1: now also C46.2, R50.1
- net Y_lLIM_2: now reaches J10.2 (Pin_2)
- net Y_lLIM_2: now also C44.2, R47.1
- new net: C21.1, C30.2, U5.8 (5VOUT)
- new net: J11.3 (Pin_3), R46.1
- new net: J11.4 (Pin_4), R48.1
- new net: R37.2, R38.1, U4.9 (MS1/AD0)
- new net: C32.2, R12.1, U5.27 (BRB)
- new net: R25.2, R29.2, U5.11 (DIAG)
- new net: R20.2, R21.1, U5.9 (MS1/AD0)
- new net: R22.2, R23.1, U5.7 (SPREAD)
- new net: C57.1, J12.1 (Pin_1), U4.24 (OA1)
- new net: C61.1, J12.4 (Pin_4), U4.1 (OB2)
- new net: D5.2 (A), R29.1
- new net: R18.1, R19.2, U5.10 (MS2/AD1)
- new net: C29.2, U5.17 (VREF)
- new net: C31.2, R14.1, U5.23 (BRA)
- new net: C20.1, U5.4 (CPO)
- new net: C20.2, U5.5 (CPI)
- new net: C22.2, U5.6 (VCP)
- new net: C10.1, R13.1, U2.6 (COMP)
- new net: C9.1, R13.2
- new net: R39.2, R40.1, U4.10 (MS2/AD1)
- new net: R44.2, R45.2, U4.11 (DIAG)
- new net: C51.2, U4.17 (VREF)
- new net: C59.1, J12.2 (Pin_2), U4.21 (OA2)
- new net: C55.2, R53.1, U4.23 (BRA)
- new net: C60.1, J12.3 (Pin_3), U4.26 (OB1)
- new net: C49.2, R52.1, U4.27 (BRB)
- new net: C48.1, U4.4 (CPO)
- new net: C48.2, U4.5 (CPI)
- new net: C45.2, U4.6 (VCP)
- new net: R35.2, R36.1, U4.7 (SPREAD)
- new net: C53.2, C56.1, U4.8 (5VOUT)
- new net: R15.2, R16.1
- new net: C11.1, U2.1 (BOOT)
- new net: C11.2, L1.1, U2.3 (PH)
- new net: R16.2, R17.1, U2.5 (VSENSE)
- new net: R11.1, R5.2, U2.7 (EN)
- new net: C12.1, U2.8 (SS)
- new net: D3.2 (A), R8.2
- new net: C65.1, U6.14 (CPL)
- new net: C65.2, U6.13 (CPH)
- new net: D1.2 (A), R9.2
- new net: C64.1, U6.12 (VCP)
- new net: D6.2 (A), R45.1
- new net +5V: C13.1, C14.1, C16.1, C18.1, L1.2, R15.1, U3.3 (VI)
- new net XY_ENC_CLK: R32.2, R46.2
- new net XY_UART_RX: R27.2, R42.2, U4.14 (~{PD}/UART), U5.14 (~{PD}/UART)
- new net XY_UART_TX: R27.1, R42.1
- new net X_DIAG: R25.1
- new net X_EN: R24.1, U5.2 (~{EN})
- new net X_ENC_DO: R31.2
- new net X_STDBY: R28.1, U5.20 (STDBY)
- new net X_STEP: U5.16 (STEP), U5.19 (DIR)
- new net Y_DIAG: R44.1
- new net Y_EN: R41.1, U4.2 (~{EN})
- new net Y_ENC_CS: J11.2 (Pin_2), R51.2
- new net Y_ENC_DO: R48.2
- new net Y_ENC_INDEX: J11.1 (Pin_1), R49.2
- new net Y_STDBY: R43.1, U4.20 (STDBY)
- new net Y_STEP: U4.16 (STEP), U4.19 (DIR)
- new net Z_EN: U6.1 (EN/IN1)
- new net Z_FAULT: R54.2, U6.4 (NFAULT)
- new net Z_PH: U6.2 (PH/IN2)
- new net Z_SLEEP: U6.3 (NSLEEP)
- no-connect marks 0 -> 5
Other:
- note added: "0603"
- note added: "100V"
- note added: "1W"
- note added: "2010"
- note added: "2220"
- note added: "50V"
- moved on the sheet: J1, J13, J14, J15, J16, J17, J18, J19, J2, J20, J21, J3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

Commit message: m
Parts:
- removed D4: MBRS340, Diode_SMD:D_SMC, symbol Diode:MBRS340
- removed J17, J19: Conn_01x02, Library:B2BXHAMLFSN, symbol Connector_Generic:Conn_01x02
- removed J2: 23117633, Library:23117633, symbol Connector:DE15_Socket_HighDensity
- removed J3, J4: 57478404, Library:57478404, symbol Connector:DE9_Pins
- removed J5: 0039301040, Library:0039301040, symbol Connector_Generic:Conn_01x04
- removed R28: 100k, Resistor_SMD:R_0603_1608Metric, symbol Device:R_Small
- removed R31, R32, R46, R48: 33, Resistor_SMD:R_0603_1608Metric, symbol Device:R_Small
- removed U6: DRV8876PWPR, SOP65P640X120-17N, symbol Library:DRV8876PWPR
- added C100, C101, C102, C98: 4.7nF, Capacitor_SMD:C_0805_2012Metric, symbol Device:C_Small
- added C103: 4.7uF, Capacitor_SMD:C_0805_2012Metric, symbol Device:C_Small
- added C104, C105, C106, C107, C108, C109, C110, C112, C113, C60, C63, C66, C67, C74, C75, C76, C77, C79, C80, C82, C83, C84, C86, C87, C89, C90, C91, C92, C93, C94, C95, C96, C97, C99: 100nF, Capacitor_SMD:C_0603_1608Metric, symbol Device:C_Small
- added C111: 1uF, Capacitor_SMD:C_0603_1608Metric, symbol Device:C_Small
- added C114, C115: 10pf, Capacitor_SMD:C_0603_1608Metric, symbol Device:C_Small
- added C116, C117: 2.2uF, Capacitor_SMD:C_1206_3216Metric, symbol Device:C_Small
- added C20, C41: 1uF, Capacitor_SMD:C_1210_3225Metric, symbol Device:C_Small
- added C68, C78, C85: 220uF, Capacitor_SMD:CP_Elec_8x10, symbol Device:C_Polarized_Small
- added C70: 10uF, Capacitor_SMD:C_2220_5750Metric, symbol Device:C_Small
- added C81, C88: 22nF, Capacitor_SMD:C_0603_1608Metric, symbol Device:C_Small
- added D10, D11, D12, D13, D14, D15, D16, D17, D18, D19, D20, D4, D7, D8, D9: CDSOD323-T03C, Diode_SMD:D_SOD-323, symbol Diode:ESD9B5.0ST5G
- added J1: 44068-0057, Library:44068-0057, symbol Connector_Generic:Conn_01x06
- added J11, J14: B2B-XH-AM, Library:B2BXHAMLFSN, symbol Connector_Generic:Conn_01x02
- added J18: B4B-XH-AM, Library:B4BXHAM, symbol Connector_Generic:Conn_01x04
- added J21: 10090929S154VLF, Library:10090929S154VLF, symbol Connector:DE15_Socket_HighDensity_MountingHoles
- added J22, J23: LD09S24A4GV00LF, Library:LD09S24A4GV00LF, symbol Connector:DE9_Pins_MountingHoles
- added L2: FCM1608KF-601T05, Inductor_SMD:L_0603_1608Metric, symbol Device:L_Small
- added Q1: BSS84, Package_TO_SOT_SMD:SOT-23, symbol Transistor_FET:BSS84
- added Q2: 2N7002, Package_TO_SOT_SMD:SOT-23, symbol Transistor_FET:2N7002
- added R10, R100, R102, R11, R110, R12, R27, R44, R64, R74, R83, R84, R85, R86, R87, R88, R95, R96, R97, R98, R99: 10k, Resistor_SMD:R_0603_1608Metric, symbol Device:R_Small
- added R103, R104, R111, R58, R59, R61, R65, R66, R67, R68, R70, R75, R76, R77, R78, R80, R89, R90, R91, R92, R93, R94: 0, Resistor_SMD:R_0603_1608Metric, symbol Device:R_Small
- added R105, R107, R108, R109: 0, Resistor_SMD:R_0805_2012Metric, symbol Device:R_Small
- added R106: 47, Resistor_SMD:R_0603_1608Metric, symbol Device:R_Small
- added R112: 33k, Resistor_SMD:R_0603_1608Metric, symbol Device:R_Small
- added R113: 82k, Resistor_SMD:R_0603_1608Metric, symbol Device:R_Small
- added R128, R129, R130, R131, R132, R133, R134, R135, R136, R137, R138, R139, R140, R141, R142: 1k, Resistor_SMD:R_0805_2012Metric, symbol Device:R_Small
- added R19, R36: 1.1, Resistor_SMD:R_0603_1608Metric, symbol Device:R_Small
- added R33: 100k, Resistor_SMD:R_0603_1608Metric, symbol Device:R_Small
- added R60: 1.62k, Resistor_SMD:R_0603_1608Metric, symbol Device:R_Small
- added R62, R63, R73, R81, R82: 10K, Resistor_SMD:R_0603_1608Metric, symbol Device:R_Small
- added R69, R79: 3.3k, Resistor_SMD:R_0603_1608Metric, symbol Device:R_Small
- added R71, R72: 2.2k, Resistor_SMD:R_0603_1608Metric, symbol Device:R_Small
- added RV1: 10k, Library:3314J-1, symbol Device:R_Potentiometer
- added SW2: SW_Push, Library:SKRKAEE010, symbol Switch:SW_Push
- added SW3: CJS1201A, Library:CJS1201A, symbol Switch:SW_SPDT
- added U10, U12, U13: DRV8876PWPR, Library:SOP65P640X120-17N, symbol Library:DRV8876PWPR
- added U11, U6, U7, U8, U9: SN74LVC2G17DBV, Package_TO_SOT_SMD:SOT-23-6, symbol Library:SN74LVC2G17DBV
- added U14: USBLC6-2SC6, Package_TO_SOT_SMD:SOT-23-6, symbol Power_Protection:USBLC6-2SC6
- added U15: 74LVC1G17, Package_TO_SOT_SMD:SOT-353_SC-70-5, symbol 74xGxx:74LVC1G17
- added U16: STM32F446VETx, Package_QFP:LQFP-100_14x14mm_P0.5mm, symbol MCU_ST_STM32F4:STM32F446VETx
- added Y1: X322516MMB4SI, Library:X322516MMB4SI, symbol Device:Crystal_GND24
- C1: renamed from C2; footprint (none) -> Capacitor_SMD:C_0603_1608Metric
- C10: renamed from C7; footprint (none) -> Capacitor_SMD:C_1210_3225Metric
- C11: renamed from C8; footprint (none) -> Capacitor_SMD:C_1210_3225Metric
- C12: renamed from C15; footprint (none) -> Capacitor_SMD:C_0603_1608Metric
- C13: renamed from C12; footprint (none) -> Capacitor_SMD:C_0603_1608Metric
- C14: renamed from C10; footprint (none) -> Capacitor_SMD:C_0603_1608Metric
- C15: renamed from C9; footprint (none) -> Capacitor_SMD:C_0603_1608Metric
- C16: renamed from C18; footprint (none) -> Capacitor_SMD:C_1210_3225Metric
- C17: renamed from C16; footprint (none) -> Capacitor_SMD:C_0603_1608Metric
- C18: renamed from C19; footprint (none) -> Capacitor_SMD:C_0603_1608Metric
- C19: renamed from C17; footprint (none) -> Capacitor_SMD:C_1210_3225Metric
- C2: renamed from C1; footprint (none) -> Capacitor_SMD:C_1210_3225Metric
- C21: renamed from C28; footprint (none) -> Capacitor_SMD:C_0603_1608Metric
- C22: renamed from C26; footprint (none) -> Capacitor_SMD:C_0603_1608Metric
- C23: renamed from C25; footprint (none) -> Capacitor_SMD:C_2220_5750Metric
- C24: footprint (none) -> Capacitor_SMD:C_2220_5750Metric
- C27: renamed from C22; footprint (none) -> Capacitor_SMD:C_0603_1608Metric
- C28: renamed from C29; footprint (none) -> Capacitor_SMD:C_0603_1608Metric
- C29: renamed from C30; footprint (none) -> Capacitor_SMD:C_0603_1608Metric
- C3: renamed from C4; footprint (none) -> Capacitor_SMD:C_0603_1608Metric
- C30: renamed from C21; footprint (none) -> Capacitor_SMD:C_0805_2012Metric
- C31: renamed from C20; footprint (none) -> Capacitor_SMD:C_0805_2012Metric
- C32: renamed from C36; footprint (none) -> Capacitor_SMD:C_0402_1005Metric
- C33: renamed from C35; footprint (none) -> Capacitor_SMD:C_0402_1005Metric
- C34: footprint (none) -> Capacitor_SMD:C_0402_1005Metric
- C35: renamed from C33; footprint (none) -> Capacitor_SMD:C_0402_1005Metric
- C36: renamed from C32; footprint (none) -> Capacitor_SMD:C_0603_1608Metric
- C37: renamed from C31; footprint (none) -> Capacitor_SMD:C_0603_1608Metric
- C38: renamed from C37; footprint (none) -> Capacitor_SMD:C_0603_1608Metric
- C39: renamed from C38; footprint (none) -> Capacitor_SMD:C_0603_1608Metric
- C40: renamed from C41; footprint (none) -> Capacitor_SMD:C_0603_1608Metric
- C42: renamed from C47; footprint (none) -> Capacitor_SMD:C_0603_1608Metric
- C43: renamed from C50; footprint (none) -> Capacitor_SMD:C_2220_5750Metric
- C44: renamed from C52; footprint (none) -> Capacitor_SMD:C_2220_5750Metric
- C47: renamed from C45; footprint (none) -> Capacitor_SMD:C_0603_1608Metric
- C48: renamed from C51; footprint (none) -> Capacitor_SMD:C_0603_1608Metric
- C49: renamed from C53; footprint (none) -> Capacitor_SMD:C_0603_1608Metric
- C50: renamed from C56; footprint (none) -> Capacitor_SMD:C_0805_2012Metric
- C51: renamed from C48; footprint (none) -> Capacitor_SMD:C_0805_2012Metric
- C52: renamed from C57; footprint (none) -> Capacitor_SMD:C_0402_1005Metric
- C53: renamed from C59; footprint (none) -> Capacitor_SMD:C_0402_1005Metric
- C54: renamed from C60; footprint (none) -> Capacitor_SMD:C_0402_1005Metric
- C55: renamed from C61; footprint (none) -> Capacitor_SMD:C_0402_1005Metric
- C56: renamed from C49; footprint (none) -> Capacitor_SMD:C_0603_1608Metric
- C57: renamed from C55; footprint (none) -> Capacitor_SMD:C_0603_1608Metric
- C58: renamed from C44; footprint (none) -> Capacitor_SMD:C_0603_1608Metric
- C59: renamed from C46; footprint (none) -> Capacitor_SMD:C_0603_1608Metric
- C6: renamed from C3; footprint (none) -> Capacitor_SMD:C_0603_1608Metric
- C61: renamed from C40; footprint (none) -> Capacitor_SMD:C_0603_1608Metric
- C62: renamed from C39; footprint (none) -> Capacitor_SMD:C_0201_0603Metric
- C64: renamed from C42; footprint (none) -> Capacitor_SMD:C_0603_1608Metric
- C65: renamed from C43; footprint (none) -> Capacitor_SMD:C_0603_1608Metric
- C7: renamed from C11; footprint (none) -> Capacitor_SMD:C_0603_1608Metric
- C71: renamed from C63; footprint (none) -> Capacitor_SMD:C_0603_1608Metric
- C72: renamed from C64; footprint (none) -> Capacitor_SMD:C_0603_1608Metric
- C73: renamed from C65; footprint (none) -> Capacitor_SMD:C_0603_1608Metric
- C8: renamed from C13; footprint (none) -> Capacitor_SMD:C_1206_3216Metric
- C9: renamed from C14; footprint (none) -> Capacitor_SMD:C_1206_3216Metric
- D1: renamed from D3; footprint LED_SMD:LED_0805_2012Metric -> LED_SMD:LED_0603_1608Metric
- D2: renamed from D1; footprint LED_SMD:LED_0805_2012Metric -> LED_SMD:LED_0603_1608Metric
- D5, D6: footprint LED_SMD:LED_0805_2012Metric -> LED_SMD:LED_0603_1608Metric
- J10: renamed from J14; value Conn_01x03 -> B3B-XH-AM
- J12: renamed from J18; value Conn_01x04 -> B4B-XH-AM
- J13: renamed from J16; value Conn_01x02 -> B2B-XH-AM
- J15: renamed from J20; value Conn_01x03 -> B3B-XH-AM
- J16: renamed from J21; value Conn_01x10 -> B10B-XH-AM
- J19: renamed from J1; value 670689000 -> 5787834-1; footprint Library:670689000 -> Library:5787834-1
- J20: renamed from J6; value Conn_Coaxial -> 031532951RFX; footprint (none) -> Library:031532951RFX
- J9: renamed from J15; value Conn_01x04 -> B4B-XH-AM
- R14: renamed from R5; value ~ -> (none)
- R17: renamed from R11; value ~ -> (none)
- SW1: footprint (none) -> Library:SKRKAEE010
- renumbered C23 to C25, C27 to C26, C5 to C4, C54 to C45, C58 to C46, C6 to C5, C62 to C69, D2 to D3, J8 to J2, J7 to J3, J12 to J4, J10 to J5, J9 to J6, J11 to J7, J13 to J8, R10 to R1, R15 to R13, R16 to R15, R13 to R16, R17 to R18, R8 to R2, R22 to R20, R20 to R21, R19 to R22, R27 to R23, R23 to R24, R21 to R25, R18 to R26, R25 to R28, R9 to R3, R12 to R30, R14 to R31, R24 to R32, R30 to R34, R26 to R35, R35 to R37, R37 to R38, R7 to R4, R42 to R40, R36 to R41, R38 to R42, R40 to R43, R44 to R45, R41 to R46, R43 to R47, R45 to R48, R52 to R49, R1 to R5, R53 to R50, R47 to R51, R50 to R52, R34 to R53, R33 to R54, R49 to R55, R51 to R56, R54 to R57, R2 to R6, R3 to R7, R4 to R8, R6 to R9, U5 to U4, U4 to U5
Connections:
- net +12V: now also J16.1 (Pin_1), U1.10 (OUT_5), U1.11 (OUT_6), U1.12 (OUT_7), U1.13 (OUT_8), U1.19 (OUT_9), U1.20 (OUT_10), U1.21 (OUT_11), U1.22 (OUT_12), U1.23 (OUT_13), U1.24 (OUT_14), U1.6 (OUT_1), U1.7 (OUT_2), U1.8 (OUT_3), U1.9 (OUT_4), C20.1, C41.1, C68.1, C70.1, C78.1, C79.1, C80.2, C85.1, C86.1, C87.2, J21.6, J21.7, J22.9, J23.9, U10.11 (VM), U12.11 (VM), U13.11 (VM); no longer R1.1, U1.14 (DRAIN_2), U1.15 (DRAIN_3), U1.16 (DRAIN_4), U1.17 (DRAIN_5), U1.18 (DRAIN_6), U1.26 (SENSE), U1.38 (DRAIN_8)
- net +3.3V: now also J12.1 (Pin_1), J16.2 (Pin_2), C103.2, C104.2, C105.2, C106.2, C107.2, C108.2, C109.2, C60.2, C63.2, C66.2, C67.2, C74.2, C82.2, C83.2, C99.2, L2.2, R111.1, R112.2, R27.2, R44.2, R58.1, R62.2, R63.2, R64.1, R65.1, R66.1, R71.2, R72.2, R73.2, R74.1, R75.1, R76.1, R81.2, R82.2, R83.1, R84.1, R85.1, R86.1, R87.1, R88.1, RV1.1, SW3.3 (C), U11.5 (V_{CC}), U15.5 (VCC), U16.100 (VDD), U16.11 (VDD), U16.19 (VDD), U16.28 (VDD), U16.50 (VDD), U16.75 (VDD), U6.5 (V_{CC}), U7.5 (V_{CC}), U8.5 (V_{CC}), U9.5 (V_{CC})
- net +5V: now also J18.3 (Pin_3), J21.10, J22.1, J23.1, R102.2; no longer C16.1, C17.1, U3.3 (VI)
- net GND: now also J10.3 (Pin_3), J12.4 (Pin_4), J13.2 (Pin_2), J15.3 (Pin_3), J16.3 (Pin_3), J16.4 (Pin_4), J19.4 (GND), J20.2 (Ext), J20.3 (Ext), J20.4 (Ext), J20.5 (Ext), J9.4 (Pin_4), C100.1, C101.2, C102.2, C103.1, C104.1, C105.1, C106.1, C107.1, C108.1, C109.1, C110.1, C111.1, C112.1, C113.1, C114.1, C115.1, C116.1, C117.1, C60.1, C63.1, C66.1, C67.1, C68.2, C70.2, C74.1, C75.1, C76.1, C77.1, C78.2, C79.2, C82.1, C83.1, C84.1, C85.2, C86.2, C89.1, C90.1, C91.1, C92.1, C93.1, C94.1, C95.1, C96.1, C97.1, C98.1, C99.1, D10.2 (A2), D11.2 (A2), D12.2 (A2), D13.2 (A2), D14.2 (A2), D15.2 (A2), D16.2 (A2), D17.2 (A2), D18.2 (A2), D19.2 (A2), D20.2 (A2), D4.2 (A2), D7.2 (A2), D8.2 (A2), D9.2 (A2), J1.2 (Pin_2), J1.3 (Pin_3), J18.4 (Pin_4), J21.11, J21.12, J21.13, J21.14, J21.15, J22.6, J22.7, J22.8, J23.6, J23.7, J23.8, Q2.2 (S), R100.2, R105.1, R107.1, R108.2, R109.2, R11.1, R113.1, R12.1, R19.2, R33.2, R36.2, R59.2, R60.2, R61.2, R67.2, R68.2, R69.2, R70.2, R77.2, R78.2, R79.2, R80.2, R95.2, R96.2, R97.2, R98.2, R99.2, RV1.3, SW2.1, SW3.1 (A), U10.15 (GND), U10.17 (EP), U10.9 (PGND), U11.2 (GND), U12.15 (GND), U12.17 (EP), U12.9 (PGND), U13.15 (GND), U13.17 (EP), U13.9 (PGND), U14.2 (GND), U15.3 (GND), U16.10 (VSS), U16.20 (VSSA), U16.27 (VSS), U16.49 (VSS), U16.74 (VSS), U16.99 (VSS), U6.2 (GND), U7.2 (GND), U8.2 (GND), U9.2 (GND), Y1.2 (G), Y1.4 (G)
- net VIN: now also J1.5 (Pin_5), J1.6 (Pin_6)
- net XY_ENC_CLK: now also U7.1 (1A), U9.1 (1A)
- net X_ENC_CS: now also U7.3 (2A); no longer J6.2 (Pin_2), R54.2
- net X_ENC_DO: now also U6.6 (1Y)
- net X_ENC_INDEX: now also U6.4 (2Y); no longer J6.1 (Pin_1), R53.2
- net X_STDBY: now also R27.1, R33.1
- net X_STEP: no longer U4.19 (DIR)
- net X_lLIM_1: now also J10.1 (Pin_1), C77.2, R63.1
- net X_lLIM_2: now also J10.2 (Pin_2), C76.2, R62.1
- net Y_ENC_CS: now also U9.3 (2A); no longer J7.2 (Pin_2), R56.2
- net Y_ENC_DO: now also U8.6 (1Y)
- net Y_ENC_INDEX: now also U8.4 (2Y); no longer J7.1 (Pin_1), R55.2
- net Y_STDBY: now also R44.1
- net Y_STEP: no longer U5.19 (DIR)
- net Z_EN: now also U10.1 (EN/IN1), U10.3 (NSLEEP)
- net Z_FAULT: now also U10.4 (NFAULT)
- net Z_PH: now also U10.2 (PH/IN2)
- net Y_ENC_CLK_OUTPUT: now reaches J7.3 (Pin_3)
- net Y_ENC_CLK_OUTPUT: now also U9.6 (1Y)
- net Y_ENC_DO_INPUT: now reaches J7.4 (Pin_4)
- net Y_ENC_DO_INPUT: now also U8.1 (1A)
- net at J20.1 (In): now also R106.1
- net X_ENC_DO_INPUT: now reaches J6.4 (Pin_4)
- net X_ENC_DO_INPUT: now also U6.1 (1A)
- net X_ENC_CLK_OUTPUT: now reaches J6.3 (Pin_3)
- net X_ENC_CLK_OUTPUT: now also U7.6 (1Y)
- net at C73.1: now also U10.14 (CPL)
- net at C73.2: now also U10.13 (CPH)
- net at J8.1 (Pin_1): now also U10.8 (OUT1)
- net at J8.2 (Pin_2): now also U10.10 (OUT2)
- net J_lLIM: now reaches J13.1 (Pin_1)
- net J_lLIM: now also C84.2, R73.1
- net F_lLIM_1: now reaches J15.1 (Pin_1)
- net F_lLIM_1: now also C90.2, R82.1
- net F_lLIM_2: now reaches J15.2 (Pin_2)
- net F_lLIM_2: now also C89.2, R81.1
- net at C72.1: now also U10.12 (VCP)
- net USB_VBUS: now reaches J19.1 (VBUS)
- net USB_VBUS: now also C97.2, R112.1, R113.2, U14.5 (VBUS), U16.68 (PA9)
- net at J19.2 (D-): now also U14.3 (I/O2)
- net at J19.3 (D+): now also U14.1 (I/O1)
- net USB_SH: now reaches J19.5 (Shield)
- net USB_SH: now also J19.6 (Shield), C98.2, R105.2
- net +5VSB: now reaches J9.1 (Pin_1)
- net +5VSB: now also C16.1, C17.1, U3.3 (VI), C75.2, J1.4 (Pin_4), Q1.2 (S), R10.2
- net at J9.2 (Pin_2): now also U11.1 (1A)
- net at J9.3 (Pin_3): now also U11.3 (2A)
- net at J16.10 (Pin_10): now also R94.1
- net at J16.5 (Pin_5): now also R89.1
- net at J16.6 (Pin_6): now also R90.1
- net at J16.7 (Pin_7): now also R91.1
- net at J16.8 (Pin_8): now also R92.1
- net at J16.9 (Pin_9): now also R93.1
- net SDA: now reaches J12.2 (Pin_2)
- net SDA: now also J12.3 (Pin_3), R71.1, R72.1
- new net: R76.2, R78.1, U13.16 (PMODE)
- new net: R106.2, U15.4
- new net: J21.2, R129.1
- new net: R58.2, R59.1, U10.16 (PMODE)
- new net: RV1.2, U10.5 (VREF)
- new net: R61.1, U10.7 (IMODE)
- new net: J23.4, R136.1
- new net: J23.2, R138.1
- new net: R65.2, R67.1, U12.5 (VREF)
- new net: R75.2, R77.1, U13.5 (VREF)
- new net: R1.1, U1.14 (DRAIN_2), U1.15 (DRAIN_3), U1.16 (DRAIN_4), U1.17 (DRAIN_5), U1.18 (DRAIN_6), U1.26 (SENSE), U1.38 (DRAIN_8)
- new net: C117.2, U16.73 (VCAP_2)
- new net: Q1.1 (G), Q2.3 (D), R10.1
- new net: J14.1 (Pin_1), U13.8 (OUT1)
- new net: J14.2 (Pin_2), U13.10 (OUT2)
- new net: J21.1, R128.1
- new net: C115.2, U16.13 (PH1), Y1.3
- new net: C20.2, R19.1
- new net: C88.1, U13.14 (CPL)
- new net: C88.2, U13.13 (CPH)
- new net: R104.2, U14.4 (I/O2)
- new net: R103.2, U14.6 (I/O1)
- new net: J22.5, R139.1
- new net: C114.2, U16.12 (PH0), Y1.1
- new net: J23.3, R137.1
- new net: J22.4, R140.1
- new net: J23.5, R135.1
- new net: J21.9, R132.1
- new net: J22.2, R142.1
- new net: J22.3, R141.1
- new net: R66.2, R68.1, U12.16 (PMODE)
- new net: J21.3, R131.1
- new net: J21.4, R133.1
- new net: J21.5, R134.1
- new net: J21.8, R130.1
- new net: C41.2, R36.1
- new net: C116.2, U16.48 (VCAP_1)
- new net: C81.1, U12.14 (CPL)
- new net: C81.2, U12.13 (CPH)
- new net: C87.1, U13.12 (VCP)
- new net: R110.2, U16.94 (BOOT0)
- new net: J11.2 (Pin_2), U12.10 (OUT2)
- new net: C80.1, U12.12 (VCP)
- new net: R70.1, U12.7 (IMODE)
- new net: J11.1 (Pin_1), U12.8 (OUT1)
- new net: R110.1, SW3.2 (B)
- new net: R80.1, U13.7 (IMODE)
- new net ACC1_GPIO_1: D13.1 (A1), D8.1 (A1), R135.2, R139.2
- new net ACC1_GPIO_2: D12.1 (A1), D7.1 (A1), R136.2, R140.2
- new net ACC1_SH: C102.1, J23.MH1 (PAD), J23.MH2 (PAD), R109.1
- new net ACC1_UART_RX: D10.1 (A1), D9.1 (A1), R138.2, R142.2
- new net ACC1_UART_TX: D11.1 (A1), D4.1 (A1), R137.2, R141.2
- new net ACC2_SH: C101.1, J22.MH1 (PAD), J22.MH2 (PAD), R108.1
- new net EXP_GPIO_1: C96.2, R88.2, R89.2
- new net EXP_GPIO_2: C95.2, R87.2, R90.2, R99.1
- new net EXP_GPIO_3: C94.2, R86.2, R91.2, R98.1
- new net EXP_GPIO_4: C93.2, R85.2, R92.2, R97.1
- new net EXP_GPIO_5: C92.2, R84.2, R93.2, R96.1
- new net EXP_GPIO_6: C91.2, R100.1, R83.2, R94.2, R95.1
- new net FAN1_PWM: J18.1 (Pin_1)
- new net FAN1_RPM: J18.2 (Pin_2), R102.1
- new net F_EN: U13.1 (EN/IN1), U13.3 (NSLEEP)
- new net F_FAULT: R74.2, U13.4 (NFAULT)
- new net F_PH: U13.2 (PH/IN2)
- new net F_SENSE: R79.1, U13.6 (IPROPI)
- new net J_EN: U12.1 (EN/IN1), U12.3 (NSLEEP)
- new net J_FAULT: R64.2, U12.4 (NFAULT)
- new net J_PH: U12.2 (PH/IN2)
- new net J_SENSE: R69.1, U12.6 (IPROPI)
- new net MCU_RESET: C113.2, SW2.2, U16.14 (NRST)
- new net PSU_EN: J1.1 (Pin_1), Q1.3 (D), R11.2
- new net PWR_EN: Q2.1 (G), R12.2
- new net REMOTE_GPIO_1: D18.1 (A1), R130.2
- new net REMOTE_GPIO_2: D17.1 (A1), R131.2
- new net REMOTE_GPIO_3: D16.1 (A1), R132.2
- new net REMOTE_GPIO_4: D15.1 (A1), R133.2
- new net REMOTE_GPIO_5: D14.1 (A1), R134.2
- new net REMOTE_SH: C100.2, J21.MH1, J21.MH2, R107.2
- new net REMOTE_UART_RX: D19.1 (A1), R129.2
- new net REMOTE_UART_TX: D20.1 (A1), R128.2
- new net SWCLK: U16.76 (PA14)
- new net SWDIO: U16.72 (PA13)
- new net SWO: U16.89 (PB3)
- new net SYNC_OUT: U15.2
- new net USB_N: R104.1, U16.71 (PA12)
- new net USB_P: R103.1, R111.2, U16.70 (PA11)
- new net VDDA: C110.2, C111.2, C112.2, L2.1, U16.21 (VREF+), U16.22 (VDDA), U16.6 (VBAT)
- new net X_DIR: U4.19 (DIR)
- new net X_ENC_CS_OUTPUT: J6.2 (Pin_2), R54.2, U7.4 (2Y)
- new net X_ENC_INDEX_INPUT: J6.1 (Pin_1), R53.2, U6.3 (2A)
- new net Y_DIR: U5.19 (DIR)
- new net Y_ENC_CS_OUTPUT: J7.2 (Pin_2), R56.2, U9.4 (2Y)
- new net Y_ENC_INDEX_INPUT: J7.1 (Pin_1), R55.2, U8.3 (2A)
- new net Z_ENC_A: U11.6 (1Y)
- new net Z_ENC_B: U11.4 (2Y)
- new net Z_SENSE: R60.1, U10.6 (IPROPI)
- no-connect marks 5 -> 78
Other:
- moved on the sheet: C1, C10, C11, C12, C13, C14, C15, C16, C17, C18, C19, C2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

Commit message: m
Parts:
- removed C1, C104, C105, C106, C107, C108, C109, C110, C112, C113, C12, C17, C18, C21, C22, C27, C28, C29, C3, C36, C37, C38, C39, C40, C42, C47, C48, C49, C56, C57, C58, C59, C60, C63, C65, C66, C67, C7, C71, C72, C74, C75, C76, C77, C79, C80, C82, C83, C84, C86, C87, C89, C90, C91, C92, C93, C94, C95, C96, C97, C99: 100nF, Capacitor_SMD:C_0603_1608Metric, symbol Device:C_Small
- removed C10, C11, C16: 10uF, Capacitor_SMD:C_1210_3225Metric, symbol Device:C_Small
- removed C100, C101, C102, C98: 4.7nF, Capacitor_SMD:C_0805_2012Metric, symbol Device:C_Small
- removed C103, C30, C50: 4.7uF, Capacitor_SMD:C_0805_2012Metric, symbol Device:C_Small
- removed C111, C61, C64: 1uF, Capacitor_SMD:C_0603_1608Metric, symbol Device:C_Small
- removed C114, C115: 10pf, Capacitor_SMD:C_0603_1608Metric, symbol Device:C_Small
- removed C116, C117: 2.2uF, Capacitor_SMD:C_1206_3216Metric, symbol Device:C_Small
- removed C13: 10nF, Capacitor_SMD:C_0603_1608Metric, symbol Device:C_Small
- removed C14: 120pF, Capacitor_SMD:C_0603_1608Metric, symbol Device:C_Small
- removed C15: 12nF, Capacitor_SMD:C_0603_1608Metric, symbol Device:C_Small
- removed C19, C2: 22uF, Capacitor_SMD:C_1210_3225Metric, symbol Device:C_Small
- removed C20, C41: 1uF, Capacitor_SMD:C_1210_3225Metric, symbol Device:C_Small
- removed C23, C24, C43, C44, C70: 10uF, Capacitor_SMD:C_2220_5750Metric, symbol Device:C_Small
- removed C25, C26, C45, C46: 100uF, Capacitor_SMD:CP_Elec_8x10, symbol Device:C_Polarized_Small
- removed C31, C51: 22nF, Capacitor_SMD:C_0805_2012Metric, symbol Device:C_Small
- removed C32, C33, C34, C35, C52, C53, C54, C55: 470pF, Capacitor_SMD:C_0402_1005Metric, symbol Device:C_Small
- removed C4, C5, C68, C69, C78, C85: 220uF, Capacitor_SMD:CP_Elec_8x10, symbol Device:C_Polarized_Small
- removed C6: 33nF, Capacitor_SMD:C_0603_1608Metric, symbol Device:C_Small
- removed C62: 100nF, Capacitor_SMD:C_0201_0603Metric, symbol Device:C_Small
- removed C73, C81, C88: 22nF, Capacitor_SMD:C_0603_1608Metric, symbol Device:C_Small
- removed C8, C9: 47uF, Capacitor_SMD:C_1206_3216Metric, symbol Device:C_Small
- removed D1, D5, D6: RED, LED_SMD:LED_0603_1608Metric, symbol Device:LED
- removed D10, D11, D12, D13, D14, D15, D16, D17, D18, D19, D20, D4, D7, D8, D9: CDSOD323-T03C, Diode_SMD:D_SOD-323, symbol Diode:ESD9B5.0ST5G
- removed D2: GREEN, LED_SMD:LED_0603_1608Metric, symbol Device:LED
- removed D3: SMAJ15A, Diode_SMD:D_SMA, symbol Diode:SMAJ15A
- removed J1: 44068-0057, Library:44068-0057, symbol Connector_Generic:Conn_01x06
- removed J10, J15, J3, J5: B3B-XH-AM, Library:B3BXHAMLFSN, symbol Connector_Generic:Conn_01x03
- removed J11, J13, J14, J8: B2B-XH-AM, Library:B2BXHAMLFSN, symbol Connector_Generic:Conn_01x02
- removed J12, J18, J2, J4, J9: B4B-XH-AM, Library:B4BXHAM, symbol Connector_Generic:Conn_01x04
- removed J16: B10B-XH-AM, Library:B10BXHAMLFSN, symbol Connector_Generic:Conn_01x10
- removed J19: 5787834-1, Library:5787834-1, symbol Connector:USB_B
- removed J20: 031532951RFX, Library:031532951RFX, symbol Library:Conn_Coaxial
- removed J21: 10090929S154VLF, Library:10090929S154VLF, symbol Connector:DE15_Socket_HighDensity_MountingHoles
- removed J22, J23: LD09S24A4GV00LF, Library:LD09S24A4GV00LF, symbol Connector:DE9_Pins_MountingHoles
- removed J6, J7: B6B-XH-AM, Library:B6BXHAMLFSN, symbol Connector_Generic:Conn_01x06
- removed L1: 15uH, Library:XAL6060153MEC, symbol Device:L_Iron
- removed L2: FCM1608KF-601T05, Inductor_SMD:L_0603_1608Metric, symbol Device:L_Small
- removed Q1: BSS84, Package_TO_SOT_SMD:SOT-23, symbol Transistor_FET:BSS84
- removed Q2: 2N7002, Package_TO_SOT_SMD:SOT-23, symbol Transistor_FET:2N7002
- removed R1: 0.002, Resistor_SMD:R_2512_6332Metric, symbol Device:R_Small
- removed R10, R100, R102, R11, R110, R12, R27, R44, R53, R54, R55, R56, R57, R6, R64, R74, R83, R84, R85, R86, R87, R88, R95, R96, R97, R98, R99: 10k, Resistor_SMD:R_0603_1608Metric, symbol Device:R_Small
- removed R103, R104, R111, R20, R21, R22, R24, R25, R26, R28, R37, R38, R39, R41, R42, R43, R45, R58, R59, R61, R65, R66, R67, R68, R70, R75, R76, R77, R78, R80, R89, R90, R91, R92, R93, R94: 0, Resistor_SMD:R_0603_1608Metric, symbol Device:R_Small
- removed R105, R107, R108, R109: 0, Resistor_SMD:R_0805_2012Metric, symbol Device:R_Small
- removed R106: 47, Resistor_SMD:R_0603_1608Metric, symbol Device:R_Small
- removed R112: 33k, Resistor_SMD:R_0603_1608Metric, symbol Device:R_Small
- removed R113: 82k, Resistor_SMD:R_0603_1608Metric, symbol Device:R_Small
- removed R128, R129, R130, R131, R132, R133, R134, R135, R136, R137, R138, R139, R140, R141, R142: 1k, Resistor_SMD:R_0805_2012Metric, symbol Device:R_Small
- removed R13, R4: 51.1, Resistor_SMD:R_0603_1608Metric, symbol Device:R_Small
- removed R14, R17: (no value), Resistor_SMD:R_0603_1608Metric, symbol Device:R_Small
- removed R15, R33, R47: 100k, Resistor_SMD:R_0603_1608Metric, symbol Device:R_Small
- removed R16: 3.74k, Resistor_SMD:R_0603_1608Metric, symbol Device:R_Small
- removed R18: 19.1k, Resistor_SMD:R_0603_1608Metric, symbol Device:R_Small
- removed R19, R36: 1.1, Resistor_SMD:R_0603_1608Metric, symbol Device:R_Small
- removed R2, R3: 2k, Resistor_SMD:R_0603_1608Metric, symbol Device:R_Small
- removed R23, R40: 1k, Resistor_SMD:R_0603_1608Metric, symbol Device:R_Small
- removed R29, R48: 1K, Resistor_SMD:R_0603_1608Metric, symbol Device:R_Small
- removed R30, R31, R49, R50: 0.1, Resistor_SMD:R_0603_1608Metric, symbol Device:R_Small
- removed R32, R46: 20k, Resistor_SMD:R_0603_1608Metric, symbol Device:R_Small
- removed R34, R35, R51, R52, R62, R63, R73, R81, R82: 10K, Resistor_SMD:R_0603_1608Metric, symbol Device:R_Small
- removed R5: 15k, Resistor_SMD:R_0603_1608Metric, symbol Device:R_Small
- removed R60: 1.62k, Resistor_SMD:R_0603_1608Metric, symbol Device:R_Small
- removed R69, R79: 3.3k, Resistor_SMD:R_0603_1608Metric, symbol Device:R_Small
- removed R7: 130k, Resistor_SMD:R_0603_1608Metric, symbol Device:R_Small
- removed R71, R72: 2.2k, Resistor_SMD:R_0603_1608Metric, symbol Device:R_Small
- removed R8: 64.9k, Resistor_SMD:R_0603_1608Metric, symbol Device:R_Small
- removed R9: 1.58k, Resistor_SMD:R_0603_1608Metric, symbol Device:R_Small
- removed RV1: 10k, Library:3314J-1, symbol Device:R_Potentiometer
- removed SW1: RESET, Library:SKRKAEE010, symbol Switch:SW_Push
- removed SW2: SW_Push, Library:SKRKAEE010, symbol Switch:SW_Push
- removed SW3: CJS1201A, Library:CJS1201A, symbol Switch:SW_SPDT
- removed U1: TPS24751RUVR, Library:TPS24751RUVR, symbol Library:TPS24751RUVR
- removed U10, U12, U13: DRV8876PWPR, Library:SOP65P640X120-17N, symbol Library:DRV8876PWPR
- removed U11, U6, U7, U8, U9: SN74LVC2G17DBV, Package_TO_SOT_SMD:SOT-23-6, symbol Library:SN74LVC2G17DBV
- removed U14: USBLC6-2SC6, Package_TO_SOT_SMD:SOT-23-6, symbol Power_Protection:USBLC6-2SC6
- removed U15: 74LVC1G17, Package_TO_SOT_SMD:SOT-353_SC-70-5, symbol 74xGxx:74LVC1G17
- removed U16: STM32F446VETx, Package_QFP:LQFP-100_14x14mm_P0.5mm, symbol MCU_ST_STM32F4:STM32F446VETx
- removed U2: TPS54336ADDA, Package_SO:TI_SO-PowerPAD-8_ThermalVias, symbol Regulator_Switching:TPS54336ADDA
- removed U3: AMS1117-3.3, Package_TO_SOT_SMD:SOT-223-3_TabPin2, symbol Regulator_Linear:AMS1117-3.3
- removed U4, U5: TMC2209-LA, Package_DFN_QFN:VQFN-28-1EP_5x5mm_P0.5mm_EP3.7x3.7mm_ThermalVias, symbol Driver_Motor:TMC2209-LA
- removed Y1: X322516MMB4SI, Library:X322516MMB4SI, symbol Device:Crystal_GND24
Connections:
- no-connect marks 78 -> 0
Other:
- added sheet DC_DRIVERS (DC_DRIVERS.kicad_sch)
- added sheet IO (IO.kicad_sch)
- added sheet LIM_ENC (LIM_ENC.kicad_sch)
- added sheet MCU (MCU.kicad_sch)
- added sheet POWER_INPUT (POWER_INPUT.kicad_sch)
- added sheet PWR_REG (PWR_REG.kicad_sch)
- added sheet X_Driver (X_Driver.kicad_sch)
- added sheet Y_DRIVER (Y_DRIVER.kicad_sch)
- note removed: "0603"
- note removed: "100V"
- note removed: "1W"
- note removed: "2010"
- note removed: "2220"
- note removed: "50V"

Commit message: m
Other:
- sheet IO ports: added none; removed ACC1_GPIO1, ACC1_GPIO2, ACC1_RX, ACC1_TX, ACC2_GPIO1, ACC2_GPIO2, ACC2_RX, ACC2_TX, REMOTE_GPIO1, REMOTE_GPIO2, REMOTE_GPIO3, REMOTE_GPIO4, REMOTE_GPIO5, REMOTE_RX, REMOTE_TX
Changed lines of the file:
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@@
-			)
-		)
-		(pin "ACC1_GPIO1" bidirectional
-			(at 132.08 152.4 90)
-			(effects
-				(font
-					(size 1.27 1.27)
-				)
-				(justify right)
-			)
-		)
-		(pin "ACC1_GPIO2" bidirectional
-			(at 134.62 152.4 90)
-			(effects
-				(font
-					(size 1.27 1.27)
-				)
-				(justify right)
-			)
-		)
-		(pin "ACC1_RX" input
-			(at 129.54 152.4 90)
-			(effects
-				(font
-					(size 1.27 1.27)
-				)
-				(justify right)
-			)
-		)
-		(pin "ACC1_TX" output
-			(at 127 152.4 90)
-			(effects
-				(font
-					(size 1.27 1.27)
-				)
-				(justify right)
-			)
-		)
-		(pin "ACC2_GPIO1" bidirectional
-			(at 143.51 152.4 90)
-			(effects
-				(font
-					(size 1.27 1.27)
-				)
-				(justify right)
-			)
-		)
-		(pin "ACC2_GPIO2" bidirectional
-			(at 146.05 152.4 90)
-			(effects
-				(font
-					(size 1.27 1.27)
-				)
-				(justify right)
-			)
-		)
-		(pin "ACC2_RX" input
-			(at 140.97 152.4 90)
-			(effects
-				(font
-					(size 1.27 1.27)
-				)
-				(justify right)
-			)
-		)
-		(pin "ACC2_TX" output
-			(at 138.43 152.4 90)
-			(effects
-				(font
-					(size 1.27 1.27)
-				)
-				(justify right)
-			)
-		)
-		(pin "REMOTE_GPIO1" bidirectional
-			(at 158.75 152.4 90)
-			(effects
-				(font
-					(size 1.27 1.27)
-				)
-				(justify right)
-			)
-		)
-		(pin "REMOTE_GPIO2" bidirectional
-			(at 161.29 152.4 90)
-			(effects
-				(font
-					(size 1.27 1.27)
-				)
-				(justify right)
-			)
-		)
-		(pin "REMOTE_GPIO3" bidirectional
-			(at 163.83 152.4 90)
-			(effects
-				(font
-					(size 1.27 1.27)
-				)
-				(justify right)
-			)
-		)
-		(pin "REMOTE_GPIO4" bidirectional
-			(at 166.37 152.4 90)
-			(effects
-				(font
-					(size 1.27 1.27)
-				)
-				(justify right)
-			)
-		)
-		(pin "REMOTE_GPIO5" bidirectional
-			(at 168.91 152.4 90)
-			(effects
-				(font
-					(size 1.27 1.27)
-				)
-				(justify right)
-			)
-		)
-		(pin "REMOTE_RX" input
-			(at 156.21 152.4 90)
-			(effects
-				(font
-					(size 1.27 1.27)
-				)
-				(justify right)
-			)
-		)
-		(pin "REMOTE_TX" output
-			(at 153.67 152.4 90)
-			(effects
-				(font
-					(size 1.27 1.27)
-				)
-				(justify right)
 			)
 		)
