File: hardware/Ziess-Microsope-Controller_Main_board/Ziess-Microsope-Controller_Main_board.kicad_sch (KiCad schematic)
At the start: 0 parts

Commit message: m
Parts:
- added H1, H2, H3, H4: MountingHole, MountingHole:MountingHole_3.2mm_M3_DIN965_Pad_TopBottom, symbol Mechanical:MountingHole

Commit message: m
Parts:
- removed H1, H2, H3, H4: MountingHole, MountingHole:MountingHole_3.2mm_M3_DIN965_Pad_TopBottom, symbol Mechanical:MountingHole
- added H1, H2, H3, H4: MountingHole_Pad, MountingHole:MountingHole_3.2mm_M3_DIN965_Pad_TopBottom, symbol Mechanical:MountingHole_Pad
Connections:
- new net GND: H1.1, H2.1, H3.1, H4.1

Commit message: m
Other:
- sheet X_Driver renamed X_DRIVER
- removed sheet IO
- added sheet ACC1 (ACC1.kicad_sch)
- added sheet ACC2 (ACC2.kicad_sch)
- added sheet ACC3 (ACC3.kicad_sch)
- added sheet USB_SYNC (USB_SYNC.kicad_sch)
- sheet X_DRIVER: file X_Driver.kicad_sch -> X_DRIVER.kicad_sch
- moved on the sheet: H1, H2, H3, H4
