File: hardware/Ziess-Microsope-Controller_Main_board/Ziess-Microsope-Controller_Main_board.kicad_sch (KiCad schematic)
At the start: 4 parts

Commit message: m
Other:
- sheet POWER_INPUT ports: added 12V_SENSE; removed none
- sheet PWR_REG ports: added 5V_PG; removed 12V_PRES
- moved on the sheet: H1, H2, H3, H4
Changed lines of the file:
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@@
 	)
 	(junction
-		(at -10.16 170.18)
+		(at 63.5 172.72)
 		(diameter 0)
 		(color 0 0 0 0)
 	)
 	(junction
-		(at -10.16 165.1)
+		(at 63.5 167.64)
 		(diameter 0)
 		(color 0 0 0 0)
@@
 	)
 	(junction
-		(at -10.16 175.26)
+		(at 63.5 177.8)
 		(diameter 0)
 		(color 0 0 0 0)
@@
 	(wire
 		(pts
-			(xy -12.7 175.26) (xy -10.16 175.26)
+			(xy 60.96 177.8) (xy 63.5 177.8)
 		)
 		(stroke
@@
 	(wire
 		(pts
-			(xy -12.7 160.02) (xy -10.16 160.02)
+			(xy 60.96 162.56) (xy 63.5 162.56)
 		)
 		(stroke
@@
 	(wire
 		(pts
-			(xy -12.7 165.1) (xy -10.16 165.1)
+			(xy 60.96 167.64) (xy 63.5 167.64)
 		)
 		(stroke
@@
 	(wire
 		(pts
-			(xy -12.7 170.18) (xy -10.16 170.18)
+			(xy 60.96 172.72) (xy 63.5 172.72)
 		)
 		(stroke
@@
 	(wire
 		(pts
-			(xy -10.16 165.1) (xy -10.16 170.18)
+			(xy 63.5 167.64) (xy 63.5 172.72)
 		)
 		(stroke
@@
 	(wire
 		(pts
-			(xy -10.16 175.26) (xy -10.16 177.8)
+			(xy 63.5 177.8) (xy 63.5 180.34)
 		)
 		(stroke
@@
 	(wire
 		(pts
-			(xy -10.16 160.02) (xy -10.16 165.1)
+			(xy 63.5 162.56) (xy 63.5 167.64)
 		)
 		(stroke
@@
 	(wire
 		(pts
-			(xy -10.16 170.18) (xy -10.16 175.26)
+			(xy 63.5 172.72) (xy 63.5 177.8)
 		)
 		(stroke
@@
 	(symbol
 		(lib_id "Mechanical:MountingHole_Pad")
-		(at -15.24 175.26 90)
+		(at 58.42 177.8 90)
 		(unit 1)
 		(body_style 1)
@@
 		(dnp no)
 		(property "Reference" "H4"
-			(at -20.32 175.26 90)
+			(at 53.34 177.8 90)
 			(show_name no)
 			(do_not_autoplace no)
@@
 		)
 		(property "Value" "MountingHole_Pad"
-			(at -16.51 171.45 90)
+			(at 57.15 173.99 90)
 			(hide yes)
 			(show_name no)
@@
 		)
 		(property "Footprint" "MountingHole:MountingHole_3.2mm_M3_DIN965_Pad_TopBottom"
-			(at -15.24 175.26 0)
+			(at 58.42 177.8 0)
 			(hide yes)
 			(show_name no)
@@
 		)
 		(property "Datasheet" ""
-			(at -15.24 175.26 0)
+			(at 58.42 177.8 0)
 			(hide yes)
 			(show_name no)
@@
 		)
 		(property "Description" "Mounting Hole with connection"
-			(at -15.24 175.26 0)
+			(at 58.42 177.8 0)
 			(hide yes)
 			(show_name no)
@@
 	(symbol
 		(lib_id "Mechanical:MountingHole_Pad")
-		(at -15.24 165.1 90)
+		(at 58.42 167.64 90)
 		(unit 1)
 		(body_style 1)
@@
 		(dnp no)
 		(property "Reference" "H2"
-			(at -20.32 165.1 90)
+			(at 53.34 167.64 90)
 			(show_name no)
 			(do_not_autoplace no)
@@
 		)
 		(property "Value" "MountingHole_Pad"
-			(at -16.51 161.29 90)
+			(at 57.15 163.83 90)
 			(hide yes)
 			(show_name no)
@@
 		)
 		(property "Footprint" "MountingHole:MountingHole_3.2mm_M3_DIN965_Pad_TopBottom"
-			(at -15.24 165.1 0)
+			(at 58.42 167.64 0)
 			(hide yes)
 			(show_name no)
@@
 		)
 		(property "Datasheet" ""
-			(at -15.24 165.1 0)
+			(at 58.42 167.64 0)
 			(hide yes)
 			(show_name no)
@@
 		)
 		(property "Description" "Mounting Hole with connection"
-			(at -15.24 165.1 0)
+			(at 58.42 167.64 0)
 			(hide yes)
 			(show_name no)
@@
 	(symbol
 		(lib_id "Mechanical:MountingHole_Pad")
-		(at -15.24 160.02 90)
+		(at 58.42 162.56 90)
 		(unit 1)
 		(body_style 1)
@@
 		(dnp no)
 		(property "Reference" "H1"
-			(at -20.32 160.02 90)
+			(at 53.34 162.56 90)
 			(show_name no)
 			(do_not_autoplace no)
@@
 		)
 		(property "Value" "MountingHole_Pad"
-			(at -16.51 156.21 90)
+			(at 57.15 158.75 90)
 			(hide yes)
 			(show_name no)
@@
 		)
 		(property "Footprint" "MountingHole:MountingHole_3.2mm_M3_DIN965_Pad_TopBottom"
-			(at -15.24 160.02 0)
+			(at 58.42 162.56 0)
 			(hide yes)
 			(show_name no)
@@
 		)
 		(property "Datasheet" ""
-			(at -15.24 160.02 0)
+			(at 58.42 162.56 0)
 			(hide yes)
 			(show_name no)
@@
 		)
 		(property "Description" "Mounting Hole with connection"
-			(at -15.24 160.02 0)
+			(at 58.42 162.56 0)
 			(hide yes)
 			(show_name no)
@@
 	(symbol
 		(lib_id "power:GND")
-		(at -10.16 177.8 0)
+		(at 63.5 180.34 0)
 		(unit 1)
 		(body_style 1)
@@
 		(fields_autoplaced yes)
 		(property "Reference" "#PWR0164"
-			(at -10.16 184.15 0)
+			(at 63.5 186.69 0)
 			(hide yes)
 			(show_name no)
@@
 		)
 		(property "Value" "GND"
-			(at -10.16 182.245 0)
+			(at 63.5 184.785 0)
 			(hide yes)
 			(show_name no)
@@
 		)
 		(property "Footprint" ""
-			(at -10.16 177.8 0)
+			(at 63.5 180.34 0)
 			(hide yes)
 			(show_name no)
@@
 		)
 		(property "Datasheet" ""
-			(at -10.16 177.8 0)
+			(at 63.5 180.34 0)
 			(hide yes)
 			(show_name no)
@@
 		)
 		(property "Description" "Power symbol creates a global label with name \"GND\" , ground"
-			(at -10.16 177.8 0)
+			(at 63.5 180.34 0)
 			(hide yes)
 			(show_name no)
@@
 	(symbol
 		(lib_id "Mechanical:MountingHole_Pad")
-		(at -15.24 170.18 90)
+		(at 58.42 172.72 90)
 		(unit 1)
 		(body_style 1)
@@
 		(dnp no)
 		(property "Reference" "H3"
-			(at -20.32 170.18 90)
+			(at 53.34 172.72 90)
 			(show_name no)
 			(do_not_autoplace no)
@@
 		)
 		(property "Value" "MountingHole_Pad"
-			(at -16.51 166.37 90)
+			(at 57.15 168.91 90)
 			(hide yes)
 			(show_name no)
@@
 		)
 		(property "Footprint" "MountingHole:MountingHole_3.2mm_M3_DIN965_Pad_TopBottom"
-			(at -15.24 170.18 0)
+			(at 58.42 172.72 0)
 			(hide yes)
 			(show_name no)
@@
 		)
 		(property "Datasheet" ""
-			(at -15.24 170.18 0)
+			(at 58.42 172.72 0)
 			(hide yes)
 			(show_name no)
@@
 		)
 		(property "Description" "Mounting Hole with connection"
-			(at -15.24 170.18 0)
+			(at 58.42 172.72 0)
 			(hide yes)
 			(show_name no)
@@
 			)
 		)
-		(pin "+5VSB" input
+		(pin "+5VSB" output
 			(at 64.77 21.59 0)
 			(effects
@@
 			)
 		)
+		(pin "12V_SENSE" output
+			(at 64.77 50.8 0)
+			(effects
+				(font
+					(size 1.27 1.27)
+				)
+				(justify right)
+			)
+		)
 		(instances
 			(project "Ziess-Microsope-Controller_Main_board"
@@
 			)
 		)
-		(pin "Y_ENC_DO" input
+		(pin "Y_ENC_DO" output
 			(at 64.77 92.71 0)
 			(effects
@@
 			)
 		)
-		(pin "Y_ENC_INDEX" input
+		(pin "Y_ENC_INDEX" output
 			(at 64.77 87.63 0)
 			(effects
@@
 			)
 		)
-		(pin "12V_PRES" output
+		(pin "5V_PG" output
 			(at 111.76 35.56 0)
 			(effects

Commit message: m
Other:
- sheet ACC2 ports: added ACC2_DIR, ACC2_IMON, ACC2_PG, ACC2_PRESENT, ACC2_PWR_EN, ACC2_PWR_FLG, ACC2_RX, ACC2_TX; removed ACC1_DIR, ACC1_IMON, ACC1_PG, ACC1_PRESENT, ACC1_PWR_EN, ACC1_PWR_FLG, ACC1_RX, ACC1_TX
- sheet ACC3 ports: added ACC3_DIR, ACC3_IMON, ACC3_PG, ACC3_PRESENT, ACC3_PWR_EN, ACC3_PWR_FLG, ACC3_RX, ACC3_TX; removed ACC1_DIR, ACC1_IMON, ACC1_PG, ACC1_PRESENT, ACC1_PWR_EN, ACC1_PWR_FLG, ACC1_RX, ACC1_TX
- sheet MCU ports: added none; removed 12V_EN, 12V_PRES, ACC1_GPIO1, ACC1_GPIO2, ACC1_RX, ACC1_TX, ACC2_GPIO1, ACC2_GPIO2, ACC2_RX, ACC2_TX, F_EN, F_FAULT, F_LIM_1, F_LIM_2, F_NSLEEP, F_PH, F_SENSE, INPUT_IMON, J_EN, J_ENC_OUT, J_ENC_SCL, J_ENC_SDA, J_FAULT, J_LIM, J_NSLEEP, J_PH, J_SENSE, REMOTE_GPIO1, REMOTE_GPIO2, REMOTE_GPIO3, REMOTE_GPIO4, REMOTE_GPIO5, REMOTE_RX, REMOTE_TX, SYNC_OUT, USB_DN, USB_DP, USB_VBUS, XY_ENC_CLK, XY_UART_RX, XY_UART_TX, X_DIAG, X_DIR, X_EN, X_ENC_CS, X_ENC_DO, X_ENC_INDEX, X_LIM_1, X_LIM_2, X_STDBY, X_STEP, Y_DIAG, Y_DIR, Y_EN, Y_ENC_CS, Y_ENC_DO, Y_ENC_INDEX, Y_LIM_1, Y_LIM_2, Y_STDBY, Y_STEP, Z_EN, Z_ENC_A, Z_ENC_B, Z_FAULT, Z_LIM_1, Z_LIM_2, Z_NSLEEP, Z_PH, Z_SENSE
- sheet POWER_INPUT ports: added none; removed +12V, +5VSB
- sheet PWR_REG ports: added none; removed +12V, +5VSB
