File: hardware/Ziess-Microsope-Controller_Main_board/IO.kicad_sch (KiCad schematic)
At the start: 41 parts, among them J16 Conn_01x34, U15 USBLC6-2SC6, U16 74LVC1G17

Commit message: m
Connections:
- net at J16.17 (Pin_17), R106.1: now also D10.1 (A1); no longer D16.1 (A1)
- net at J16.24 (Pin_24), R111.1: now also D15.1 (A1); no longer D11.1 (A1)
- net at J16.22 (Pin_22), R110.1: now also D14.1 (A1); no longer D12.1 (A1)
- net at J16.28 (Pin_28), R114.1: now also D18.1 (A1); no longer D8.1 (A1)
- net at J16.19 (Pin_19), R108.1: now also D12.1 (A1); no longer D14.1 (A1)
- net at J16.27 (Pin_27), R113.1: now also D17.1 (A1); no longer D9.1 (A1)
- net at J16.16 (Pin_16), R105.1: now also D9.1 (A1); no longer D17.1 (A1)
- net at J16.30 (Pin_30), R115.1: now also D19.1 (A1); no longer D7.1 (A1)
- net at J16.31 (Pin_31), R116.1: now also D20.1 (A1); no longer D6.1 (A1)
- net at J16.15 (Pin_15), R104.1: now also D8.1 (A1); no longer D18.1 (A1)
- net at J16.13 (Pin_13), R103.1: now also D7.1 (A1); no longer D19.1 (A1)
- net at J16.12 (Pin_12), R102.1: now also D6.1 (A1); no longer D20.1 (A1)
- net at J16.18 (Pin_18), R107.1: now also D11.1 (A1); no longer D15.1 (A1)
- net at J16.25 (Pin_25), R112.1: now also D16.1 (A1); no longer D10.1 (A1)

Commit message: m
Parts:
- removed D10, D11, D12, D13, D14, D15, D16, D17, D18, D19, D20, D6, D7, D8, D9: CDSOD323-T03C, Diode_SMD:D_SOD-323, symbol Diode:ESD9B5.0ST5G
- removed J16: Conn_01x34, Library:F52Q1A7H111034, symbol Connector_Generic:Conn_01x34
- removed R102, R103, R104, R106, R107, R108, R109, R110, R111, R112, R113, R114, R115, R116: 1k, Resistor_SMD:R_0805_2012Metric, symbol Device:R_Small
- added C122: 4.7nF, Capacitor_SMD:C_0805_2012Metric, symbol Device:C_Small
- added J19: 5787834-1, Library:5787834-1, symbol Connector:USB_B
- added J20: 031532951RFX, Library:031532951RFX, symbol Library:Conn_Coaxial
- added J22, J23: LD09S24A4GV00LF, Library:LD09S24A4GV00LF, symbol Connector:DE9_Pins_MountingHoles
- R105: value 1k -> 0; now not fitted; now left out of the parts list
Connections:
- net GND: now also R105.1, C122.1, J19.4 (GND), J20.2 (Ext), J20.3 (Ext), J20.4 (Ext), J20.5 (Ext)
- net USB_DN: now also R100.1; no longer R100.2
- net USB_DP: now also R99.1; no longer R99.2
- net USB_VBUS: now also J19.1 (VBUS)
- net at U15.4 (I/O2): now also J19.2 (D-); no longer R100.1
- net at R101.2: now also J20.1 (In)
- net at R98.2, U15.1 (I/O1): now also R99.2
- net at U15.3 (I/O2): now also R100.2
- net at U15.6 (I/O1): now also J19.3 (D+); no longer R99.1
- net REMOTE_GPIO2 renamed USB_SH
- net USB_SH: now also C122.2, J19.5 (Shield), J19.6 (Shield)
- new net: J22.MH1 (PAD), J22.MH2 (PAD)
- new net: J23.MH1 (PAD), J23.MH2 (PAD)
Other:
- moved on the sheet: C99, R101, R98, U16

Commit message: m
Parts:
- removed J22, J23: LD09S24A4GV00LF, Library:LD09S24A4GV00LF, symbol Connector:DE9_Pins_MountingHoles
- added C123, C124, C126: 100nF, Capacitor_SMD:C_0603_1608Metric, symbol Device:C_Small
- added C125: 4.7uF, Capacitor_SMD:C_0603_1608Metric, symbol Device:C_Small
- added D6: BZT52C5V6, Diode_SMD:D_SOD-123F, symbol Diode:BZT52Bxx
- added J16, J21: Conn_01x10, symbol Connector_Generic:Conn_01x10
- added L3, L4: 10uH, Library:8200, symbol Device:L_Small
- added PS1: NXJ1S1205MC-R13, Library:NXJ1S1205MCR13, symbol Library:NXJ1S1205MC-R13
- added R102, R103: 0, Resistor_SMD:R_0603_1608Metric, symbol Device:R_Small
- added U19: ISO1430DWR, Library:SOIC127P1030X265-16N, symbol Library:ISO1430DWR
Connections:
- net +3.3V: now also C123.2, U19.1 (VCC1)
- net GND: now also C123.1, C124.1, PS1.1 (-VIN), U19.2 (GND1_1), U19.8 (GND1_2)
- new net: C125.2, C126.1, D6.1 (K), L4.2, U19.16 (VCC2)
- new net: R103.2, U19.12 (A)
- new net: L4.1, PS1.14 (NC), PS1.8 (+VOUT)
- new net: R102.2, U19.13 (B)
- new net: U19.4 (~{RE}), U19.5 (DE)
- new net: C124.2, L3.1
- new net: L3.2, PS1.3 (+VIN)
- new net GND_ISO1: C125.1, C126.2, D6.2 (A), PS1.7 (-VOUT), U19.15 (GND2_2), U19.9 (GND2_1)
- no-connect marks 0 -> 4
Other:
- moved on the sheet: C99, J20, R101, U16

Commit message: m
Parts:
- added C127: 100nF, Capacitor_SMD:C_0402_1005Metric, symbol Device:C_Small
- added C128: 100nF, Capacitor_SMD:C_1206_3216Metric, symbol Device:C_Small
- added C129: 10uF, Capacitor_SMD:C_1206_3216Metric, symbol Device:C_Small
- added C130: C_Polarized_Small, Capacitor_SMD:CP_Elec_4x3, symbol Device:C_Polarized_Small
- added C131: 100nF, Capacitor_SMD:C_0603_1608Metric, symbol Device:C_Small
- added C132: 1uF, Capacitor_SMD:C_0603_1608Metric, symbol Device:C_Small
- added D7: RED, LED_SMD:LED_0603_1608Metric, symbol Device:LED
- added D9: SMAJ12A, Diode_SMD:D_SMC, symbol Diode:SMAJ12A
- added Q3: 2N7002, Package_TO_SOT_SMD:SOT-23, symbol Transistor_FET:2N7002
- added R104, R108, R109, R113, R114, R115: 10k, Resistor_SMD:R_0603_1608Metric, symbol Device:R_Small
- added R106, R107: 33, Resistor_SMD:R_0603_1608Metric, symbol Device:R_Small
- added R110: 100, Resistor_SMD:R_0603_1608Metric, symbol Device:R_Small
- added R111, R112: 390k, Resistor_SMD:R_0603_1608Metric, symbol Device:R_Small
- added R116: 1.5k, Resistor_SMD:R_0603_1608Metric, symbol Device:R_Small
- added U20: TPS259472LRPWR, Library:TPS259472LRPWR, symbol Library:TPS259472LRPWR
- C124: footprint Capacitor_SMD:C_0603_1608Metric -> Capacitor_SMD:C_1206_3216Metric
- C125: footprint Capacitor_SMD:C_0603_1608Metric -> Capacitor_SMD:C_0805_2012Metric
- J21: footprint (none) -> Library:BM10BGHSTBT
- R102, R103: value 0 -> 33
Connections:
- net +3.3V: now also R115.2, R116.2
- net GND: now also J21.10 (Pin_10), J21.3 (Pin_3), J21.4 (Pin_4), J21.7 (Pin_7), C127.1, C128.1, C129.1, C130.2, C131.1, C132.1, D9.2 (A2), Q3.2 (S), R104.1, R109.1, R111.1, R112.1, R114.1, U20.8 (GND)
- net at R103.1: now also J21.6 (Pin_6)
- net at J21.1 (Pin_1): now also J21.2 (Pin_2), C129.2, C130.1, D9.1 (A1), R113.1, U20.6 (OUT)
- net at J21.5 (Pin_5): now also R102.1
- net at U19.3 (R): now also R106.1
- net at U19.4 (~{RE}), U19.5 (DE): now also R104.2
- net at U19.6 (D): now also R107.1
- new net: C131.2, C132.2, R108.2, U20.5 (IN)
- new net: Q3.1 (G), R115.1, U20.3 (PG/_AUXOFF)
- new net: D7.1 (K), Q3.3 (D)
- new net: D7.2 (A), R116.1
- new net: R108.1, R109.2, R110.1, U20.1 (EN/UVLO_1), U20.11 (EN/UVLO_2)
- new net: C128.2, U20.10 (ITIMER_1), U20.14 (ITIMER_2)
- new net: R113.2, R114.2, U20.12 (PGTH/_~{FLT_2}), U20.4 (PGTH/_~{FLT_1})
- new net: C127.2, U20.13 (DVDT_2), U20.7 (DVDT_1)
- new net: R111.2, U20.2 (OVLO/_OVCSEL)
- new net: R112.2, U20.9 (ILM)
- new net RS_PWR_EN: R110.2
Other:
- moved on the sheet: C123, C124, C125, C126, D6, J21, L3, L4, PS1, R102, R103, U19
