File: hardware/Ziess-Microsope-Controller_Main_board/IO.kicad_sch (KiCad schematic)
At the start: 49 parts, among them J16 Conn_01x10, J19 5787834-1, J20 031532951RFX, J21 Conn_01x10, Q3 2N7002, U15 USBLC6-2SC6, U16 74LVC1G17, U19 ISO1430DWR, U20 TPS259472LRPWR

Commit message: m
Parts:
- removed C122: 4.7nF, Capacitor_SMD:C_0805_2012Metric, symbol Device:C_Small
- removed C123, C126, C98: 100nF, Capacitor_SMD:C_0603_1608Metric, symbol Device:C_Small
- removed C124: 100nF, Capacitor_SMD:C_1206_3216Metric, symbol Device:C_Small
- removed C125: 4.7uF, Capacitor_SMD:C_0805_2012Metric, symbol Device:C_Small
- removed D6: BZT52C5V6, Diode_SMD:D_SOD-123F, symbol Diode:BZT52Bxx
- removed J19: 5787834-1, Library:5787834-1, symbol Connector:USB_B
- removed L3, L4: 10uH, Library:8200, symbol Device:L_Small
- removed PS1: NXJ1S1205MC-R13, Library:NXJ1S1205MCR13, symbol Library:NXJ1S1205MC-R13
- removed R105: 0, Resistor_SMD:R_0805_2012Metric, symbol Device:R_Small
- removed R107: 33, Resistor_SMD:R_0603_1608Metric, symbol Device:R_Small
- removed U19: ISO1430DWR, Library:SOIC127P1030X265-16N, symbol Library:ISO1430DWR
- added C133: 1uF, Capacitor_SMD:C_0603_1608Metric, symbol Device:C_Small
- added C134: 100nF, Capacitor_SMD:C_0603_1608Metric, symbol Device:C_Small
- added C135: 100nF, Capacitor_SMD:C_1206_3216Metric, symbol Device:C_Small
- added C136: 100nF, Capacitor_SMD:C_0402_1005Metric, symbol Device:C_Small
- added C137: 10uF, Capacitor_SMD:C_1206_3216Metric, symbol Device:C_Small
- added C138: C_Polarized_Small, Capacitor_SMD:CP_Elec_4x3, symbol Device:C_Polarized_Small
- added D10: SMAJ12A, Diode_SMD:D_SMC, symbol Diode:SMAJ12A
- added D8: RED, LED_SMD:LED_0603_1608Metric, symbol Device:LED
- added IC1: TRS3122ERGER, QFN50P400X400X100-25N-D, symbol Library:TRS3122ERGER
- added J18: B4B-XH-AM, Library:BM04BGHSTBTLFSN, symbol Connector_Generic:Conn_01x04
- added J22: Conn_01x10, Library:BM10BGHSTBT, symbol Connector_Generic:Conn_01x10
- added Q4: 2N7002, Package_TO_SOT_SMD:SOT-23, symbol Transistor_FET:2N7002
- added R136: 100, Resistor_SMD:R_0603_1608Metric, symbol Device:R_Small
- added R138, R139, R142, R143, R144: 10k, Resistor_SMD:R_0603_1608Metric, symbol Device:R_Small
- added R140, R141: 390k, Resistor_SMD:R_0603_1608Metric, symbol Device:R_Small
- added R145: 1.5k, Resistor_SMD:R_0603_1608Metric, symbol Device:R_Small
- added U21: TPS259472LRPWR, Library:TPS259472LRPWR, symbol Library:TPS259472LRPWR
- J20: footprint Library:031532951RFX -> Library:U.FL-R-SMT-1_10_
- R102, R103, R106: value 33 -> 0
- R104: value 10k -> 0
- R98: now left out of the parts list
Connections:
- net +3.3V: now also R144.2, R145.2
- net GND: now also J20.1 (Ext), C133.1, C134.1, C135.1, C136.1, C137.1, C138.2, D10.2 (A2), J18.1 (Pin_1), J22.3 (Pin_3), J22.4 (Pin_4), Q4.2 (S), R138.1, R140.1, R141.1, R143.1, U21.8 (GND); no longer J20.3 (Ext), J20.4 (Ext), J20.5 (Ext), J21.10 (Pin_10), J21.7 (Pin_7), R104.1
- net RS_PWR_EN: now also R136.2
- net USB_DN: now also R100.2; no longer R100.1
- net USB_DP: now also R98.2, R99.2; no longer R99.1
- net USB_VBUS: now also J18.4 (Pin_4)
- net at U15.3 (I/O2): now also J18.2 (Pin_2); no longer R100.2
- net at U15.4 (I/O2): now also R100.1
- net at U15.6 (I/O1): now also R99.1
- net at R103.1: no longer J21.6 (Pin_6)
- net at R103.2: now also J21.6 (Pin_6)
- net at R101.2: now also J20.3 (In); no longer J20.1 (In)
- net at R102.1: no longer J21.5 (Pin_5)
- net at R102.2: now also J21.5 (Pin_5)
- net at R104.2: now also J22.5 (Pin_5)
- net at R106.2: now also J22.6 (Pin_6)
- new net: C133.2, C134.2, R139.2, U21.5 (IN)
- new net: C136.2, U21.13 (DVDT_2), U21.7 (DVDT_1)
- new net: C137.2, C138.1, D10.1 (A1), J22.1 (Pin_1), J22.2 (Pin_2), R142.1, U21.6 (OUT)
- new net: Q4.1 (G), R144.1, U21.3 (PG/_AUXOFF)
- new net: J18.3 (Pin_3), U15.1 (I/O1)
- new net: R136.1, R138.2, R139.1, U21.1 (EN/UVLO_1), U21.11 (EN/UVLO_2)
- new net: D8.1 (K), Q4.3 (D)
- new net: C135.2, U21.10 (ITIMER_1), U21.14 (ITIMER_2)
- new net: R142.2, R143.2, U21.12 (PGTH/_~{FLT_2}), U21.4 (PGTH/_~{FLT_1})
- new net: R140.2, U21.2 (OVLO/_OVCSEL)
- new net: R141.2, U21.9 (ILM)
- new net: D8.2 (A), R145.1
- no-connect marks 4 -> 0
Other:
- moved on the sheet: J21

Commit message: m
Parts:
- removed J16: Conn_01x10, symbol Connector_Generic:Conn_01x10
Connections:
- net at R106.1: now also IC1.9 (DIN2)
- net at R102.1: now also IC1.12 (ROUT1)
- net at R103.1: now also IC1.10 (DIN1)
- net at R104.1: now also IC1.11 (ROUT2)
Other:
- moved on the sheet: C127, C128, C129, C130, C131, C132, C133, C134, C135, C136, C137, C138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
