File: hardware/Ziess-Microsope-Controller_Main_board/Ziess-Microsope-Controller_Main_board.kicad_pcb (KiCad board)
At the start: 2 copper layers, 6 parts, among them J1 670689000, J2 23117633, J3 57478404, J4 57478404, J5 0039301040, J6 0731000105

Commit message: m
Parts:
- added C1: 100nF, Capacitor_SMD:C_0603_1608Metric, F.Cu at (147.3, 629.4)
- added C10: 10uF, Capacitor_SMD:C_1210_3225Metric, F.Cu at (107.9, -45.8)
- added C100: 4.7nF, Capacitor_SMD:C_0805_2012Metric, B.Cu at (79.2, 638.8)
- added C101: 4.7nF, Capacitor_SMD:C_0805_2012Metric, B.Cu at (118.0, 638.7)
- added C102: 4.7nF, Capacitor_SMD:C_0805_2012Metric, B.Cu at (118.0, 618.8)
- added C103: 4.7uF, Capacitor_SMD:C_0805_2012Metric, F.Cu at (142.6, 93.0)
- added C104: 100nF, Capacitor_SMD:C_0603_1608Metric, F.Cu at (157.2, 56.9)
- added C105: 100nF, Capacitor_SMD:C_0603_1608Metric, F.Cu at (157.2, 59.4)
- added C106: 100nF, Capacitor_SMD:C_0603_1608Metric, F.Cu at (157.2, 62.0)
- added C107: 100nF, Capacitor_SMD:C_0603_1608Metric, F.Cu at (157.2, 64.5)
- added C108: 100nF, Capacitor_SMD:C_0603_1608Metric, F.Cu at (157.2, 67.0)
- added C109: 100nF, Capacitor_SMD:C_0603_1608Metric, F.Cu at (157.2, 69.5)
- added C11: 10uF, Capacitor_SMD:C_1210_3225Metric, F.Cu at (107.9, -41.5)
- added C110: 100nF, Capacitor_SMD:C_0603_1608Metric, F.Cu at (157.2, 72.0)
- added C111: 1uF, Capacitor_SMD:C_0603_1608Metric, F.Cu at (157.2, 74.5)
- added C112: 100nF, Capacitor_SMD:C_0603_1608Metric, F.Cu at (157.2, 77.0)
- added C113: 100nF, Capacitor_SMD:C_0603_1608Metric, F.Cu at (157.2, 79.5)
- added C114: 10pf, Capacitor_SMD:C_0603_1608Metric, F.Cu at (157.2, 82.0)
- added C115: 10pf, Capacitor_SMD:C_0603_1608Metric, F.Cu at (143.2, 54.0)
- added C116: 2.2uF, Capacitor_SMD:C_1206_3216Metric, F.Cu at (117.5, 90.0)
- added C117: 2.2uF, Capacitor_SMD:C_1206_3216Metric, F.Cu at (117.5, 93.3)
- added C12: 100nF, Capacitor_SMD:C_0603_1608Metric, F.Cu at (19.5, -108.7)
- added C13: 10nF, Capacitor_SMD:C_0603_1608Metric, F.Cu at (19.5, -106.2)
- added C14: 120pF, Capacitor_SMD:C_0603_1608Metric, F.Cu at (19.5, -103.7)
- added C15: 12nF, Capacitor_SMD:C_0603_1608Metric, F.Cu at (19.5, -101.2)
- added C16: 10uF, Capacitor_SMD:C_1210_3225Metric, F.Cu at (107.9, -37.3)
- added C17: 100nF, Capacitor_SMD:C_0603_1608Metric, F.Cu at (19.5, -98.7)
- added C18: 100nF, Capacitor_SMD:C_0603_1608Metric, F.Cu at (19.5, -96.2)
- added C19: 22uF, Capacitor_SMD:C_1210_3225Metric, F.Cu at (107.9, -33.0)
- added C2: 22uF, Capacitor_SMD:C_1210_3225Metric, B.Cu at (139.2, 633.1)
- added C20: 1uF, Capacitor_SMD:C_1210_3225Metric, F.Cu at (-99.0, -46.2)
- added C21: 100nF, Capacitor_SMD:C_0603_1608Metric, F.Cu at (-187.4, -111.0)
- added C22: 100nF, Capacitor_SMD:C_0603_1608Metric, F.Cu at (-187.4, -108.5)
- added C23: 10uF, Capacitor_SMD:C_2220_5750Metric, F.Cu at (-106.1, -66.1)
- added C24: 10uF, Capacitor_SMD:C_2220_5750Metric, F.Cu at (-106.1, -59.1)
- added C25: 100uF, Capacitor_SMD:CP_Elec_8x10, F.Cu at (-143.2, -112.8)
- added C26: 100uF, Capacitor_SMD:CP_Elec_8x10, F.Cu at (-143.2, -102.9)
- added C27: 100nF, Capacitor_SMD:C_0603_1608Metric, F.Cu at (-187.4, -106.0)
- added C28: 100nF, Capacitor_SMD:C_0603_1608Metric, F.Cu at (-187.4, -103.5)
- added C29: 100nF, Capacitor_SMD:C_0603_1608Metric, F.Cu at (-187.4, -101.0)
- added C3: 100nF, Capacitor_SMD:C_0603_1608Metric, B.Cu at (145.2, 622.5)
- added C30: 4.7uF, Capacitor_SMD:C_0805_2012Metric, F.Cu at (-88.8, -68.0)
- added C31: 22nF, Capacitor_SMD:C_0805_2012Metric, F.Cu at (-88.8, -65.0)
- added C32: 470pF, Capacitor_SMD:C_0402_1005Metric, F.Cu at (-123.4, -51.8)
- added C33: 470pF, Capacitor_SMD:C_0402_1005Metric, F.Cu at (-123.4, -49.8)
- added C34: 470pF, Capacitor_SMD:C_0402_1005Metric, F.Cu at (-123.4, -47.8)
- added C35: 470pF, Capacitor_SMD:C_0402_1005Metric, F.Cu at (-123.4, -45.8)
- added C36: 100nF, Capacitor_SMD:C_0603_1608Metric, F.Cu at (-187.4, -98.5)
- added C37: 100nF, Capacitor_SMD:C_0603_1608Metric, F.Cu at (-187.4, -96.0)
- added C38: 100nF, Capacitor_SMD:C_0603_1608Metric, F.Cu at (-187.4, -93.5)
- added C39: 100nF, Capacitor_SMD:C_0603_1608Metric, F.Cu at (-187.4, -91.0)
- added C4: 220uF, Capacitor_SMD:CP_Elec_8x10, F.Cu at (151.2, 615.0)
- added C40: 100nF, Capacitor_SMD:C_0603_1608Metric, F.Cu at (-167.5, -317.7)
- added C41: 1uF, Capacitor_SMD:C_1210_3225Metric, F.Cu at (-83.2, -223.4)
- added C42: 100nF, Capacitor_SMD:C_0603_1608Metric, F.Cu at (-167.5, -315.1)
- added C43: 10uF, Capacitor_SMD:C_2220_5750Metric, F.Cu at (-90.2, -233.7)
- added C44: 10uF, Capacitor_SMD:C_2220_5750Metric, F.Cu at (-90.2, -226.8)
- added C45: 100uF, Capacitor_SMD:CP_Elec_8x10, F.Cu at (-127.4, -274.6)
- added C46: 100uF, Capacitor_SMD:CP_Elec_8x10, F.Cu at (-115.6, -314.0)
- added C47: 100nF, Capacitor_SMD:C_0603_1608Metric, F.Cu at (-167.5, -312.6)
- added C48: 100nF, Capacitor_SMD:C_0603_1608Metric, F.Cu at (-167.5, -310.1)
- added C49: 100nF, Capacitor_SMD:C_0603_1608Metric, F.Cu at (-167.5, -307.6)
- added C5: 220uF, Capacitor_SMD:CP_Elec_8x10, F.Cu at (151.2, 605.4)
- added C50: 4.7uF, Capacitor_SMD:C_0805_2012Metric, F.Cu at (-73.0, -243.6)
- added C51: 22nF, Capacitor_SMD:C_0805_2012Metric, F.Cu at (-73.0, -240.5)
- added C52: 470pF, Capacitor_SMD:C_0402_1005Metric, F.Cu at (-107.6, -225.4)
- added C53: 470pF, Capacitor_SMD:C_0402_1005Metric, F.Cu at (-107.6, -223.4)
- added C54: 470pF, Capacitor_SMD:C_0402_1005Metric, F.Cu at (-107.6, -221.5)
- added C55: 470pF, Capacitor_SMD:C_0402_1005Metric, F.Cu at (-107.6, -219.5)
- added C56: 100nF, Capacitor_SMD:C_0603_1608Metric, F.Cu at (-167.5, -305.1)
- added C57: 100nF, Capacitor_SMD:C_0603_1608Metric, F.Cu at (-167.5, -302.6)
- added C58: 100nF, Capacitor_SMD:C_0603_1608Metric, F.Cu at (-167.5, -300.1)
- added C59: 100nF, Capacitor_SMD:C_0603_1608Metric, F.Cu at (-167.5, -297.6)
- added C6: 33nF, Capacitor_SMD:C_0603_1608Metric, F.Cu at (150.8, 624.5)
- added C60: 100nF, Capacitor_SMD:C_0603_1608Metric, F.Cu at (-322.9, -244.1)
- added C61: 1uF, Capacitor_SMD:C_0603_1608Metric, F.Cu at (-322.9, -241.6)
- added C62: 100nF, Capacitor_SMD:C_0201_0603Metric, F.Cu at (-292.3, -161.0)
- added C63: 100nF, Capacitor_SMD:C_0603_1608Metric, F.Cu at (-322.9, -239.1)
- added C64: 1uF, Capacitor_SMD:C_0603_1608Metric, F.Cu at (-322.9, -236.5)
- added C65: 100nF, Capacitor_SMD:C_0603_1608Metric, F.Cu at (-322.9, -234.0)
- added C66: 100nF, Capacitor_SMD:C_0603_1608Metric, F.Cu at (-322.9, -231.5)
- added C67: 100nF, Capacitor_SMD:C_0603_1608Metric, F.Cu at (-322.9, -229.0)
- added C68: 220uF, Capacitor_SMD:CP_Elec_8x10, F.Cu at (-407.4, 247.9)
- added C69: 220uF, Capacitor_SMD:CP_Elec_8x10, F.Cu at (-422.8, 247.8)
- added C7: 100nF, Capacitor_SMD:C_0603_1608Metric, F.Cu at (19.5, -111.2)
- added C70: 10uF, Capacitor_SMD:C_2220_5750Metric, F.Cu at (-415.1, 248.2)
- added C71: 100nF, Capacitor_SMD:C_0603_1608Metric, F.Cu at (-416.1, 240.8)
- added C72: 100nF, Capacitor_SMD:C_0603_1608Metric, F.Cu at (-416.1, 242.8)
- added C73: 22nF, Capacitor_SMD:C_0603_1608Metric, F.Cu at (-426.3, 241.2)
- added C74: 100nF, Capacitor_SMD:C_0603_1608Metric, F.Cu at (135.5, -273.2)
- added C75: 100nF, Capacitor_SMD:C_0603_1608Metric, F.Cu at (135.5, -270.6)
- added C76: 100nF, Capacitor_SMD:C_0603_1608Metric, F.Cu at (135.5, -268.1)
- added C77: 100nF, Capacitor_SMD:C_0603_1608Metric, F.Cu at (135.5, -265.6)
- added C78: 220uF, Capacitor_SMD:CP_Elec_8x10, F.Cu at (-240.5, 204.3)
- added C79: 100nF, Capacitor_SMD:C_0603_1608Metric, F.Cu at (-288.5, 181.1)
- added C8: 47uF, Capacitor_SMD:C_1206_3216Metric, F.Cu at (30.7, -23.7)
- added C80: 100nF, Capacitor_SMD:C_0603_1608Metric, F.Cu at (-288.5, 183.7)
- added C81: 22nF, Capacitor_SMD:C_0603_1608Metric, F.Cu at (-288.5, 186.2)
- added C82: 100nF, Capacitor_SMD:C_0603_1608Metric, F.Cu at (-288.5, 188.7)
- added C83: 100nF, Capacitor_SMD:C_0603_1608Metric, F.Cu at (-288.5, 191.2)
- added C84: 100nF, Capacitor_SMD:C_0603_1608Metric, F.Cu at (-288.5, 193.7)
- added C85: 220uF, Capacitor_SMD:CP_Elec_8x10, F.Cu at (-590.5, 204.2)
- added C86: 100nF, Capacitor_SMD:C_0603_1608Metric, F.Cu at (-638.4, 186.2)
- added C87: 100nF, Capacitor_SMD:C_0603_1608Metric, F.Cu at (-638.4, 188.7)
- added C88: 22nF, Capacitor_SMD:C_0603_1608Metric, F.Cu at (-638.4, 191.2)
- added C89: 100nF, Capacitor_SMD:C_0603_1608Metric, F.Cu at (-439.1, -60.5)
- added C9: 47uF, Capacitor_SMD:C_1206_3216Metric, F.Cu at (30.7, -20.3)
- added C90: 100nF, Capacitor_SMD:C_0603_1608Metric, F.Cu at (-439.1, -58.0)
- added C91: 100nF, Capacitor_SMD:C_0603_1608Metric, F.Cu at (401.6, 31.0)
- added C92: 100nF, Capacitor_SMD:C_0603_1608Metric, F.Cu at (401.6, 33.5)
- added C93: 100nF, Capacitor_SMD:C_0603_1608Metric, F.Cu at (401.6, 36.0)
- added C94: 100nF, Capacitor_SMD:C_0603_1608Metric, F.Cu at (401.6, 38.5)
- added C95: 100nF, Capacitor_SMD:C_0603_1608Metric, F.Cu at (405.6, -6.68)
- added C96: 100nF, Capacitor_SMD:C_0603_1608Metric, F.Cu at (405.6, -4.17)
- added C97: 100nF, Capacitor_SMD:C_0603_1608Metric, F.Cu at (31.6, 627.1)
- added C98: 4.7nF, Capacitor_SMD:C_0805_2012Metric, F.Cu at (33.8, 646.8)
- added C99: 100nF, Capacitor_SMD:C_0603_1608Metric, F.Cu at (79.9, 619.3)
- added D1: RED, LED_SMD:LED_0603_1608Metric, F.Cu at (154.2, 626.4)
- added D10: CDSOD323-T03C, Diode_SMD:D_SOD-323, B.Cu at (109.5, 634.9)
- added D11: CDSOD323-T03C, Diode_SMD:D_SOD-323, B.Cu at (106.8, 634.9)
- added D12: CDSOD323-T03C, Diode_SMD:D_SOD-323, B.Cu at (104.0, 634.9)
- added D13: CDSOD323-T03C, Diode_SMD:D_SOD-323, B.Cu at (101.3, 634.9)
- added D14: CDSOD323-T03C, Diode_SMD:D_SOD-323, B.Cu at (58.8, 634.9)
- added D15: CDSOD323-T03C, Diode_SMD:D_SOD-323, B.Cu at (61.6, 634.9)
- added D16: CDSOD323-T03C, Diode_SMD:D_SOD-323, B.Cu at (64.4, 634.9)
- added D17: CDSOD323-T03C, Diode_SMD:D_SOD-323, B.Cu at (67.1, 634.9)
- added D18: CDSOD323-T03C, Diode_SMD:D_SOD-323, B.Cu at (69.9, 634.9)
- added D19: CDSOD323-T03C, Diode_SMD:D_SOD-323, B.Cu at (72.7, 634.9)
- added D2: GREEN, LED_SMD:LED_0603_1608Metric, F.Cu at (154.2, 624.6)
- added D20: CDSOD323-T03C, Diode_SMD:D_SOD-323, B.Cu at (75.4, 634.9)
- added D3: SMAJ15A, Diode_SMD:D_SMA, B.Cu at (140.4, 636.8)
- added D4: CDSOD323-T03C, Diode_SMD:D_SOD-323, B.Cu at (106.8, 614.9)
- added D5: RED, LED_SMD:LED_0603_1608Metric, F.Cu at (-87.4, -93.2)
- added D6: RED, LED_SMD:LED_0603_1608Metric, F.Cu at (-71.6, -272.1)
- added D7: CDSOD323-T03C, Diode_SMD:D_SOD-323, B.Cu at (104.0, 614.9)
- added D8: CDSOD323-T03C, Diode_SMD:D_SOD-323, B.Cu at (101.3, 614.9)
- added D9: CDSOD323-T03C, Diode_SMD:D_SOD-323, B.Cu at (109.5, 614.9)
- added J10: B3B-XH-AM, Library:B3BXHAMLFSN, F.Cu at (190.1, -202.5)
- added J11: B2B-XH-AM, Library:B2BXHAMLFSN, F.Cu at (83.8, 548.0)
- added J12: B4B-XH-AM, Library:B4BXHAM, F.Cu at (-254.4, 250.6)
- added J13: B2B-XH-AM, Library:B2BXHAMLFSN, F.Cu at (-223.4, 260.3)
- added J14: B2B-XH-AM, Library:B2BXHAMLFSN, F.Cu at (63.0, 548.9)
- added J15: B3B-XH-AM, Library:B3BXHAMLFSN, F.Cu at (-384.5, -13.7)
- added J16: B10B-XH-AM, Library:B10BXHAMLFSN, F.Cu at (459.4, -2.98)
- added J18: B4B-XH-AM, Library:B4BXHAM, F.Cu at (435.7, 90.5)
- added J19: 5787834-1, Library:5787834-1, F.Cu at (32.5, 631.6)
- added J20: 031532951RFX, Library:031532951RFX, F.Cu at (66.4, 621.9)
- added J21: 10090929S154VLF, Library:10090929S154VLF, F.Cu at (71.4, 643.8)
- added J22: LD09S24A4GV00LF, Library:LD09S24A4GV00LF, F.Cu at (112.2, 644.4)
- added J23: LD09S24A4GV00LF, Library:LD09S24A4GV00LF, F.Cu at (112.3, 624.4)
- added J7: B6B-XH-AM, Library:B6BXHAMLFSN, F.Cu at (-261.1, -245.3)
- added J8: B2B-XH-AM, Library:B2BXHAMLFSN, F.Cu at (109.0, 547.8)
- added J9: B4B-XH-AM, Library:B4BXHAM, F.Cu at (169.6, -202.5)
- added L1: 15uH, Library:XAL6060153MEC, F.Cu at (23.1, -20.5)
- added L2: FCM1608KF-601T05, Inductor_SMD:L_0603_1608Metric, F.Cu at (143.2, 56.5)
- added Q1: BSS84, Package_TO_SOT_SMD:SOT-23, F.Cu at (118.3, -34.9)
- added Q2: 2N7002, Package_TO_SOT_SMD:SOT-23, F.Cu at (118.3, -30.4)
- added R1: 0.002, Resistor_SMD:R_2512_6332Metric, F.Cu at (136.6, 630.9)
- added R10: 10k, Resistor_SMD:R_0603_1608Metric, F.Cu at (35.5, -93.6)
- added R100: 10k, Resistor_SMD:R_0603_1608Metric, F.Cu at (429.7, 3.36)
- added R102: 10k, Resistor_SMD:R_0603_1608Metric, F.Cu at (429.7, 8.38)
- added R103: 0, Resistor_SMD:R_0603_1608Metric, F.Cu at (31.4, 622.1)
- added R104: 0, Resistor_SMD:R_0603_1608Metric, F.Cu at (33.4, 622.1)
- added R105: 0, Resistor_SMD:R_0805_2012Metric, F.Cu at (31.2, 646.8)
- added R106: 47, Resistor_SMD:R_0603_1608Metric, F.Cu at (76.0, 622.0)
- added R107: 0, Resistor_SMD:R_0805_2012Metric, B.Cu at (81.7, 638.8)
- added R108: 0, Resistor_SMD:R_0805_2012Metric, B.Cu at (120.5, 638.7)
- added R109: 0, Resistor_SMD:R_0805_2012Metric, B.Cu at (120.5, 618.8)
- added R11: 10k, Resistor_SMD:R_0603_1608Metric, F.Cu at (35.5, -91.1)
- added R110: 10k, Resistor_SMD:R_0603_1608Metric, F.Cu at (115.7, 68.5)
- added R111: 0, Resistor_SMD:R_0603_1608Metric, F.Cu at (34.2, 618.0)
- added R112: 33k, Resistor_SMD:R_0603_1608Metric, F.Cu at (25.9, 618.1)
- added R113: 82k, Resistor_SMD:R_0603_1608Metric, F.Cu at (29.1, 618.1)
- added R12: 10k, Resistor_SMD:R_0603_1608Metric, F.Cu at (35.5, -88.6)
- added R128: 1k, Resistor_SMD:R_0805_2012Metric, B.Cu at (75.4, 638.8)
- added R129: 1k, Resistor_SMD:R_0805_2012Metric, B.Cu at (72.7, 638.8)
- added R13: 51.1, Resistor_SMD:R_0603_1608Metric, F.Cu at (35.5, -86.1)
- added R130: 1k, Resistor_SMD:R_0805_2012Metric, B.Cu at (69.9, 638.8)
- added R131: 1k, Resistor_SMD:R_0805_2012Metric, B.Cu at (67.1, 638.8)
- added R132: 1k, Resistor_SMD:R_0805_2012Metric, B.Cu at (64.4, 638.8)
- added R133: 1k, Resistor_SMD:R_0805_2012Metric, B.Cu at (61.6, 638.8)
- added R134: 1k, Resistor_SMD:R_0805_2012Metric, B.Cu at (58.8, 638.8)
- added R135: 1k, Resistor_SMD:R_0805_2012Metric, B.Cu at (101.3, 618.8)
- added R136: 1k, Resistor_SMD:R_0805_2012Metric, B.Cu at (104.0, 618.8)
- added R137: 1k, Resistor_SMD:R_0805_2012Metric, B.Cu at (106.8, 618.8)
- added R138: 1k, Resistor_SMD:R_0805_2012Metric, B.Cu at (109.5, 618.8)
- added R139: 1k, Resistor_SMD:R_0805_2012Metric, B.Cu at (101.3, 638.7)
- added R14: ~, Resistor_SMD:R_0603_1608Metric, F.Cu at (35.5, -83.6)
- added R140: 1k, Resistor_SMD:R_0805_2012Metric, B.Cu at (104.0, 638.7)
- added R141: 1k, Resistor_SMD:R_0805_2012Metric, B.Cu at (106.8, 638.7)
- added R142: 1k, Resistor_SMD:R_0805_2012Metric, B.Cu at (109.5, 638.7)
- added R15: 100k, Resistor_SMD:R_0603_1608Metric, F.Cu at (35.5, -81.1)
- added R16: 3.74k, Resistor_SMD:R_0603_1608Metric, F.Cu at (35.5, -78.6)
- added R17: ~, Resistor_SMD:R_0603_1608Metric, F.Cu at (35.5, -76.1)
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Connections:
- J1 pad 1: (no net) -> PSU_EN
- J1 pad 2: (no net) -> GND
- J1 pad 3: (no net) -> GND
- J1 pad 4: (no net) -> +5VSB
- J2 pad 1: (no net) -> Net-(J2-Pin_1)
- J2 pad 2: (no net) -> Net-(J2-Pin_2)
- J2 pad 3: (no net) -> Net-(J2-Pin_3)
- J2 pad 4: (no net) -> Net-(J2-Pin_4)
- J3 pad 1: (no net) -> X_lLIM_1
- J3 pad 2: (no net) -> X_lLIM_2
- J3 pad 3: (no net) -> GND
- J4 pad 1: (no net) -> Net-(J4-Pin_1)
- J4 pad 2: (no net) -> Net-(J4-Pin_2)
- J4 pad 3: (no net) -> Net-(J4-Pin_3)
- J4 pad 4: (no net) -> Net-(J4-Pin_4)
- J5 pad 1: (no net) -> Y_lLIM_1
- J5 pad 2: (no net) -> Y_lLIM_2
- J5 pad 3: (no net) -> GND
- J6 pad 1: (no net) -> /X_ENC_INDEX_INPUT
- J6 pad 2: (no net) -> /X_ENC_CS_OUTPUT
- J6 pad 3: (no net) -> /X_ENC_CLK_OUTPUT

Commit message: m
Parts:
- removed C19: 22uF, Capacitor_SMD:C_1210_3225Metric
- removed C22: 100nF, Capacitor_SMD:C_0603_1608Metric
- removed J19: 5787834-1, Library:5787834-1
- removed J20: 031532951RFX, Library:031532951RFX
- removed J21: 10090929S154VLF, Library:10090929S154VLF
- removed J22, J23: LD09S24A4GV00LF, Library:LD09S24A4GV00LF
- removed R138, R139, R140, R141, R142: 1k, Resistor_SMD:R_0805_2012Metric
- removed R38: 0, Resistor_SMD:R_0603_1608Metric
- removed R55, R98: 10k, Resistor_SMD:R_0603_1608Metric
- removed the REF** at (12.0, 651.5)
- removed the REF** at (162.9, 650.5)
- added C118: 10pf, Capacitor_SMD:C_0603_1608Metric, F.Cu at (376.5, 122.2)
- added C119: 2.2uF, Capacitor_SMD:C_1206_3216Metric, F.Cu at (399.8, 111.3)
- added C120: 2.2uF, Capacitor_SMD:C_1206_3216Metric, F.Cu at (399.8, 114.6)
- added C121: 1nF, Capacitor_SMD:C_0603_1608Metric, F.Cu at (248.6, 97.4)
- added J17: B10B-XH-AM, Library:B10BXHAMLFSN, F.Cu at (370.5, 114.5)
- added R101: 47, Resistor_SMD:R_0603_1608Metric, F.Cu at (127.6, 176.3)
- added R114: 1k, Resistor_SMD:R_0805_2012Metric, F.Cu at (123.4, 161.4)
- added R115: 1k, Resistor_SMD:R_0805_2012Metric, F.Cu at (123.4, 164.4)
- added R116: 1k, Resistor_SMD:R_0805_2012Metric, F.Cu at (123.4, 167.3)
- added R117: 10k, Resistor_SMD:R_0603_1608Metric, F.Cu at (376.5, 127.2)
- added R118: 10k, Resistor_SMD:R_0603_1608Metric, F.Cu at (376.5, 129.7)
- added R119: 10k, Resistor_SMD:R_0603_1608Metric, F.Cu at (376.5, 132.2)
- added R120: 10k, Resistor_SMD:R_0603_1608Metric, F.Cu at (376.5, 134.8)
- added R121: 10k, Resistor_SMD:R_0603_1608Metric, F.Cu at (376.5, 137.3)
- added R122: 10k, Resistor_SMD:R_0603_1608Metric, F.Cu at (380.5, 119.7)
- added R123: 0, Resistor_SMD:R_0603_1608Metric, F.Cu at (380.5, 122.2)
- added R124: 0, Resistor_SMD:R_0603_1608Metric, F.Cu at (380.5, 124.7)
- added R125: 0, Resistor_SMD:R_0603_1608Metric, F.Cu at (380.5, 127.2)
- added R126: 0, Resistor_SMD:R_0603_1608Metric, F.Cu at (380.5, 129.7)
- added R127: 0, Resistor_SMD:R_0603_1608Metric, F.Cu at (380.5, 132.2)
- added R33: 0, Resistor_SMD:R_0603_1608Metric, F.Cu at (367.7, 174.5)
- added REF**: MountingHole_4.3mm_M4_DIN965_Pad_TopBottom, MountingHole:MountingHole_4.3mm_M4_DIN965_Pad_TopBottom, F.Cu at (162.3, 87.0)
- added REF**: MountingHole_4.3mm_M4_DIN965_Pad_TopBottom, MountingHole:MountingHole_4.3mm_M4_DIN965_Pad_TopBottom, F.Cu at (197.0, 51.8)
- added REF**: MountingHole_4.3mm_M4_DIN965_Pad_TopBottom, MountingHole:MountingHole_4.3mm_M4_DIN965_Pad_TopBottom, F.Cu at (197.0, 126.3)
- added REF**: MountingHole_4.3mm_M4_DIN965_Pad_TopBottom, MountingHole:MountingHole_4.3mm_M4_DIN965_Pad_TopBottom, F.Cu at (86.5, 51.8)
- added REF**: MountingHole_4.3mm_M4_DIN965_Pad_TopBottom, MountingHole:MountingHole_4.3mm_M4_DIN965_Pad_TopBottom, F.Cu at (86.5, 126.3)
- added REF**: MountingHole_4.3mm_M4_DIN965_Pad_TopBottom, MountingHole:MountingHole_4.3mm_M4_DIN965_Pad_TopBottom, F.Cu at (121.1, 87.0)
- added U17: STM32F446VETx, Package_QFP:LQFP-100_14x14mm_P0.5mm, F.Cu at (395.8, 127.7)
- C10, C11: value 10uF -> 22uF; footprint Capacitor_SMD:C_1210_3225Metric -> Capacitor_SMD:C_0805_2012Metric
- C100: value 4.7nF -> 4.7uF; moved to F.Cu
- C101, C102: value 4.7nF -> 100nF; footprint Capacitor_SMD:C_0805_2012Metric -> Capacitor_SMD:C_0603_1608Metric; moved to F.Cu
- C103, C50: value 4.7uF -> 100nF; footprint Capacitor_SMD:C_0805_2012Metric -> Capacitor_SMD:C_0603_1608Metric
- C108, C83, C90: value 100nF -> 1uF
- C111: value 1uF -> 100nF
- C114, C115: value 10pf -> 100nF
- C116: value 2.2uF -> 100nF; footprint Capacitor_SMD:C_1206_3216Metric -> Capacitor_SMD:C_0603_1608Metric
- C117: value 2.2uF -> 10pf; footprint Capacitor_SMD:C_1206_3216Metric -> Capacitor_SMD:C_0603_1608Metric
- C13, C14, C15: footprint Capacitor_SMD:C_0603_1608Metric -> Capacitor_SMD:C_0402_1005Metric
- C16: value 10uF -> 4.7uF; footprint Capacitor_SMD:C_1210_3225Metric -> Capacitor_SMD:C_0603_1608Metric
- C2: footprint Capacitor_SMD:C_1210_3225Metric -> Capacitor_SMD:C_0805_2012Metric; moved to F.Cu
- C20, C41: value 1uF -> 100nF; footprint Capacitor_SMD:C_1210_3225Metric -> Capacitor_SMD:C_0603_1608Metric
- C23: value 10uF -> 4.7uF; footprint Capacitor_SMD:C_2220_5750Metric -> Capacitor_SMD:C_0603_1608Metric
- C24, C44, C70: value 10uF -> 100nF; footprint Capacitor_SMD:C_2220_5750Metric -> Capacitor_SMD:C_0603_1608Metric
- C25: value 100uF -> 1uF; footprint Capacitor_SMD:CP_Elec_8x10 -> Capacitor_SMD:C_1210_3225Metric
- C26, C45: value 100uF -> 100nF; footprint Capacitor_SMD:CP_Elec_8x10 -> Capacitor_SMD:C_0603_1608Metric
- C28, C29, C47: value 100nF -> 10uF; footprint Capacitor_SMD:C_0603_1608Metric -> Capacitor_SMD:C_2220_5750Metric
- C3, D10, D11, D12, D13, D14, D15, D16, D17, D18, D19, D20, D3, D7, D8, D9: moved to F.Cu
- C30: value 4.7uF -> 100uF; footprint Capacitor_SMD:C_0805_2012Metric -> Capacitor_SMD:CP_Elec_8x10
- C31: value 22nF -> 100uF; footprint Capacitor_SMD:C_0805_2012Metric -> Capacitor_SMD:CP_Elec_8x10
- C32, C33, C34, C52: value 470pF -> 100nF; footprint Capacitor_SMD:C_0402_1005Metric -> Capacitor_SMD:C_0603_1608Metric
- C35, C53: value 470pF -> 4.7uF; footprint Capacitor_SMD:C_0402_1005Metric -> Capacitor_SMD:C_0805_2012Metric
- C36: value 100nF -> 22nF; footprint Capacitor_SMD:C_0603_1608Metric -> Capacitor_SMD:C_0805_2012Metric
- C37, C38, C39, C40, C56, C57, C58: value 100nF -> 470pF; footprint Capacitor_SMD:C_0603_1608Metric -> Capacitor_SMD:C_0402_1005Metric
- C43: value 10uF -> 1uF; footprint Capacitor_SMD:C_2220_5750Metric -> Capacitor_SMD:C_1210_3225Metric
- C46: value 100uF -> 10uF; footprint Capacitor_SMD:CP_Elec_8x10 -> Capacitor_SMD:C_2220_5750Metric
- C48, C49: value 100nF -> 100uF; footprint Capacitor_SMD:C_0603_1608Metric -> Capacitor_SMD:CP_Elec_8x10
- C51: value 22nF -> 100nF; footprint Capacitor_SMD:C_0805_2012Metric -> Capacitor_SMD:C_0603_1608Metric
- C54: value 470pF -> 22nF; footprint Capacitor_SMD:C_0402_1005Metric -> Capacitor_SMD:C_0805_2012Metric
- C61: value 1uF -> 220uF; footprint Capacitor_SMD:C_0603_1608Metric -> Capacitor_SMD:CP_Elec_8x10
- C62: footprint Capacitor_SMD:C_0201_0603Metric -> Capacitor_SMD:C_0603_1608Metric
- C64: value 1uF -> 22nF
- C66, C67: value 100nF -> 220uF; footprint Capacitor_SMD:C_0603_1608Metric -> Capacitor_SMD:CP_Elec_8x10
- C68: value 220uF -> 10uF; footprint Capacitor_SMD:CP_Elec_8x10 -> Capacitor_SMD:C_2220_5750Metric
- C69, C78, C85: value 220uF -> 100nF; footprint Capacitor_SMD:CP_Elec_8x10 -> Capacitor_SMD:C_0603_1608Metric
- C71, C76: value 100nF -> 22nF
- C73: value 22nF -> 220uF; footprint Capacitor_SMD:C_0603_1608Metric -> Capacitor_SMD:CP_Elec_8x10
- C8, C9: footprint Capacitor_SMD:C_1206_3216Metric -> Capacitor_SMD:C_1210_3225Metric
- C81, C88: value 22nF -> 100nF
- C84: footprint Capacitor_SMD:C_0603_1608Metric -> Capacitor_SMD:C_0201_0603Metric
- C98: value 4.7nF -> 100nF; footprint Capacitor_SMD:C_0805_2012Metric -> Capacitor_SMD:C_0603_1608Metric
- D4: value CDSOD323-T03C -> RED; footprint Diode_SMD:D_SOD-323 -> LED_SMD:LED_0603_1608Metric; moved to F.Cu
- D6: value RED -> CDSOD323-T03C; footprint LED_SMD:LED_0603_1608Metric -> Diode_SMD:D_SOD-323
- J1: value 44068-0057 -> 0430450606; footprint Library:44068-0057 -> Library:0430450606
- J10, J15: footprint Library:B3BXHAMLFSN -> Library:BM03BGHSTBTLFSN
- J11: value B2B-XH-AM -> B4B-XH-AM; footprint Library:B2BXHAMLFSN -> Library:BM04BGHSTBTLFSN
- J12: value B4B-XH-AM -> B2B-XH-AM; footprint Library:B4BXHAM -> Library:BM02B-GHS-TBT_1
- J13, J14: value B2B-XH-AM -> B6B-XH-AM; footprint Library:B2BXHAMLFSN -> Library:BM06BGHSTBTLFSN
- J16: value B10B-XH-AM -> Conn_01x34; footprint Library:B10BXHAMLFSN -> Library:F52Q1A7H111034
- J18: footprint Library:B4BXHAM -> Library:BM04BGHSTBTLFSN
- J2: footprint Library:B4BXHAM -> Connector_Molex:Molex_Micro-Fit_3.0_43045-0418_2x02-1MP_P3.00mm_Vertical
- J3: value B3B-XH-AM -> B4B-XH-AM; footprint Library:B3BXHAMLFSN -> Connector_Molex:Molex_Micro-Fit_3.0_43045-0418_2x02-1MP_P3.00mm_Vertical
- J4: value B4B-XH-AM -> B2B-XH-AM; footprint Library:B4BXHAM -> Library:43650-02YY_242526
- J5: value B3B-XH-AM -> B2B-XH-AM; footprint Library:B3BXHAMLFSN -> Library:43650-02YY_242526
- J6: value B6B-XH-AM -> B2B-XH-AM; footprint Library:B6BXHAMLFSN -> Library:43650-02YY_242526
- J7: value B6B-XH-AM -> B3B-XH-AM; footprint Library:B6BXHAMLFSN -> Library:BM03BGHSTBTLFSN
- J8: value B2B-XH-AM -> B3B-XH-AM; footprint Library:B2BXHAMLFSN -> Library:BM03BGHSTBTLFSN
- J9: value B4B-XH-AM -> B6B-XH-AM; footprint Library:B4BXHAM -> Library:BM06BGHSTBTLFSN
- L1: value 15uH -> 12uH; footprint Library:XAL6060153MEC -> Library:SRP6060FA150M
- R1: footprint Resistor_SMD:R_2512_6332Metric -> Resistor_SMD:R_1206_3216Metric
- R100, R27, R44, R99: value 10k -> 0
- R102, R110: value 10k -> 1k; footprint Resistor_SMD:R_0603_1608Metric -> Resistor_SMD:R_0805_2012Metric
- R103, R104, R111: value 0 -> 1k; footprint Resistor_SMD:R_0603_1608Metric -> Resistor_SMD:R_0805_2012Metric
- R105, R28, R45: value 0 -> 1k
- R106: value 47 -> 1k; footprint Resistor_SMD:R_0603_1608Metric -> Resistor_SMD:R_0805_2012Metric
- R107, R108, R109: value 0 -> 1k; moved to F.Cu
- R112: value 33k -> 1k; footprint Resistor_SMD:R_0603_1608Metric -> Resistor_SMD:R_0805_2012Metric
- R113: value 82k -> 1k; footprint Resistor_SMD:R_0603_1608Metric -> Resistor_SMD:R_0805_2012Metric
- R128, R137: value 1k -> 0; footprint Resistor_SMD:R_0805_2012Metric -> Resistor_SMD:R_0603_1608Metric; moved to F.Cu
- R129, R130, R131, R132, R133, R134, R135, R136: value 1k -> 10k; footprint Resistor_SMD:R_0805_2012Metric -> Resistor_SMD:R_0603_1608Metric; moved to F.Cu
- R19: value 1.1 -> 33k
- R2, R3: value 2k -> 1.5k
- R20: value 0 -> 19.1k
- R21, R70: value 0 -> 10k
- R22, R39: value 0 -> 1.1
- R23, R40: value 1k -> 22
- R24, R41, R91, R92, R93: value 0 -> 22
- R29, R48: value 1K -> 0
- R30, R31, R50: value 0.1 -> 0
- R32: value 20k -> 10k
- R34, R51: value 10K -> 1K
- R35, R52: value 10K -> 0.1
- R36: value 1.1 -> 0.1
- R37: value 0 -> 20k
- R4: value 51.1 -> 36
- R46: value 20k -> 0
- R47: value 100k -> 0
- R49: value 0.1 -> 10k
- R53: value 10k -> 0.1
- R54: value 10k -> 20k
- R57: value 10k -> 1k
- R60: value 1.62k -> 11k
- R62, R73: value 10K -> 0
- R63: value 10K -> 6.8k
- R69: value 3.3k -> 1.62k
- R71: value 2.2k -> 1k
- R72: value 2.2k -> 0
- R74: value 10k -> 11k
- R77: value 0 -> 6.8k
- R78, R80, R94: value 0 -> 10K
- R79: value 3.3k -> 10K
- R8: value 64.9k -> 47k
- R82: value 10K -> 10k
- R84, R85, R88, R95: value 10k -> 10K
- R89, R90: value 0 -> 2.2k
- R9: value 1.58k -> 1.3k
- R96: value 10k -> 33k
- R97: value 10k -> 82k
- SW1: footprint Library:SKRKAEE010 -> Library:PTS526SM15SMTR2LFS
- U10, U12, U13: value DRV8876PWPR -> SN74LVC2G17DBV; footprint Library:SOP65P640X120-17N -> Package_TO_SOT_SMD:SOT-23-6
- U14: value USBLC6-2SC6 -> SN74LVC2G17DBV
- U15: value 74LVC1G17 -> USBLC6-2SC6; footprint Package_TO_SOT_SMD:SOT-353_SC-70-5 -> Package_TO_SOT_SMD:SOT-23-6
- U16: value STM32F446VETx -> 74LVC1G17; footprint Package_QFP:LQFP-100_14x14mm_P0.5mm -> Package_TO_SOT_SMD:SOT-353_SC-70-5
- U4: value TMC2209-LA -> TPS2116DRL; footprint Package_DFN_QFN:VQFN-28-1EP_5x5mm_P0.5mm_EP3.7x3.7mm_ThermalVias -> Package_TO_SOT_SMD:SOT-583-8
- U6: value SN74LVC2G17DBV -> TMC2209-LA; footprint Package_TO_SOT_SMD:SOT-23-6 -> Package_DFN_QFN:VQFN-28-1EP_5x5mm_P0.5mm_EP3.7x3.7mm_ThermalVias
- U7, U8, U9: value SN74LVC2G17DBV -> DRV8876PWPR; footprint Package_TO_SOT_SMD:SOT-23-6 -> Library:SOP65P640X120-17N
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Connections:
- net /VIN renamed /POWER_INPUT/VIN
- net INPUT_IMON renamed /MCU/INPUT_IMON
- net PSU_EN renamed /POWER_INPUT/PWR_EN
- net X_DIAG renamed /X_Driver/XY_UART_TX
- net X_ENC_CS renamed /DC_DRIVERS/J_NSLEEP
- net Y_DIAG renamed /Y_DRIVER/XY_UART_TX
- net Y_ENC_CS renamed /DC_DRIVERS/F_NSLEEP
- C100 pad 2: /REMOTE_SH -> +3.3V
- C101 pad 1: /ACC2_SH -> GND
- C101 pad 2: GND -> +3.3V
- C102 pad 1: /ACC1_SH -> GND
- C102 pad 2: GND -> +3.3V
- C107 pad 2: +3.3V -> VDDA
- C108 pad 2: +3.3V -> VDDA
- C110 pad 2: VDDA -> EXP_GPIO_6
- C111 pad 2: VDDA -> EXP_GPIO_5
- C112 pad 2: VDDA -> EXP_GPIO_4
- C113 pad 2: MCU_RESET -> EXP_GPIO_3
- C114 pad 2: Net-(U16-PH0) -> EXP_GPIO_2
- C115 pad 2: Net-(U16-PH1) -> EXP_GPIO_1
- C116 pad 2: Net-(U16-VCAP_1) -> MCU_RESET
- C117 pad 2: Net-(U16-VCAP_2) -> Net-(U17-PH0)
- C16 pad 1: +5VSB -> +5V
- C17 pad 1: +5VSB -> +5V
- C18 pad 1: +3.3V -> Net-(U3-VI)
- C18 pad 2: GND -> /MCU/12V_PRES
- C20 pad 1: +12V -> Net-(U3-VI)
- C20 pad 2: Net-(C20-Pad2) -> GND
- C23 pad 1: +12V -> +5VSB
- C24 pad 1: +12V -> +5VSB
- C25 pad 2: GND -> Net-(C25-Pad2)
- C26 pad 1: +12V -> +3.3V
- C27 pad 2: Net-(U4-VCP) -> GND
- C28 pad 1: GND -> +12V
- C28 pad 2: Net-(U4-VREF) -> GND
- C29 pad 1: GND -> +12V
- C29 pad 2: Net-(U4-5VOUT) -> GND
- C30 pad 1: Net-(U4-5VOUT) -> +12V
- C31 pad 1: Net-(U4-CPO) -> +12V
- C31 pad 2: Net-(U4-CPI) -> GND
- C32 pad 1: Net-(J2-Pin_1) -> +12V
- C32 pad 2: GND -> Net-(U5-VCP)
- C33 pad 1: Net-(J2-Pin_2) -> GND
- C33 pad 2: GND -> Net-(U5-VREF)
- C34 pad 1: Net-(J2-Pin_3) -> GND
- C34 pad 2: GND -> Net-(U5-5VOUT)
- C35 pad 1: Net-(J2-Pin_4) -> Net-(U5-5VOUT)
- C36 pad 1: GND -> Net-(U5-CPO)
- C36 pad 2: Net-(U4-BRB) -> Net-(U5-CPI)
- C37 pad 1: GND -> Net-(J2-Pin_1)
- C37 pad 2: Net-(U4-BRA) -> GND
- C38 pad 1: GND -> Net-(J2-Pin_2)
- C38 pad 2: X_lLIM_2 -> GND
- C39 pad 1: GND -> Net-(J2-Pin_3)
- C39 pad 2: X_lLIM_1 -> GND
- C40 pad 1: +3.3V -> Net-(J2-Pin_4)
- C41 pad 1: +12V -> GND
- C41 pad 2: Net-(C41-Pad2) -> Net-(U5-BRB)
- C42 pad 1: +12V -> GND
- C42 pad 2: GND -> Net-(U5-BRA)
- C43 pad 2: GND -> Net-(C43-Pad2)
- C44 pad 1: +12V -> +3.3V
- C47 pad 2: Net-(U5-VCP) -> GND
- C48 pad 1: GND -> +12V
- C48 pad 2: Net-(U5-VREF) -> GND
- C49 pad 1: GND -> +12V
- C49 pad 2: Net-(U5-5VOUT) -> GND
- C50 pad 1: Net-(U5-5VOUT) -> +12V
- C50 pad 2: GND -> Net-(U6-VCP)
- C51 pad 1: Net-(U5-CPO) -> GND
- C51 pad 2: Net-(U5-CPI) -> Net-(U6-VREF)
- C52 pad 1: Net-(J4-Pin_1) -> GND
- C52 pad 2: GND -> Net-(U6-5VOUT)
- C53 pad 1: Net-(J4-Pin_2) -> Net-(U6-5VOUT)
- C54 pad 1: Net-(J4-Pin_3) -> Net-(U6-CPO)
- C54 pad 2: GND -> Net-(U6-CPI)
- C55 pad 1: Net-(J4-Pin_4) -> Net-(J3-Pin_1)
- C56 pad 1: GND -> Net-(J3-Pin_2)
- C56 pad 2: Net-(U5-BRB) -> GND
- C57 pad 1: GND -> Net-(J3-Pin_3)
- C57 pad 2: Net-(U5-BRA) -> GND
- C58 pad 1: GND -> Net-(J3-Pin_4)
- C58 pad 2: Y_lLIM_2 -> GND
- C59 pad 2: Y_lLIM_1 -> Net-(U6-BRB)
- C60 pad 2: +3.3V -> Net-(U6-BRA)
- C61 pad 1: GND -> +12V
- C61 pad 2: +3.3V -> GND
- C62 pad 1: GND -> +12V
- C62 pad 2: +3.3V -> GND
- C63 pad 1: GND -> Net-(U7-VCP)
- C63 pad 2: +3.3V -> +12V
- C64 pad 1: GND -> Net-(U7-CPL)
- C64 pad 2: +3.3V -> Net-(U7-CPH)
- C65 pad 2: +3.3V -> /DC_DRIVERS/J_FAULT
- C66 pad 1: GND -> +12V
- C66 pad 2: +3.3V -> GND
- C67 pad 1: GND -> +12V
- C67 pad 2: +3.3V -> GND
- C70 pad 1: +12V -> Net-(U8-VCP)
- C70 pad 2: GND -> +12V
- C71 pad 1: +12V -> Net-(U8-CPL)
- C71 pad 2: GND -> Net-(U8-CPH)
- C72 pad 1: Net-(U10-VCP) -> GND
- C72 pad 2: +12V -> /DC_DRIVERS/Z_FAULT
- C73 pad 1: Net-(U10-CPL) -> +12V
- C73 pad 2: Net-(U10-CPH) -> GND
- C74 pad 1: GND -> +12V
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Other:
- board outline added: 120 x 100 mm

Commit message: m
Parts:
- removed the D20 at (118.6, 125.7)
- removed the R106 at (114.6, 173.2)
- removed the R111 at (119.0, 170.3)
- added D6: CDSOD323-T03C, Diode_SMD:D_SOD-323, F.Cu at (116.3, 128.1)
- added R106: 1k, Resistor_SMD:R_0805_2012Metric, F.Cu at (130.2, 161.2)
- added R106: 1k, Resistor_SMD:R_0805_2012Metric, F.Cu at (123.9, 124.7)
- added R111: 1k, Resistor_SMD:R_0805_2012Metric, F.Cu at (133.4, 124.7)
- added R111: 1k, Resistor_SMD:R_0805_2012Metric, F.Cu at (134.6, 161.2)
- moved R100 63.4 mm to (100.8, 116.4), turned to 90 degrees
- moved R101 62.9 mm to (111.9, 115.4), turned to -90 degrees
- moved R99 62.0 mm to (98.9, 116.4), turned to 90 degrees
- moved R113 54.6 mm to (137.2, 124.7), turned to 90 degrees
- moved U16 53.3 mm to (113.8, 120.9), turned to 90 degrees
- moved R107 52.7 mm to (125.8, 124.7), turned to 90 degrees
- moved R112 51.2 mm to (135.3, 124.7), turned to 90 degrees
- moved R116 46.9 mm to (142.9, 124.7), turned to 90 degrees
- moved R105 46.2 mm to (122.0, 124.7), turned to 90 degrees
- moved R96 44.7 mm to (100.8, 130.4)
- moved R97 44.7 mm to (100.8, 132.9)
- moved R110 44.4 mm to (131.5, 124.7), turned to 90 degrees
- moved C98 43.7 mm to (100.9, 126.6)
- moved R115 43.4 mm to (141.0, 124.7), turned to 90 degrees
- moved R104 43.0 mm to (120.1, 124.7), turned to 90 degrees
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- renumbered D6 to D20
Connections:
- J16 pad 13: Net-(D19-A1) -> Net-(D7-A1)
- J16 pad 15: Net-(D18-A1) -> Net-(D8-A1)
- J16 pad 16: Net-(D17-A1) -> Net-(D9-A1)
- J16 pad 17: Net-(D16-A1) -> Net-(D10-A1)
- J16 pad 18: Net-(D15-A1) -> Net-(D11-A1)
- J16 pad 19: Net-(D14-A1) -> Net-(D12-A1)
- J16 pad 22: Net-(D12-A1) -> Net-(D14-A1)
- J16 pad 24: Net-(D11-A1) -> Net-(D15-A1)
- J16 pad 25: Net-(D10-A1) -> Net-(D16-A1)
- J16 pad 27: Net-(D9-A1) -> Net-(D17-A1)
- J16 pad 28: Net-(D8-A1) -> Net-(D18-A1)
- J16 pad 30: Net-(D7-A1) -> Net-(D19-A1)
- R100 pad 1: Net-(J16-Pin_8) -> Net-(R100-Pad1)
- R100 pad 2: Net-(R100-Pad2) -> /IO/USB_DN
- R103 pad 1: Net-(D19-A1) -> Net-(D7-A1)
- R104 pad 1: Net-(D18-A1) -> Net-(D8-A1)
- R105 pad 1: Net-(D17-A1) -> Net-(D9-A1)
- R107 pad 1: Net-(D15-A1) -> Net-(D11-A1)
- R108 pad 1: Net-(D14-A1) -> Net-(D12-A1)
- R110 pad 1: Net-(D12-A1) -> Net-(D14-A1)
- R112 pad 1: Net-(D10-A1) -> Net-(D16-A1)
- R113 pad 1: Net-(D9-A1) -> Net-(D17-A1)
- R114 pad 1: Net-(D8-A1) -> Net-(D18-A1)
- R115 pad 1: Net-(D7-A1) -> Net-(D19-A1)
- R99 pad 1: Net-(J16-Pin_7) -> Net-(R99-Pad1)
- R99 pad 2: Net-(R99-Pad2) -> /IO/USB_DP
- U15 pad 1: /IO/USB_DP -> Net-(J16-Pin_7)
- U15 pad 3: /IO/USB_DN -> Net-(J16-Pin_8)
- U15 pad 4: Net-(R100-Pad2) -> Net-(R100-Pad1)
- U15 pad 6: Net-(R99-Pad2) -> Net-(R99-Pad1)
Routing:
- net Net-(D6-A1): track 0.00 -> 7.04 mm
- net Net-(D8-A1): track 0.00 -> 6.22 mm
- net Net-(D9-A1): track 0.00 -> 5.12 mm
- net Net-(D20-A1): track 0.00 -> 4.80 mm
- net Net-(D10-A1): track 0.00 -> 4.50 mm
- net Net-(D18-A1): track 0.00 -> 4.47 mm
- net Net-(D19-A1): track 0.00 -> 4.42 mm
- net Net-(D16-A1): track 0.00 -> 4.13 mm
- net Net-(D11-A1): track 0.00 -> 4.13 mm
- net Net-(D17-A1): track 0.00 -> 4.09 mm
- net Net-(D14-A1): track 0.00 -> 3.80 mm
- net Net-(D13-A1): track 0.00 -> 3.79 mm
- net Net-(D15-A1): track 0.00 -> 3.76 mm
- net Net-(D12-A1): track 0.00 -> 3.75 mm
- net GND: track 0.00 -> 1.01 mm, vias 0 -> 1
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
Commit message: m
Parts:
- removed C1, C101, C102, C103, C104, C105, C106, C107, C109, C110, C111, C112, C113, C114, C115, C116, C12, C17, C18, C20, C21, C24, C26, C27, C3, C32, C33, C34, C41, C42, C44, C45, C50, C51, C52, C59, C60, C62, C63, C65, C69, C7, C70, C72, C74, C75, C77, C78, C79, C80, C81, C82, C85, C86, C87, C88, C89, C91, C92, C93, C94, C95, C96, C97, C98, C99: 100nF, Capacitor_SMD:C_0603_1608Metric
- removed C10, C11, C2: 22uF, Capacitor_SMD:C_0805_2012Metric
- removed C100, C35, C53: 4.7uF, Capacitor_SMD:C_0805_2012Metric
- removed C108, C83, C90: 1uF, Capacitor_SMD:C_0603_1608Metric
- removed C117, C118: 10pf, Capacitor_SMD:C_0603_1608Metric
- removed C119, C120: 2.2uF, Capacitor_SMD:C_1206_3216Metric
- removed C121: 1nF, Capacitor_SMD:C_0603_1608Metric
- removed C13: 10nF, Capacitor_SMD:C_0402_1005Metric
- removed C14: 120pF, Capacitor_SMD:C_0402_1005Metric
- removed C15: 12nF, Capacitor_SMD:C_0402_1005Metric
- removed C16, C23: 4.7uF, Capacitor_SMD:C_0603_1608Metric
- removed C25, C43: 1uF, Capacitor_SMD:C_1210_3225Metric
- removed C28, C29, C46, C47, C68: 10uF, Capacitor_SMD:C_2220_5750Metric
- removed C30, C31, C48, C49: 100uF, Capacitor_SMD:CP_Elec_8x10
- removed C36, C54: 22nF, Capacitor_SMD:C_0805_2012Metric
- removed C37, C38, C39, C40, C55, C56, C57, C58: 470pF, Capacitor_SMD:C_0402_1005Metric
- removed C4, C5, C61, C66, C67, C73: 220uF, Capacitor_SMD:CP_Elec_8x10
- removed C6: 33nF, Capacitor_SMD:C_0603_1608Metric
- removed C64, C71, C76: 22nF, Capacitor_SMD:C_0603_1608Metric
- removed C8, C9: 47uF, Capacitor_SMD:C_1210_3225Metric
- removed C84: 100nF, Capacitor_SMD:C_0201_0603Metric
- removed D1, D4, D5: RED, LED_SMD:LED_0603_1608Metric
- removed D10, D11, D12, D13, D14, D15, D16, D17, D18, D19, D20, D6, D7, D8, D9: CDSOD323-T03C, Diode_SMD:D_SOD-323
- removed D2: GREEN, LED_SMD:LED_0603_1608Metric
- removed D3: SMAJ15A, Diode_SMD:D_SMA
- removed J1: 0430450606, Library:0430450606
- removed J10, J15, J7, J8: B3B-XH-AM, Library:BM03BGHSTBTLFSN
- removed J11, J18: B4B-XH-AM, Library:BM04BGHSTBTLFSN
- removed J12: B2B-XH-AM, Library:BM02B-GHS-TBT_1
- removed J13, J14, J9: B6B-XH-AM, Library:BM06BGHSTBTLFSN
- removed J16: Conn_01x34, Library:F52Q1A7H111034
- removed J17: B10B-XH-AM, Library:B10BXHAMLFSN
- removed J2, J3: B4B-XH-AM, Connector_Molex:Molex_Micro-Fit_3.0_43045-0418_2x02-1MP_P3.00mm_Vertical
- removed J4, J5, J6: B2B-XH-AM, Library:43650-02YY_242526
- removed L1: 12uH, Library:SRP6060FA150M
- removed L2: FCM1608KF-601T05, Inductor_SMD:L_0603_1608Metric
- removed Q1: BSS84, Package_TO_SOT_SMD:SOT-23
- removed Q2: 2N7002, Package_TO_SOT_SMD:SOT-23
- removed R1: 0.002, Resistor_SMD:R_1206_3216Metric
- removed R10, R11, R117, R118, R119, R12, R120, R121, R122, R129, R130, R131, R132, R133, R134, R135, R136, R21, R32, R49, R56, R6, R64, R70, R82, R83, R86, R87: 10k, Resistor_SMD:R_0603_1608Metric
- removed R100, R123, R124, R125, R126, R127, R128, R137, R25, R26, R27, R29, R30, R31, R33, R42, R43, R44, R46, R47, R48, R50, R58, R59, R61, R62, R65, R66, R67, R68, R72, R73, R75, R76, R99: 0, Resistor_SMD:R_0603_1608Metric
- removed R101: 47, Resistor_SMD:R_0603_1608Metric
- removed R102, R103, R104, R105, R106 (x2), R107, R108, R109, R110, R111 (x2), R112, R113, R114, R115, R116: 1k, Resistor_SMD:R_0805_2012Metric
- removed R13: 51.1, Resistor_SMD:R_0603_1608Metric
- removed R14, R17: ~, Resistor_SMD:R_0603_1608Metric
- removed R15: 100k, Resistor_SMD:R_0603_1608Metric
- removed R16: 3.74k, Resistor_SMD:R_0603_1608Metric
- removed R18, R20: 19.1k, Resistor_SMD:R_0603_1608Metric
- removed R19, R96: 33k, Resistor_SMD:R_0603_1608Metric
- removed R2, R3: 1.5k, Resistor_SMD:R_0603_1608Metric
- removed R22, R39: 1.1, Resistor_SMD:R_0603_1608Metric
- removed R23, R24, R40, R41, R91, R92, R93: 22, Resistor_SMD:R_0603_1608Metric
- removed R28, R45, R57, R71: 1k, Resistor_SMD:R_0603_1608Metric
- removed R34, R51: 1K, Resistor_SMD:R_0603_1608Metric
- removed R35, R36, R52, R53: 0.1, Resistor_SMD:R_0603_1608Metric
- removed R37, R54: 20k, Resistor_SMD:R_0603_1608Metric
- removed R4: 36, Resistor_SMD:R_0603_1608Metric
- removed R5: 15k, Resistor_SMD:R_0603_1608Metric
- removed R60, R74: 11k, Resistor_SMD:R_0603_1608Metric
- removed R63, R77: 6.8k, Resistor_SMD:R_0603_1608Metric
- removed R69: 1.62k, Resistor_SMD:R_0603_1608Metric
- removed R7: 130k, Resistor_SMD:R_0603_1608Metric
- removed R78, R79, R80, R81, R84, R85, R88, R94, R95: 10K, Resistor_SMD:R_0603_1608Metric
- removed R8: 47k, Resistor_SMD:R_0603_1608Metric
- removed R89, R90: 2.2k, Resistor_SMD:R_0603_1608Metric
- removed R9: 1.3k, Resistor_SMD:R_0603_1608Metric
- removed R97: 82k, Resistor_SMD:R_0603_1608Metric
- removed REF** (x6): MountingHole_4.3mm_M4_DIN965_Pad_TopBottom, MountingHole:MountingHole_4.3mm_M4_DIN965_Pad_TopBottom
- removed RV1: 10k, Library:3314J-1
- removed SW1: RESET, Library:PTS526SM15SMTR2LFS
- removed SW2: SW_Push, Library:SKRKAEE010
- removed SW3: CJS1201A, Library:CJS1201A
- removed U1: TPS24751RUVR, Library:TPS24751RUVR
- removed U10, U11, U12, U13, U14: SN74LVC2G17DBV, Package_TO_SOT_SMD:SOT-23-6
- removed U15: USBLC6-2SC6, Package_TO_SOT_SMD:SOT-23-6
- removed U16: 74LVC1G17, Package_TO_SOT_SMD:SOT-353_SC-70-5
- removed U17: STM32F446VETx, Package_QFP:LQFP-100_14x14mm_P0.5mm
- removed U2: TPS54336ADDA, Package_SO:TI_SO-PowerPAD-8_ThermalVias
- removed U3: AMS1117-3.3, Package_TO_SOT_SMD:SOT-223-3_TabPin2
- removed U4: TPS2116DRL, Package_TO_SOT_SMD:SOT-583-8
- removed U5, U6: TMC2209-LA, Package_DFN_QFN:VQFN-28-1EP_5x5mm_P0.5mm_EP3.7x3.7mm_ThermalVias
- removed U7, U8, U9: DRV8876PWPR, Library:SOP65P640X120-17N
- removed Y1: X322516MMB4SI, Library:X322516MMB4SI
- added J**: LD09S24A4GV00LF, Library:LD09S24A4GV00LF, F.Cu at (100.2, 139.3)
- added J**: 5787834-1, Library:5787834-1, F.Cu at (34.3, 135.5)
- added J**: 44068-0057, Library:44068-0057, F.Cu at (181.3, 142.9)
- added J**: LD09S24A4GV00LF, Library:LD09S24A4GV00LF, F.Cu at (95.3, 176.6)
- added J**: 031532951RFX, Library:031532951RFX, F.Cu at (153.9, 140.8)
- added J**: 10090929S154VLF, Library:10090929S154VLF, F.Cu at (133.2, 138.8)
Routing:
- net Net-(D6-A1): track 7.04 -> 0.00 mm
- net Net-(D8-A1): track 6.22 -> 0.00 mm
- net Net-(D9-A1): track 5.12 -> 0.00 mm
- net Net-(D20-A1): track 4.80 -> 0.00 mm
- net Net-(D10-A1): track 4.50 -> 0.00 mm
- net Net-(D18-A1): track 4.47 -> 0.00 mm
- net Net-(D19-A1): track 4.42 -> 0.00 mm
- net Net-(D16-A1): track 4.13 -> 0.00 mm
- net Net-(D11-A1): track 4.13 -> 0.00 mm
- net Net-(D17-A1): track 4.09 -> 0.00 mm
- net Net-(D14-A1): track 3.80 -> 0.00 mm
- net Net-(D13-A1): track 3.79 -> 0.00 mm
- net Net-(D15-A1): track 3.76 -> 0.00 mm
- net Net-(D12-A1): track 3.75 -> 0.00 mm
- net GND: track 1.01 -> 0.00 mm, vias 1 -> 0
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Other:
- board size 120 x 100 mm -> 118 x 126 mm

Commit message: m
Parts:
- removed the J** at (133.2, 138.8)
- moved J** 81.1 mm to (72.9, 144.4)
- moved J** 45.8 mm to (99.2, 131.0), turned to 180 degrees
- moved J** 42.1 mm to (139.2, 142.0), turned to 180 degrees
- moved J** 40.7 mm to (72.9, 122.8)
- moved J** 7.72 mm to (99.2, 147.0), turned to 180 degrees
Other:
- outline, holes or cut-outs redrawn
