File: hardware/Ziess-Microsope-Controller_Main_board/Ziess-Microsope-Controller_Main_board.kicad_pcb (KiCad board)
At the start: 2 copper layers, 118 x 126 mm, 5 parts

Commit message: m
Parts:
- removed the J** at (99.2, 147.0)
- removed the J** at (72.9, 122.8)
- removed the J** at (139.2, 142.0)
- removed the J** at (99.2, 131.0)
- removed the J** at (72.9, 144.4)
- added C1: 100nF, Capacitor_SMD:C_0603_1608Metric, F.Cu at (421.9, 129.8)
- added C10: 22uF, Capacitor_SMD:C_0805_2012Metric, F.Cu at (393.4, 171.1)
- added C100: 4.7uF, Capacitor_SMD:C_0805_2012Metric, F.Cu at (414.9, 99.2)
- added C101: 100nF, Capacitor_SMD:C_0603_1608Metric, F.Cu at (383.1, 74.5)
- added C102: 100nF, Capacitor_SMD:C_0603_1608Metric, F.Cu at (383.1, 77.0)
- added C103: 100nF, Capacitor_SMD:C_0603_1608Metric, F.Cu at (383.1, 79.5)
- added C104: 100nF, Capacitor_SMD:C_0603_1608Metric, F.Cu at (383.1, 82.0)
- added C105: 100nF, Capacitor_SMD:C_0603_1608Metric, F.Cu at (383.1, 84.5)
- added C106: 100nF, Capacitor_SMD:C_0603_1608Metric, F.Cu at (383.1, 87.0)
- added C107: 100nF, Capacitor_SMD:C_0603_1608Metric, F.Cu at (383.1, 89.5)
- added C108: 1uF, Capacitor_SMD:C_0603_1608Metric, F.Cu at (383.1, 92.0)
- added C109: 100nF, Capacitor_SMD:C_0603_1608Metric, F.Cu at (387.1, 74.5)
- added C11: 22uF, Capacitor_SMD:C_0805_2012Metric, F.Cu at (393.4, 174.1)
- added C110: 100nF, Capacitor_SMD:C_0603_1608Metric, F.Cu at (387.1, 77.0)
- added C111: 100nF, Capacitor_SMD:C_0603_1608Metric, F.Cu at (387.1, 79.5)
- added C112: 100nF, Capacitor_SMD:C_0603_1608Metric, F.Cu at (387.1, 82.0)
- added C113: 100nF, Capacitor_SMD:C_0603_1608Metric, F.Cu at (387.1, 84.5)
- added C114: 100nF, Capacitor_SMD:C_0603_1608Metric, F.Cu at (387.1, 87.0)
- added C115: 100nF, Capacitor_SMD:C_0603_1608Metric, F.Cu at (387.1, 89.5)
- added C116: 100nF, Capacitor_SMD:C_0603_1608Metric, F.Cu at (387.1, 92.0)
- added C117: 10pf, Capacitor_SMD:C_0603_1608Metric, F.Cu at (391.1, 74.5)
- added C118: 10pf, Capacitor_SMD:C_0603_1608Metric, F.Cu at (391.1, 77.0)
- added C119: 2.2uF, Capacitor_SMD:C_1206_3216Metric, F.Cu at (414.4, 66.0)
- added C12: 100nF, Capacitor_SMD:C_0603_1608Metric, F.Cu at (375.5, 158.2)
- added C120: 2.2uF, Capacitor_SMD:C_1206_3216Metric, F.Cu at (414.4, 69.4)
- added C121: 1nF, Capacitor_SMD:C_0603_1608Metric, F.Cu at (421.9, 137.3)
- added C122: 4.7nF, Capacitor_SMD:C_0805_2012Metric, F.Cu at (366.5, 146.7)
- added C13: 10nF, Capacitor_SMD:C_0402_1005Metric, F.Cu at (395.5, 164.0)
- added C14: 120pF, Capacitor_SMD:C_0402_1005Metric, F.Cu at (395.5, 165.9)
- added C15: 12nF, Capacitor_SMD:C_0402_1005Metric, F.Cu at (395.5, 167.9)
- added C16: 4.7uF, Capacitor_SMD:C_0603_1608Metric, F.Cu at (375.5, 160.7)
- added C17: 100nF, Capacitor_SMD:C_0603_1608Metric, F.Cu at (375.5, 163.3)
- added C18: 100nF, Capacitor_SMD:C_0603_1608Metric, F.Cu at (375.5, 165.8)
- added C2: 22uF, Capacitor_SMD:C_0805_2012Metric, F.Cu at (434.1, 138.9)
- added C20: 100nF, Capacitor_SMD:C_0603_1608Metric, F.Cu at (375.5, 168.3)
- added C21: 100nF, Capacitor_SMD:C_0603_1608Metric, F.Cu at (375.5, 170.8)
- added C23: 4.7uF, Capacitor_SMD:C_0603_1608Metric, F.Cu at (379.5, 155.7)
- added C24: 100nF, Capacitor_SMD:C_0603_1608Metric, F.Cu at (379.5, 158.2)
- added C25: 1uF, Capacitor_SMD:C_1210_3225Metric, F.Cu at (140.6, 57.6)
- added C26: 100nF, Capacitor_SMD:C_0603_1608Metric, F.Cu at (116.0, 49.5)
- added C27: 100nF, Capacitor_SMD:C_0603_1608Metric, F.Cu at (116.0, 52.0)
- added C28: 10uF, Capacitor_SMD:C_2220_5750Metric, F.Cu at (134.4, 37.7)
- added C29: 10uF, Capacitor_SMD:C_2220_5750Metric, F.Cu at (134.4, 44.6)
- added C3: 100nF, Capacitor_SMD:C_0603_1608Metric, F.Cu at (421.9, 132.3)
- added C30: 100uF, Capacitor_SMD:CP_Elec_8x10, F.Cu at (132.0, 53.1)
- added C31: 100uF, Capacitor_SMD:CP_Elec_8x10, F.Cu at (132.0, 63.0)
- added C32: 100nF, Capacitor_SMD:C_0603_1608Metric, F.Cu at (116.0, 54.5)
- added C33: 100nF, Capacitor_SMD:C_0603_1608Metric, F.Cu at (116.0, 57.0)
- added C34: 100nF, Capacitor_SMD:C_0603_1608Metric, F.Cu at (116.0, 59.5)
- added C35: 4.7uF, Capacitor_SMD:C_0805_2012Metric, F.Cu at (140.0, 61.2)
- added C36: 22nF, Capacitor_SMD:C_0805_2012Metric, F.Cu at (140.0, 64.2)
- added C37: 470pF, Capacitor_SMD:C_0402_1005Metric, F.Cu at (140.1, 37.8)
- added C38: 470pF, Capacitor_SMD:C_0402_1005Metric, F.Cu at (140.1, 39.8)
- added C39: 470pF, Capacitor_SMD:C_0402_1005Metric, F.Cu at (140.1, 41.7)
- added C4: 220uF, Capacitor_SMD:CP_Elec_8x10, F.Cu at (442.9, 114.2)
- added C40: 470pF, Capacitor_SMD:C_0402_1005Metric, F.Cu at (140.1, 43.7)
- added C41: 100nF, Capacitor_SMD:C_0603_1608Metric, F.Cu at (147.2, 47.1)
- added C42: 100nF, Capacitor_SMD:C_0603_1608Metric, F.Cu at (154.2, 53.0)
- added C43: 1uF, Capacitor_SMD:C_1210_3225Metric, F.Cu at (448.3, 87.7)
- added C44: 100nF, Capacitor_SMD:C_0603_1608Metric, F.Cu at (423.6, 79.6)
- added C45: 100nF, Capacitor_SMD:C_0603_1608Metric, F.Cu at (423.6, 82.1)
- added C46: 10uF, Capacitor_SMD:C_2220_5750Metric, F.Cu at (442.1, 67.8)
- added C47: 10uF, Capacitor_SMD:C_2220_5750Metric, F.Cu at (442.1, 74.8)
- added C48: 100uF, Capacitor_SMD:CP_Elec_8x10, F.Cu at (439.7, 83.3)
- added C49: 100uF, Capacitor_SMD:CP_Elec_8x10, F.Cu at (439.7, 93.1)
- added C5: 220uF, Capacitor_SMD:CP_Elec_8x10, F.Cu at (442.9, 124.0)
- added C50: 100nF, Capacitor_SMD:C_0603_1608Metric, F.Cu at (423.6, 84.6)
- added C51: 100nF, Capacitor_SMD:C_0603_1608Metric, F.Cu at (423.6, 87.1)
- added C52: 100nF, Capacitor_SMD:C_0603_1608Metric, F.Cu at (423.6, 89.6)
- added C53: 4.7uF, Capacitor_SMD:C_0805_2012Metric, F.Cu at (447.7, 91.4)
- added C54: 22nF, Capacitor_SMD:C_0805_2012Metric, F.Cu at (447.7, 94.4)
- added C55: 470pF, Capacitor_SMD:C_0402_1005Metric, F.Cu at (447.8, 67.9)
- added C56: 470pF, Capacitor_SMD:C_0402_1005Metric, F.Cu at (447.8, 69.9)
- added C57: 470pF, Capacitor_SMD:C_0402_1005Metric, F.Cu at (447.8, 71.9)
- added C58: 470pF, Capacitor_SMD:C_0402_1005Metric, F.Cu at (447.8, 73.8)
- added C59: 100nF, Capacitor_SMD:C_0603_1608Metric, F.Cu at (423.6, 92.2)
- added C6: 33nF, Capacitor_SMD:C_0603_1608Metric, F.Cu at (421.9, 134.8)
- added C60: 100nF, Capacitor_SMD:C_0603_1608Metric, F.Cu at (423.6, 94.7)
- added C61: 220uF, Capacitor_SMD:CP_Elec_8x10, F.Cu at (339.6, 69.3)
- added C62: 100nF, Capacitor_SMD:C_0603_1608Metric, F.Cu at (365.0, 65.6)
- added C63: 100nF, Capacitor_SMD:C_0603_1608Metric, F.Cu at (365.0, 68.1)
- added C64: 22nF, Capacitor_SMD:C_0603_1608Metric, F.Cu at (365.0, 70.6)
- added C65: 100nF, Capacitor_SMD:C_0603_1608Metric, F.Cu at (365.0, 73.1)
- added C66: 220uF, Capacitor_SMD:CP_Elec_8x10, F.Cu at (339.6, 79.1)
- added C67: 220uF, Capacitor_SMD:CP_Elec_8x10, F.Cu at (339.6, 89.0)
- added C68: 10uF, Capacitor_SMD:C_2220_5750Metric, F.Cu at (349.6, 99.6)
- added C69: 100nF, Capacitor_SMD:C_0603_1608Metric, F.Cu at (365.0, 75.7)
- added C7: 100nF, Capacitor_SMD:C_0603_1608Metric, F.Cu at (375.5, 155.7)
- added C70: 100nF, Capacitor_SMD:C_0603_1608Metric, F.Cu at (365.0, 78.2)
- added C71: 22nF, Capacitor_SMD:C_0603_1608Metric, F.Cu at (365.0, 80.7)
- added C72: 100nF, Capacitor_SMD:C_0603_1608Metric, F.Cu at (365.0, 83.2)
- added C73: 220uF, Capacitor_SMD:CP_Elec_8x10, F.Cu at (339.6, 98.8)
- added C74: 100nF, Capacitor_SMD:C_0603_1608Metric, F.Cu at (365.0, 85.7)
- added C75: 100nF, Capacitor_SMD:C_0603_1608Metric, F.Cu at (369.1, 65.6)
- added C76: 22nF, Capacitor_SMD:C_0603_1608Metric, F.Cu at (369.1, 68.1)
- added C77: 100nF, Capacitor_SMD:C_0603_1608Metric, F.Cu at (369.1, 70.6)
- added C78: 100nF, Capacitor_SMD:C_0603_1608Metric, F.Cu at (399.8, 133.6)
- added C79: 100nF, Capacitor_SMD:C_0603_1608Metric, F.Cu at (399.8, 136.2)
- added C8: 47uF, Capacitor_SMD:C_1210_3225Metric, F.Cu at (388.3, 171.8)
- added C80: 100nF, Capacitor_SMD:C_0603_1608Metric, F.Cu at (399.8, 138.7)
- added C81: 100nF, Capacitor_SMD:C_0603_1608Metric, F.Cu at (399.8, 141.2)
- added C82: 100nF, Capacitor_SMD:C_0603_1608Metric, F.Cu at (399.8, 143.7)
- added C83: 1uF, Capacitor_SMD:C_0603_1608Metric, F.Cu at (399.8, 146.2)
- added C84: 100nF, Capacitor_SMD:C_0201_0603Metric, F.Cu at (404.2, 125.8)
- added C85: 100nF, Capacitor_SMD:C_0603_1608Metric, F.Cu at (399.8, 148.7)
- added C86: 100nF, Capacitor_SMD:C_0603_1608Metric, F.Cu at (399.8, 151.2)
- added C87: 100nF, Capacitor_SMD:C_0603_1608Metric, F.Cu at (403.8, 133.6)
- added C88: 100nF, Capacitor_SMD:C_0603_1608Metric, F.Cu at (403.8, 136.2)
- added C89: 100nF, Capacitor_SMD:C_0603_1608Metric, F.Cu at (403.8, 138.7)
- added C9: 47uF, Capacitor_SMD:C_1210_3225Metric, F.Cu at (388.3, 176.0)
- added C90: 1uF, Capacitor_SMD:C_0603_1608Metric, F.Cu at (403.8, 141.2)
- added C91: 100nF, Capacitor_SMD:C_0603_1608Metric, F.Cu at (403.8, 143.7)
- added C92: 100nF, Capacitor_SMD:C_0603_1608Metric, F.Cu at (403.8, 146.2)
- added C93: 100nF, Capacitor_SMD:C_0603_1608Metric, F.Cu at (403.8, 148.7)
- added C94: 100nF, Capacitor_SMD:C_0603_1608Metric, F.Cu at (403.8, 151.2)
- added C95: 100nF, Capacitor_SMD:C_0603_1608Metric, F.Cu at (407.8, 133.6)
- added C96: 100nF, Capacitor_SMD:C_0603_1608Metric, F.Cu at (407.8, 136.2)
- added C97: 100nF, Capacitor_SMD:C_0603_1608Metric, F.Cu at (407.8, 138.7)
- added C98: 100nF, Capacitor_SMD:C_0603_1608Metric, F.Cu at (369.4, 110.5)
- added C99: 100nF, Capacitor_SMD:C_0603_1608Metric, F.Cu at (369.4, 113.0)
- added D1: RED, LED_SMD:LED_0603_1608Metric, F.Cu at (450.7, 110.6)
- added D2: GREEN, LED_SMD:LED_0603_1608Metric, F.Cu at (450.7, 113.2)
- added D3: SMAJ15A, Diode_SMD:D_SMA, F.Cu at (449.3, 139.1)
- added D4: RED, LED_SMD:LED_0603_1608Metric, F.Cu at (140.7, 35.5)
- added D5: RED, LED_SMD:LED_0603_1608Metric, F.Cu at (448.4, 65.7)
- added J**: BM10BGHSTBT, Library:BM10BGHSTBT, F.Cu at (111.9, 125.9)
- added J**: BM06BGHSTBTLFSN, Library:BM06BGHSTBTLFSN, F.Cu at (72.9, 126.5)
- added J**: BM20BGHDSGTF, Library:BM20BGHDSGTF, F.Cu at (91.2, 125.4)
- added J**: BM10BGHSTBT, Library:BM10BGHSTBT, F.Cu at (132.1, 126.2)
- added J**: 0430450606, Library:0430450606, F.Cu at (150.4, 120.8)
- added J1: 0430450606, Library:0430450606, F.Cu at (428.4, 118.9)
- added J10: B3B-XH-AM, Library:BM03BGHSTBTLFSN, F.Cu at (378.6, 131.3)
- added J11: B4B-XH-AM, Library:BM04BGHSTBTLFSN, F.Cu at (408.7, 113.9)
- added J12: B2B-XH-AM, Library:BM02B-GHS-TBT_1, F.Cu at (406.4, 119.7)
- added J13: B6B-XH-AM, Library:BM06BGHSTBTLFSN, F.Cu at (390.8, 123.8)
- added J14: B6B-XH-AM, Library:BM06BGHSTBTLFSN, F.Cu at (390.8, 133.2)
- added J15: B3B-XH-AM, Library:BM03BGHSTBTLFSN, F.Cu at (378.6, 140.0)
- added J17: B10B-XH-AM, Library:B10BXHAMLFSN, F.Cu at (385.1, 69.3)
- added J18: B4B-XH-AM, Library:BM04BGHSTBTLFSN, F.Cu at (406.9, 96.3)
- added J19: 5787834-1, Library:5787834-1, F.Cu at (341.8, 142.3)
- added J2: B4B-XH-AM, Connector_Molex:Molex_Micro-Fit_3.0_43045-0418_2x02-1MP_P3.00mm_Vertical, F.Cu at (122.1, 41.2)
- added J20: 031532951RFX, Library:031532951RFX, F.Cu at (357.2, 147.6)
- added J22: LD09S24A4GV00LF, Library:LD09S24A4GV00LF, F.Cu at (356.0, 115.7)
- added J23: LD09S24A4GV00LF, Library:LD09S24A4GV00LF, F.Cu at (356.0, 131.3)
- added J3: B4B-XH-AM, Connector_Molex:Molex_Micro-Fit_3.0_43045-0418_2x02-1MP_P3.00mm_Vertical, F.Cu at (429.8, 71.4)
- added J4: B2B-XH-AM, Library:43650-02YY_242526, F.Cu at (354.2, 67.4)
- added J5: B2B-XH-AM, Library:43650-02YY_242526, F.Cu at (354.2, 78.0)
- added J6: B2B-XH-AM, Library:43650-02YY_242526, F.Cu at (354.2, 88.6)
- added J7: B3B-XH-AM, Library:BM03BGHSTBTLFSN, F.Cu at (378.6, 113.9)
- added J8: B3B-XH-AM, Library:BM03BGHSTBTLFSN, F.Cu at (378.6, 122.6)
- added J9: B6B-XH-AM, Library:BM06BGHSTBTLFSN, F.Cu at (390.8, 114.5)
- added L1: 12uH, Library:SRP6060FA150M, F.Cu at (389.8, 158.7)
- added L2: FCM1608KF-601T05, Inductor_SMD:L_0603_1608Metric, F.Cu at (391.1, 79.5)
- added Q1: BSS84, Package_TO_SOT_SMD:SOT-23, F.Cu at (434.3, 130.8)
- added Q2: 2N7002, Package_TO_SOT_SMD:SOT-23, F.Cu at (434.3, 135.2)
- added R1: 0.002, Resistor_SMD:R_1206_3216Metric, F.Cu at (449.8, 130.6)
- added R10: 10k, Resistor_SMD:R_0603_1608Metric, F.Cu at (429.9, 129.8)
- added R100: 0, Resistor_SMD:R_0603_1608Metric, F.Cu at (369.4, 123.1)
- added R101: 47, Resistor_SMD:R_0603_1608Metric, F.Cu at (369.4, 125.6)
- added R105: 0, Resistor_SMD:R_0805_2012Metric, F.Cu at (366.5, 149.7)
- added R11: 10k, Resistor_SMD:R_0603_1608Metric, F.Cu at (429.9, 132.3)
- added R117: 10k, Resistor_SMD:R_0603_1608Metric, F.Cu at (391.1, 82.0)
- added R118: 10k, Resistor_SMD:R_0603_1608Metric, F.Cu at (391.1, 84.5)
- added R119: 10k, Resistor_SMD:R_0603_1608Metric, F.Cu at (391.1, 87.0)
- added R12: 10k, Resistor_SMD:R_0603_1608Metric, F.Cu at (429.9, 134.8)
- added R120: 10k, Resistor_SMD:R_0603_1608Metric, F.Cu at (391.1, 89.5)
- added R121: 10k, Resistor_SMD:R_0603_1608Metric, F.Cu at (391.1, 92.0)
- added R122: 10k, Resistor_SMD:R_0603_1608Metric, F.Cu at (395.1, 74.5)
- added R123: 0, Resistor_SMD:R_0603_1608Metric, F.Cu at (395.1, 77.0)
- added R124: 0, Resistor_SMD:R_0603_1608Metric, F.Cu at (395.1, 79.5)
- added R125: 0, Resistor_SMD:R_0603_1608Metric, F.Cu at (395.1, 82.0)
- added R126: 0, Resistor_SMD:R_0603_1608Metric, F.Cu at (395.1, 84.5)
- added R127: 0, Resistor_SMD:R_0603_1608Metric, F.Cu at (395.1, 87.0)
- added R128: 0, Resistor_SMD:R_0603_1608Metric, F.Cu at (395.1, 89.5)
- added R129: 10k, Resistor_SMD:R_0603_1608Metric, F.Cu at (395.1, 92.0)
- added R13: 51.1, Resistor_SMD:R_0603_1608Metric, F.Cu at (379.5, 160.7)
- added R130: 10k, Resistor_SMD:R_0603_1608Metric, F.Cu at (399.1, 74.5)
- added R131: 10k, Resistor_SMD:R_0603_1608Metric, F.Cu at (399.1, 77.0)
- added R132: 10k, Resistor_SMD:R_0603_1608Metric, F.Cu at (399.1, 79.5)
- added R133: 10k, Resistor_SMD:R_0603_1608Metric, F.Cu at (399.1, 82.0)
- added R134: 10k, Resistor_SMD:R_0603_1608Metric, F.Cu at (399.1, 84.5)
- added R135: 10k, Resistor_SMD:R_0603_1608Metric, F.Cu at (399.1, 87.0)
- added R136: 10k, Resistor_SMD:R_0603_1608Metric, F.Cu at (399.1, 89.5)
- added R137: 0, Resistor_SMD:R_0603_1608Metric, F.Cu at (429.9, 137.3)
- added R14: ~, Resistor_SMD:R_0603_1608Metric, F.Cu at (379.5, 163.3)
- added R15: 100k, Resistor_SMD:R_0603_1608Metric, F.Cu at (379.5, 165.8)
- added R16: 3.74k, Resistor_SMD:R_0603_1608Metric, F.Cu at (379.5, 168.3)
- added R17: ~, Resistor_SMD:R_0603_1608Metric, F.Cu at (379.5, 170.8)
- added R18: 19.1k, Resistor_SMD:R_0603_1608Metric, F.Cu at (383.5, 155.7)
- added R19: 33k, Resistor_SMD:R_0603_1608Metric, F.Cu at (383.5, 158.2)
- added R2: 1.5k, Resistor_SMD:R_0603_1608Metric, F.Cu at (421.9, 139.8)
- added R20: 19.1k, Resistor_SMD:R_0603_1608Metric, F.Cu at (383.5, 160.7)
- added R21: 10k, Resistor_SMD:R_0603_1608Metric, F.Cu at (383.5, 163.3)
- added R22: 1.1, Resistor_SMD:R_0603_1608Metric, F.Cu at (116.0, 67.0)
- added R23: 22, Resistor_SMD:R_0603_1608Metric, F.Cu at (120.0, 49.5)
- added R24: 22, Resistor_SMD:R_0603_1608Metric, F.Cu at (120.0, 52.0)
- added R25: 0, Resistor_SMD:R_0603_1608Metric, F.Cu at (120.0, 54.5)
- added R26: 0, Resistor_SMD:R_0603_1608Metric, F.Cu at (120.0, 57.0)
- added R27: 0, Resistor_SMD:R_0603_1608Metric, F.Cu at (120.0, 59.5)
- added R28: 1k, Resistor_SMD:R_0603_1608Metric, F.Cu at (120.0, 62.0)
- added R29: 0, Resistor_SMD:R_0603_1608Metric, F.Cu at (120.0, 64.5)
- added R3: 1.5k, Resistor_SMD:R_0603_1608Metric, F.Cu at (421.9, 142.3)
- added R30: 0, Resistor_SMD:R_0603_1608Metric, F.Cu at (120.0, 67.0)
- added R31: 0, Resistor_SMD:R_0603_1608Metric, F.Cu at (124.0, 49.5)
- added R32: 10k, Resistor_SMD:R_0603_1608Metric, F.Cu at (124.0, 52.0)
- added R33: 0, Resistor_SMD:R_0603_1608Metric, F.Cu at (124.0, 54.5)
- added R34: 1K, Resistor_SMD:R_0603_1608Metric, F.Cu at (124.0, 57.0)
- added R35: 0.1, Resistor_SMD:R_2010_5025Metric, F.Cu at (149.6, 47.1)
- added R36: 0.1, Resistor_SMD:R_2010_5025Metric, F.Cu at (149.7, 56.6)
- added R37: 20k, Resistor_SMD:R_0603_1608Metric, F.Cu at (124.0, 64.5)
- added R39: 1.1, Resistor_SMD:R_0603_1608Metric, F.Cu at (423.6, 97.2)
- added R4: 36, Resistor_SMD:R_0603_1608Metric, F.Cu at (425.9, 129.8)
- added R40: 22, Resistor_SMD:R_0603_1608Metric, F.Cu at (427.7, 79.6)
- added R41: 22, Resistor_SMD:R_0603_1608Metric, F.Cu at (427.7, 82.1)
- added R42: 0, Resistor_SMD:R_0603_1608Metric, F.Cu at (427.7, 84.6)
- added R43: 0, Resistor_SMD:R_0603_1608Metric, F.Cu at (427.7, 87.1)
- added R44: 0, Resistor_SMD:R_0603_1608Metric, F.Cu at (427.7, 89.6)
- added R45: 1k, Resistor_SMD:R_0603_1608Metric, F.Cu at (427.7, 92.2)
- added R46: 0, Resistor_SMD:R_0603_1608Metric, F.Cu at (427.7, 94.7)
- added R47: 0, Resistor_SMD:R_0603_1608Metric, F.Cu at (427.7, 97.2)
- added R48: 0, Resistor_SMD:R_0603_1608Metric, F.Cu at (431.7, 79.6)
- added R49: 10k, Resistor_SMD:R_0603_1608Metric, F.Cu at (431.7, 82.1)
- added R5: 15k, Resistor_SMD:R_0603_1608Metric, F.Cu at (425.9, 132.3)
- added R50: 0, Resistor_SMD:R_0603_1608Metric, F.Cu at (431.7, 84.6)
- added R51: 1K, Resistor_SMD:R_0603_1608Metric, F.Cu at (431.7, 87.1)
- added R52: 0.1, Resistor_SMD:R_0603_1608Metric, F.Cu at (431.7, 89.6)
- added R53: 0.1, Resistor_SMD:R_0603_1608Metric, F.Cu at (431.7, 92.2)
- added R54: 20k, Resistor_SMD:R_0603_1608Metric, F.Cu at (431.7, 94.7)
- added R56: 10k, Resistor_SMD:R_0603_1608Metric, F.Cu at (369.1, 73.1)
- added R57: 1k, Resistor_SMD:R_0603_1608Metric, F.Cu at (369.1, 75.7)
- added R58: 0, Resistor_SMD:R_0603_1608Metric, F.Cu at (369.1, 78.2)
- added R59: 0, Resistor_SMD:R_0603_1608Metric, F.Cu at (369.1, 80.7)
- added R6: 10k, Resistor_SMD:R_0603_1608Metric, F.Cu at (425.9, 134.8)
- added R60: 11k, Resistor_SMD:R_0603_1608Metric, F.Cu at (369.1, 83.2)
- added R61: 0, Resistor_SMD:R_0603_1608Metric, F.Cu at (369.1, 85.7)
- added R62: 0, Resistor_SMD:R_0603_1608Metric, F.Cu at (373.1, 65.6)
- added R63: 6.8k, Resistor_SMD:R_0603_1608Metric, F.Cu at (373.1, 68.1)
- added R64: 10k, Resistor_SMD:R_0603_1608Metric, F.Cu at (373.1, 70.6)
- added R65: 0, Resistor_SMD:R_0603_1608Metric, F.Cu at (373.1, 73.1)
- added R66: 0, Resistor_SMD:R_0603_1608Metric, F.Cu at (373.1, 75.7)
- added R67: 0, Resistor_SMD:R_0603_1608Metric, F.Cu at (373.1, 78.2)
- added R68: 0, Resistor_SMD:R_0603_1608Metric, F.Cu at (373.1, 80.7)
- added R69: 1.62k, Resistor_SMD:R_0603_1608Metric, F.Cu at (373.1, 83.2)
- added R7: 130k, Resistor_SMD:R_0603_1608Metric, F.Cu at (425.9, 137.3)
- added R70: 10k, Resistor_SMD:R_0603_1608Metric, F.Cu at (373.1, 85.7)
- added R71: 1k, Resistor_SMD:R_0603_1608Metric, F.Cu at (377.1, 65.6)
- added R72: 0, Resistor_SMD:R_0603_1608Metric, F.Cu at (377.1, 68.1)
- added R73: 0, Resistor_SMD:R_0603_1608Metric, F.Cu at (377.1, 70.6)
- added R74: 11k, Resistor_SMD:R_0603_1608Metric, F.Cu at (377.1, 73.1)
- added R75: 0, Resistor_SMD:R_0603_1608Metric, F.Cu at (377.1, 75.7)
- added R76: 0, Resistor_SMD:R_0603_1608Metric, F.Cu at (377.1, 78.2)
- added R77: 6.8k, Resistor_SMD:R_0603_1608Metric, F.Cu at (377.1, 80.7)
- added R78: 10K, Resistor_SMD:R_0603_1608Metric, F.Cu at (407.8, 141.2)
- added R79: 10K, Resistor_SMD:R_0603_1608Metric, F.Cu at (407.8, 143.7)
- added R8: 47k, Resistor_SMD:R_0603_1608Metric, F.Cu at (425.9, 139.8)
- added R80: 10K, Resistor_SMD:R_0603_1608Metric, F.Cu at (407.8, 146.2)
- added R81: 10K, Resistor_SMD:R_0603_1608Metric, F.Cu at (407.8, 148.7)
- added R82: 10k, Resistor_SMD:R_0603_1608Metric, F.Cu at (407.8, 151.2)
- added R83: 10k, Resistor_SMD:R_0603_1608Metric, F.Cu at (411.8, 133.6)
- added R84: 10K, Resistor_SMD:R_0603_1608Metric, F.Cu at (411.8, 136.2)
- added R85: 10K, Resistor_SMD:R_0603_1608Metric, F.Cu at (411.8, 138.7)
- added R86: 10k, Resistor_SMD:R_0603_1608Metric, F.Cu at (411.8, 141.2)
- added R87: 10k, Resistor_SMD:R_0603_1608Metric, F.Cu at (411.8, 143.7)
- added R88: 10K, Resistor_SMD:R_0603_1608Metric, F.Cu at (411.8, 146.2)
- added R89: 2.2k, Resistor_SMD:R_0603_1608Metric, F.Cu at (411.8, 148.7)
- added R9: 1.3k, Resistor_SMD:R_0603_1608Metric, F.Cu at (425.9, 142.3)
- added R90: 2.2k, Resistor_SMD:R_0603_1608Metric, F.Cu at (411.8, 151.2)
- added R91: 22, Resistor_SMD:R_0603_1608Metric, F.Cu at (415.8, 133.6)
- added R92: 22, Resistor_SMD:R_0603_1608Metric, F.Cu at (415.8, 136.2)
- added R93: 22, Resistor_SMD:R_0603_1608Metric, F.Cu at (415.8, 138.7)
- added R94: 10K, Resistor_SMD:R_0603_1608Metric, F.Cu at (415.8, 141.2)
- added R95: 10K, Resistor_SMD:R_0603_1608Metric, F.Cu at (415.8, 143.7)
- added R96: 33k, Resistor_SMD:R_0603_1608Metric, F.Cu at (369.4, 115.5)
- added R97: 82k, Resistor_SMD:R_0603_1608Metric, F.Cu at (369.4, 118.1)
- added R99: 0, Resistor_SMD:R_0603_1608Metric, F.Cu at (369.4, 120.6)
- added RV1: 10k, Library:3314J-1, F.Cu at (356.9, 100.0)
- added SW1: RESET, Library:PTS526SM15SMTR2LFS, F.Cu at (441.9, 132.9)
- added SW2: SW_Push, Library:SKRKAEE010, F.Cu at (394.2, 96.3)
- added SW3: CJS1201A, Library:CJS1201A, F.Cu at (385.6, 96.8)
- added U1: TPS24751RUVR, Library:TPS24751RUVR, F.Cu at (441.1, 139.3)
- added U10: SN74LVC2G17DBV, Package_TO_SOT_SMD:SOT-23-6, F.Cu at (400.4, 111.7)
- added U11: SN74LVC2G17DBV, Package_TO_SOT_SMD:SOT-23-6, F.Cu at (400.4, 116.3)
- added U12: SN74LVC2G17DBV, Package_TO_SOT_SMD:SOT-23-6, F.Cu at (400.4, 120.9)
- added U13: SN74LVC2G17DBV, Package_TO_SOT_SMD:SOT-23-6, F.Cu at (400.4, 125.5)
- added U14: SN74LVC2G17DBV, Package_TO_SOT_SMD:SOT-23-6, F.Cu at (400.4, 130.2)
- added U15: USBLC6-2SC6, Package_TO_SOT_SMD:SOT-23-6, F.Cu at (366.8, 143.0)
- added U16: 74LVC1G17, Package_TO_SOT_SMD:SOT-353_SC-70-5, F.Cu at (366.2, 153.0)
- added U17: STM32F446VETx, Package_QFP:LQFP-100_14x14mm_P0.5mm, F.Cu at (410.4, 82.5)
- added U2: TPS54336ADDA, Package_SO:TI_SO-PowerPAD-8_ThermalVias, F.Cu at (389.8, 166.4)
- added U3: AMS1117-3.3, Package_TO_SOT_SMD:SOT-223-3_TabPin2, F.Cu at (378.4, 176.2)
- added U4: TPS2116DRL, Package_TO_SOT_SMD:SOT-583-8, F.Cu at (393.0, 177.7)
- added U5: TMC2209-LA, Package_DFN_QFN:VQFN-28-1EP_5x5mm_P0.5mm_EP3.7x3.7mm_ThermalVias, F.Cu at (141.8, 51.8)
- added U6: TMC2209-LA, Package_DFN_QFN:VQFN-28-1EP_5x5mm_P0.5mm_EP3.7x3.7mm_ThermalVias, F.Cu at (449.5, 82.0)
- added U7: DRV8876PWPR, Library:SOP65P640X120-17N, F.Cu at (367.5, 90.4)
- added U8: DRV8876PWPR, Library:SOP65P640X120-17N, F.Cu at (367.5, 97.2)
- added U9: DRV8876PWPR, Library:SOP65P640X120-17N, F.Cu at (367.5, 104.0)
- added Y1: X322516MMB4SI, Library:X322516MMB4SI, F.Cu at (416.0, 94.7)
Routing:
- net Net-(U5-BRB): track 0.00 -> 8.83 mm
- net Net-(U5-BRA): track 0.00 -> 6.02 mm
- net Net-(J2-Pin_1): track 0.00 -> 3.34 mm
- net Net-(J2-Pin_3): track 0.00 -> 3.15 mm
- added copper zone on F.Cu, net Net-(J2-Pin_1)
- added copper zone on F.Cu, net Net-(J2-Pin_3)
Other:
- outline, holes or cut-outs redrawn

Commit message: m
Parts:
- removed the J** at (91.2, 125.4)
- added PS**: NXJ1S1205MCR13, Library:NXJ1S1205MCR13, F.Cu at (124.1, 101.1)
- moved J** 17.2 mm to (94.8, 126.5)
- moved J** 13.1 mm to (119.1, 126.7)

Commit message: m
Parts:
- removed the J** at (119.1, 126.7)
- removed PS**: NXJ1S1205MCR13, Library:NXJ1S1205MCR13
- added C123: 100nF, Capacitor_SMD:C_0603_1608Metric, F.Cu at (107.3, 99.7)
- added C124: 100nF, Capacitor_SMD:C_1206_3216Metric, F.Cu at (118.2, 96.4)
- added C125: 4.7uF, Capacitor_SMD:C_0805_2012Metric, F.Cu at (116.8, 115.7)
- added C126: 100nF, Capacitor_SMD:C_0603_1608Metric, F.Cu at (107.4, 113.7)
- added C127: 100nF, Capacitor_SMD:C_0402_1005Metric, F.Cu at (128.6, 107.9)
- added C128: 100nF, Capacitor_SMD:C_0402_1005Metric, F.Cu at (128.6, 109.8)
- added C129: 10uF, Capacitor_SMD:C_1206_3216Metric, F.Cu at (131.0, 124.6)
- added C130: C_Polarized_Small, Capacitor_SMD:CP_Elec_4x3, F.Cu at (132.2, 114.2)
- added C131: 100nF, Capacitor_SMD:C_0603_1608Metric, F.Cu at (132.1, 104.3)
- added C132: 1uF, Capacitor_SMD:C_0603_1608Metric, F.Cu at (132.1, 105.9)
- added D6: BZT52C5V6, Diode_SMD:D_SOD-123F, F.Cu at (116.3, 118.1)
- added D7: RED, LED_SMD:LED_0603_1608Metric, F.Cu at (138.4, 110.2)
- added D9: SMAJ12A, Diode_SMD:D_SMC, F.Cu at (133.6, 120.0)
- added J21: Conn_01x10, Library:BM10BGHSTBT, F.Cu at (119.2, 127.2)
- added L3: 10uH, Library:8200, F.Cu at (113.7, 96.4)
- added L4: 10uH, Library:8200, F.Cu at (120.8, 115.7)
- added PS1: NXJ1S1205MC-R13, Library:NXJ1S1205MCR13, F.Cu at (117.2, 106.0)
- added Q3: 2N7002, Package_TO_SOT_SMD:SOT-23, F.Cu at (137.5, 107.3)
- added R102: 33, Resistor_SMD:R_0603_1608Metric, F.Cu at (104.5, 114.5)
- added R103: 33, Resistor_SMD:R_0603_1608Metric, F.Cu at (102.9, 114.5)
- added R104: 10k, Resistor_SMD:R_0603_1608Metric, F.Cu at (103.1, 99.0)
- added R106: 33, Resistor_SMD:R_0603_1608Metric, F.Cu at (104.8, 99.0)
- added R107: 33, Resistor_SMD:R_0603_1608Metric, F.Cu at (101.5, 99.0)
- added R108: 10k, Resistor_SMD:R_0603_1608Metric, F.Cu at (134.4, 106.8)
- added R109: 10k, Resistor_SMD:R_0603_1608Metric, F.Cu at (134.4, 109.9)
- added R110: 100, Resistor_SMD:R_0603_1608Metric, F.Cu at (135.2, 104.4)
- added R111: 390k, Resistor_SMD:R_0603_1608Metric, F.Cu at (136.0, 109.9)
- added R112: 390k, Resistor_SMD:R_0603_1608Metric, F.Cu at (127.3, 108.9)
- added R113: 10k, Resistor_SMD:R_0603_1608Metric, F.Cu at (126.5, 111.3)
- added R114: 10k, Resistor_SMD:R_0603_1608Metric, F.Cu at (126.5, 112.8)
- added R115: 10k, Resistor_SMD:R_0603_1608Metric, F.Cu at (139.4, 104.5)
- added R116: 1.5k, Resistor_SMD:R_0603_1608Metric, F.Cu at (140.1, 106.9)
- added U18: STM32F765VGTx, Package_QFP:LQFP-100_14x14mm_P0.5mm, F.Cu at (-89.9, 270.3)
- added U19: ISO1430DWR, Library:SOIC127P1030X265-16N, F.Cu at (103.8, 106.7)
- added U20: TPS259472LRPWR, Library:TPS259472LRPWR, F.Cu at (131.4, 108.9)
Routing:
- net Net-(Q3-G): track 0.00 -> 8.47 mm
- net Net-(U20-OVLO/_OVCSEL): track 0.00 -> 4.33 mm
