File: hardware/Ziess-Microsope-Controller_Main_board/Ziess-Microsope-Controller_Main_board.kicad_pcb (KiCad board)
At the start: 2 copper layers, 118 x 126 mm, 330 parts, among them J1 0430450606, J10 B3B-XH-AM, J11 B4B-XH-AM, J12 B2B-XH-AM, J13 B6B-XH-AM, J14 B6B-XH-AM, J15 B3B-XH-AM, J17 B10B-XH-AM, J18 B4B-XH-AM, J19 5787834-1, J2 B4B-XH-AM, J20 031532951RFX, J21 Conn_01x10, J22 LD09S24A4GV00LF, J23 LD09S24A4GV00LF, J3 B4B-XH-AM, J4 B2B-XH-AM, J5 B2B-XH-AM, J6 B2B-XH-AM, J7 B3B-XH-AM, J8 B3B-XH-AM, J9 B6B-XH-AM, Q1 BSS84, Q2 2N7002, Q3 2N7002, SW1 RESET, SW2 SW_Push, SW3 CJS1201A, U1 TPS24751RUVR, U10 SN74LVC2G17DBV, U11 SN74LVC2G17DBV, U12 SN74LVC2G17DBV, U13 SN74LVC2G17DBV, U14 SN74LVC2G17DBV, U15 USBLC6-2SC6, U16 74LVC1G17, U17 STM32F446VETx, U18 STM32F765VGTx, U19 ISO1430DWR, U2 TPS54336ADDA, U20 TPS259472LRPWR, U3 AMS1117-3.3, U4 TPS2116DRL, U5 TMC2209-LA, U6 TMC2209-LA, U7 DRV8876PWPR, U8 DRV8876PWPR, U9 DRV8876PWPR, Y1 X322516MMB4SI

Commit message: m
Parts:
- removed C106, C123, C126, C98: 100nF, Capacitor_SMD:C_0603_1608Metric
- removed C124: 100nF, Capacitor_SMD:C_1206_3216Metric
- removed C125: 4.7uF, Capacitor_SMD:C_0805_2012Metric
- removed the C25 at (140.6, 57.6)
- removed the C26 at (116.0, 49.5)
- removed the C27 at (116.0, 52.0)
- removed the C28 at (134.4, 37.7)
- removed the C29 at (134.4, 44.6)
- removed the C30 at (132.0, 53.1)
- removed the C31 at (132.0, 63.0)
- removed the C32 at (116.0, 54.5)
- removed the C33 at (116.0, 57.0)
- removed the C34 at (116.0, 59.5)
- removed the C35 at (140.0, 61.2)
- removed the C36 at (140.0, 64.2)
- removed the C37 at (140.1, 37.8)
- removed the C38 at (140.1, 39.8)
- removed the C39 at (140.1, 41.7)
- removed the C40 at (140.1, 43.7)
- removed the C41 at (147.2, 47.1)
- removed the C42 at (154.2, 53.0)
- removed the C61 at (339.6, 69.3)
- removed the C62 at (365.0, 65.6)
- removed the C63 at (365.0, 68.1)
- removed the C64 at (365.0, 70.6)
- removed the C65 at (365.0, 73.1)
- removed the D4 at (140.7, 35.5)
- removed D6: BZT52C5V6, Diode_SMD:D_SOD-123F
- removed J**: BM10BGHSTBT, Library:BM10BGHSTBT
- removed J**: BM06BGHSTBTLFSN, Library:BM06BGHSTBTLFSN
- removed J**: 0430450606, Library:0430450606
- removed J19: 5787834-1, Library:5787834-1
- removed the J2 at (122.1, 41.2)
- removed J23: LD09S24A4GV00LF, Library:LD09S24A4GV00LF
- removed the J4 at (354.2, 67.4)
- removed L3, L4: 10uH, Library:8200
- removed PS1: NXJ1S1205MC-R13, Library:NXJ1S1205MCR13
- removed R105: 0, Resistor_SMD:R_0805_2012Metric
- removed R107: 33, Resistor_SMD:R_0603_1608Metric
- removed the R22 at (116.0, 67.0)
- removed the R23 at (120.0, 49.5)
- removed the R24 at (120.0, 52.0)
- removed the R25 at (120.0, 54.5)
- removed the R26 at (120.0, 57.0)
- removed the R27 at (120.0, 59.5)
- removed the R28 at (120.0, 62.0)
- removed the R29 at (120.0, 64.5)
- removed the R30 at (120.0, 67.0)
- removed the R31 at (124.0, 49.5)
- removed the R32 at (124.0, 52.0)
- removed the R33 at (124.0, 54.5)
- removed the R34 at (124.0, 57.0)
- removed the R35 at (149.6, 47.1)
- removed the R36 at (149.7, 56.6)
- removed the R37 at (124.0, 64.5)
- removed the R56 at (369.1, 73.1)
- removed the R57 at (369.1, 75.7)
- removed the R58 at (369.1, 78.2)
- removed the R59 at (369.1, 80.7)
- removed the R60 at (369.1, 83.2)
- removed the R61 at (369.1, 85.7)
- removed the R62 at (373.1, 65.6)
- removed the R63 at (373.1, 68.1)
- removed U17: STM32F446VETx, Package_QFP:LQFP-100_14x14mm_P0.5mm
- removed U19: ISO1430DWR, Library:SOIC127P1030X265-16N
- removed the U5 at (141.8, 51.8)
- removed the U7 at (367.5, 90.4)
- added C127: 100nF, Capacitor_SMD:C_0402_1005Metric, F.Cu at (112.5, 220.3)
- added C128: 100nF, Capacitor_SMD:C_1206_3216Metric, F.Cu at (112.4, 222.3)
- added C129: 10uF, Capacitor_SMD:C_1206_3216Metric, F.Cu at (114.9, 237.1)
- added C130: C_Polarized_Small, Capacitor_SMD:CP_Elec_4x3, F.Cu at (116.0, 226.6)
- added C131: 100nF, Capacitor_SMD:C_0603_1608Metric, F.Cu at (115.9, 216.8)
- added C132: 1uF, Capacitor_SMD:C_0603_1608Metric, F.Cu at (115.9, 218.3)
- added C133: 1uF, Capacitor_SMD:C_0603_1608Metric, F.Cu at (437.5, 131.1)
- added C134: 100nF, Capacitor_SMD:C_0603_1608Metric, F.Cu at (437.5, 133.6)
- added C135: 100nF, Capacitor_SMD:C_1206_3216Metric, F.Cu at (458.1, 139.3)
- added C136: 100nF, Capacitor_SMD:C_0402_1005Metric, F.Cu at (441.0, 145.9)
- added C137: 10uF, Capacitor_SMD:C_1206_3216Metric, F.Cu at (458.1, 142.6)
- added C138: C_Polarized_Small, Capacitor_SMD:CP_Elec_4x3, F.Cu at (451.4, 140.5)
- added C19: 22uF, Capacitor_Tantalum_SMD:CP_EIA-3528-21_Kemet-B, F.Cu at (172.6, 85.5)
- added C22: 22uF, Capacitor_Tantalum_SMD:CP_EIA-3528-21_Kemet-B, F.Cu at (163.2, 80.8)
- added C25: 1uF, Capacitor_SMD:C_1210_3225Metric, F.Cu at (105.8, 49.4)
- added C25: 1uF, Capacitor_SMD:C_1210_3225Metric, F.Cu at (182.4, 71.9)
- added C26: 100nF, Capacitor_SMD:C_0603_1608Metric, F.Cu at (175.7, 65.6)
- added C26: 100nF, Capacitor_SMD:C_0603_1608Metric, F.Cu at (112.5, 55.7)
- added C27: 100nF, Capacitor_SMD:C_0603_1608Metric, F.Cu at (181.0, 68.6)
- added C27: 100nF, Capacitor_SMD:C_0603_1608Metric, F.Cu at (107.3, 52.7)
- added C28: 10uF, Capacitor_SMD:C_2220_5750Metric, F.Cu at (190.3, 51.1)
- added C28: 10uF, Capacitor_SMD:C_2220_5750Metric, F.Cu at (98.0, 70.2)
- added C29: 10uF, Capacitor_SMD:C_2220_5750Metric, F.Cu at (190.3, 70.2)
- added C29: 10uF, Capacitor_SMD:C_2220_5750Metric, F.Cu at (98.0, 51.1)
- added C30: 100uF, Capacitor_SMD:CP_Elec_8x10, F.Cu at (198.5, 49.7)
- added C30: 100uF, Capacitor_SMD:CP_Elec_8x10, F.Cu at (89.7, 71.6)
- added C31: 100uF, Capacitor_SMD:CP_Elec_8x10, F.Cu at (198.5, 71.6)
- added C31: 100uF, Capacitor_SMD:CP_Elec_8x10, F.Cu at (89.7, 49.7)
- added C32: 100nF, Capacitor_SMD:C_0603_1608Metric, F.Cu at (110.7, 67.8)
- added C32: 100nF, Capacitor_SMD:C_0603_1608Metric, F.Cu at (177.6, 53.5)
- added C33: 100nF, Capacitor_SMD:C_0603_1608Metric, F.Cu at (177.3, 65.6)
- added C33: 100nF, Capacitor_SMD:C_0603_1608Metric, F.Cu at (110.9, 55.7)
- added C34: 100nF, Capacitor_SMD:C_0603_1608Metric, F.Cu at (114.3, 63.3)
- added C34: 100nF, Capacitor_SMD:C_0603_1608Metric, F.Cu at (173.9, 58.0)
- added C35: 4.7uF, Capacitor_SMD:C_0805_2012Metric, F.Cu at (173.7, 56.2)
- added C35: 4.7uF, Capacitor_SMD:C_0805_2012Metric, F.Cu at (114.5, 65.1)
- added C36: 22nF, Capacitor_SMD:C_0805_2012Metric, F.Cu at (177.8, 55.7)
- added C36: 22nF, Capacitor_SMD:C_0805_2012Metric, F.Cu at (110.4, 65.6)
- added C37: 470pF, Capacitor_SMD:C_0402_1005Metric, F.Cu at (187.1, 63.1)
- added C37: 470pF, Capacitor_SMD:C_0402_1005Metric, F.Cu at (101.1, 58.2)
- added C38: 470pF, Capacitor_SMD:C_0402_1005Metric, F.Cu at (179.6, 64.8)
- added C38: 470pF, Capacitor_SMD:C_0402_1005Metric, F.Cu at (108.6, 56.5)
- added C39: 470pF, Capacitor_SMD:C_0402_1005Metric, F.Cu at (101.1, 62.9)
- added C39: 470pF, Capacitor_SMD:C_0402_1005Metric, F.Cu at (187.1, 58.4)
- added C40: 470pF, Capacitor_SMD:C_0402_1005Metric, F.Cu at (181.7, 53.9)
- added C40: 470pF, Capacitor_SMD:C_0402_1005Metric, F.Cu at (106.6, 67.4)
- added C41: 100nF, Capacitor_SMD:C_0603_1608Metric, F.Cu at (105.7, 65.4)
- added C41: 100nF, Capacitor_SMD:C_0603_1608Metric, F.Cu at (182.5, 55.9)
- added C42: 100nF, Capacitor_SMD:C_0603_1608Metric, F.Cu at (105.7, 55.8)
- added C42: 100nF, Capacitor_SMD:C_0603_1608Metric, F.Cu at (182.5, 65.5)
- added C61: 220uF, Capacitor_SMD:CP_Elec_8x10, F.Cu at (168.0, 37.5)
- added C61: 220uF, Capacitor_SMD:CP_Elec_8x10, F.Cu at (98.6, 37.5)
- added C61: 220uF, Capacitor_SMD:CP_Elec_8x10, F.Cu at (133.3, 37.5)
- added C62: 100nF, Capacitor_SMD:C_0603_1608Metric, F.Cu at (105.9, 37.4)
- added C62: 100nF, Capacitor_SMD:C_0603_1608Metric, F.Cu at (140.6, 37.4)
- added C62: 100nF, Capacitor_SMD:C_0603_1608Metric, F.Cu at (175.3, 37.4)
- added C63: 100nF, Capacitor_SMD:C_0603_1608Metric, F.Cu at (105.3, 39.9)
- added C63: 100nF, Capacitor_SMD:C_0603_1608Metric, F.Cu at (140.1, 39.9)
- added C63: 100nF, Capacitor_SMD:C_0603_1608Metric, F.Cu at (174.8, 39.9)
- added C64: 22nF, Capacitor_SMD:C_0603_1608Metric, F.Cu at (140.0, 41.5)
- added C64: 22nF, Capacitor_SMD:C_0603_1608Metric, F.Cu at (105.3, 41.5)
- added C64: 22nF, Capacitor_SMD:C_0603_1608Metric, F.Cu at (174.8, 41.5)
- added C65: 100nF, Capacitor_SMD:C_0603_1608Metric, F.Cu at (188.7, 46.3)
- added C65: 100nF, Capacitor_SMD:C_0603_1608Metric, F.Cu at (119.3, 46.3)
- added C65: 100nF, Capacitor_SMD:C_0603_1608Metric, F.Cu at (154.0, 46.3)
- added D10: SMAJ12A, Diode_SMD:D_SMC, F.Cu at (453.0, 133.7)
- added D4: RED, LED_SMD:LED_0603_1608Metric, F.Cu at (169.8, 63.0)
- added D4: RED, LED_SMD:LED_0603_1608Metric, F.Cu at (118.4, 58.3)
- added D7: RED, LED_SMD:LED_0603_1608Metric, F.Cu at (122.2, 222.6)
- added D8: RED, LED_SMD:LED_0603_1608Metric, F.Cu at (437.5, 146.2)
- added D9: SMAJ12A, Diode_SMD:D_SMC, F.Cu at (117.5, 232.5)
- added H1: MountingHole, MountingHole:MountingHole_3.2mm_M3_DIN965_Pad_TopBottom, F.Cu at (88.8, 38.5)
- added H2: MountingHole, MountingHole:MountingHole_3.2mm_M3_DIN965_Pad_TopBottom, F.Cu at (199.3, 38.5)
- added H3: MountingHole, MountingHole:MountingHole_3.2mm_M3_DIN965_Pad_TopBottom, F.Cu at (199.3, 113.0)
- added H4: MountingHole, MountingHole:MountingHole_3.2mm_M3_DIN965_Pad_TopBottom, F.Cu at (88.8, 113.0)
- added IC1: TRS3122ERGER, Library:QFN50P400X400X100-25N-D, F.Cu at (457.7, 124.3)
- added J2: B4B-XH-AM, Connector_Molex:Molex_Micro-Fit_3.0_43045-0418_2x02-1MP_P3.00mm_Vertical, F.Cu at (94.0, 60.6)
- added J2: B4B-XH-AM, Connector_Molex:Molex_Micro-Fit_3.0_43045-0418_2x02-1MP_P3.00mm_Vertical, F.Cu at (194.2, 60.7)
- added J21: Conn_01x10, Library:BM10BGHSTBT, F.Cu at (103.1, 239.5)
- added J4: B2B-XH-AM, Library:43650-02YY_242526, F.Cu at (146.2, 28.8)
- added J4: B2B-XH-AM, Library:43650-02YY_242526, F.Cu at (111.5, 28.8)
- added J4: B2B-XH-AM, Library:43650-02YY_242526, F.Cu at (181.0, 28.8)
- added Q3: 2N7002, Package_TO_SOT_SMD:SOT-23, F.Cu at (121.3, 219.8)
- added Q4: 2N7002, Package_TO_SOT_SMD:SOT-23, F.Cu at (457.7, 146.5)
- added R108: 10k, Resistor_SMD:R_0603_1608Metric, F.Cu at (118.3, 219.2)
- added R109: 10k, Resistor_SMD:R_0603_1608Metric, F.Cu at (118.3, 222.3)
- added R110: 100, Resistor_SMD:R_0603_1608Metric, F.Cu at (119.0, 216.8)
- added R111: 390k, Resistor_SMD:R_0603_1608Metric, F.Cu at (119.8, 222.3)
- added R112: 390k, Resistor_SMD:R_0603_1608Metric, F.Cu at (111.2, 221.3)
- added R113: 10k, Resistor_SMD:R_0603_1608Metric, F.Cu at (110.3, 223.7)
- added R114: 10k, Resistor_SMD:R_0603_1608Metric, F.Cu at (110.3, 225.3)
- added R115: 10k, Resistor_SMD:R_0603_1608Metric, F.Cu at (123.2, 217.0)
- added R116: 1.5k, Resistor_SMD:R_0603_1608Metric, F.Cu at (123.9, 219.3)
- added R138: 10k, Resistor_SMD:R_0603_1608Metric, F.Cu at (441.5, 133.6)
- added R139: 10k, Resistor_SMD:R_0603_1608Metric, F.Cu at (441.5, 136.1)
- added R140: 390k, Resistor_SMD:R_0603_1608Metric, F.Cu at (441.5, 138.7)
- added R141: 390k, Resistor_SMD:R_0603_1608Metric, F.Cu at (441.5, 141.2)
- added R142: 10k, Resistor_SMD:R_0603_1608Metric, F.Cu at (441.5, 143.7)
- added R143: 10k, Resistor_SMD:R_0603_1608Metric, F.Cu at (445.5, 131.1)
- added R144: 10k, Resistor_SMD:R_0603_1608Metric, F.Cu at (445.5, 133.6)
- added R145: 1.5k, Resistor_SMD:R_0603_1608Metric, F.Cu at (445.5, 136.1)
- added R22: 1.1, Resistor_SMD:R_0603_1608Metric, F.Cu at (105.7, 52.7)
- added R22: 1.1, Resistor_SMD:R_0603_1608Metric, F.Cu at (182.5, 68.6)
- added R23: 22, Resistor_SMD:R_0603_1608Metric, F.Cu at (112.8, 52.2)
- added R23: 22, Resistor_SMD:R_0603_1608Metric, F.Cu at (175.4, 69.1)
- added R24: 22, Resistor_SMD:R_0603_1608Metric, F.Cu at (178.5, 71.7)
- added R24: 22, Resistor_SMD:R_0603_1608Metric, F.Cu at (109.7, 49.6)
- added R25: 0, Resistor_SMD:R_0603_1608Metric, F.Cu at (173.1, 53.6)
- added R25: 0, Resistor_SMD:R_0603_1608Metric, F.Cu at (115.1, 67.7)
- added R26: 0, Resistor_SMD:R_0603_1608Metric, F.Cu at (169.8, 59.6)
- added R26: 0, Resistor_SMD:R_0603_1608Metric, F.Cu at (118.4, 61.7)
- added R27: 0, Resistor_SMD:R_0603_1608Metric, F.Cu at (169.8, 61.3)
- added R27: 0, Resistor_SMD:R_0603_1608Metric, F.Cu at (118.4, 60.0)
- added R28: 1k, Resistor_SMD:R_0603_1608Metric, F.Cu at (169.8, 64.7)
- added R28: 1k, Resistor_SMD:R_0603_1608Metric, F.Cu at (118.4, 56.6)
- added R29: 0, Resistor_SMD:R_0603_1608Metric, F.Cu at (113.5, 67.7)
- added R29: 0, Resistor_SMD:R_0603_1608Metric, F.Cu at (174.7, 53.6)
- added R30: 0, Resistor_SMD:R_0603_1608Metric, F.Cu at (173.0, 59.6)
- added R30: 0, Resistor_SMD:R_0603_1608Metric, F.Cu at (115.2, 61.7)
- added R31: 0, Resistor_SMD:R_0603_1608Metric, F.Cu at (115.2, 60.0)
- added R31: 0, Resistor_SMD:R_0603_1608Metric, F.Cu at (173.0, 61.3)
- added R32: 10k, Resistor_SMD:R_0603_1608Metric, F.Cu at (109.7, 52.7)
- added R32: 10k, Resistor_SMD:R_0603_1608Metric, F.Cu at (178.5, 68.6)
- added R33: 0, Resistor_SMD:R_0603_1608Metric, F.Cu at (115.2, 56.6)
- added R33: 0, Resistor_SMD:R_0603_1608Metric, F.Cu at (173.0, 64.7)
- added R34: 1K, Resistor_SMD:R_0603_1608Metric, F.Cu at (115.2, 58.3)
- added R34: 1K, Resistor_SMD:R_0603_1608Metric, F.Cu at (173.0, 63.0)
- added R35: 0.1, Resistor_SMD:R_2010_5025Metric, F.Cu at (184.9, 55.7)
- added R35: 0.1, Resistor_SMD:R_2010_5025Metric, F.Cu at (103.3, 65.6)
- added R36: 0.1, Resistor_SMD:R_2010_5025Metric, F.Cu at (184.9, 65.7)
- added R36: 0.1, Resistor_SMD:R_2010_5025Metric, F.Cu at (103.3, 55.6)
- added R37: 20k, Resistor_SMD:R_0603_1608Metric, F.Cu at (179.9, 52.8)
- added R37: 20k, Resistor_SMD:R_0603_1608Metric, F.Cu at (108.3, 68.5)
- added R38: 100k, Resistor_SMD:R_0603_1608Metric, F.Cu at (178.5, 70.1)
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Connections:
- C117 pad 2: Net-(U17-PH0) -> Net-(U18-PH1)
- C118 pad 2: Net-(U17-PH1) -> Net-(U18-PH0)
- C119 pad 2: Net-(U17-VCAP_1) -> Net-(U18-VCAP_1)
- C120 pad 2: Net-(U17-VCAP_2) -> Net-(U18-VCAP_2)
- C122 pad 2: /IO/USB_SH -> USB_VBUS
- J18 pad 1: FAN1_PWM -> GND
- J18 pad 2: FAN1_RPM -> Net-(J18-Pin_2)
- J18 pad 3: +5V -> Net-(J18-Pin_3)
- J18 pad 4: GND -> USB_VBUS
- J20 pad 1: Net-(J20-In) -> GND
- J20 pad 3: GND -> Net-(J20-In)
- J21 pad 10: GND -> unconnected-(J21-Pin_10-Pad10)
- J21 pad 7: GND -> unconnected-(J21-Pin_7-Pad7)
- J22 pad 1: unconnected-(J22-Pad1) -> Net-(D10-A1)
- J22 pad 2: unconnected-(J22-Pad2) -> Net-(D10-A1)
- J22 pad 3: unconnected-(J22-Pad3) -> GND
- J22 pad 4: unconnected-(J22-Pad4) -> GND
- J22 pad 5: unconnected-(J22-Pad5) -> Net-(J22-Pin_5)
- J22 pad 6: unconnected-(J22-Pad6) -> Net-(J22-Pin_6)
- R100 pad 1: /IO/USB_DN -> Net-(R100-Pad1)
- R100 pad 2: Net-(R100-Pad2) -> /IO/USB_DN
- R102 pad 1: Net-(J21-Pin_5) -> unconnected-(R102-Pad1)
- R102 pad 2: Net-(U19-B) -> Net-(J21-Pin_5)
- R103 pad 1: Net-(J21-Pin_6) -> unconnected-(R103-Pad1)
- R103 pad 2: Net-(U19-A) -> Net-(J21-Pin_6)
- R104 pad 1: GND -> unconnected-(R104-Pad1)
- R104 pad 2: Net-(U19-DE) -> Net-(J22-Pin_5)
- R106 pad 1: Net-(U19-R) -> unconnected-(R106-Pad1)
- R106 pad 2: unconnected-(R106-Pad2) -> Net-(J22-Pin_6)
- R134 pad 1: EXP_GPIO_6 -> EXP_GPIO_1
- R135 pad 2: Net-(U17-BOOT0) -> Net-(U18-BOOT0)
- R136 pad 1: FAN1_RPM -> Net-(U21-EN/UVLO_1)
- R136 pad 2: +5V -> /IO/RS_PWR_EN
- R99 pad 1: /IO/USB_DP -> Net-(R99-Pad1)
- R99 pad 2: Net-(R99-Pad2) -> /IO/USB_DP
- U15 pad 1: Net-(R99-Pad2) -> Net-(J18-Pin_3)
- U15 pad 3: Net-(R100-Pad2) -> Net-(J18-Pin_2)
- U15 pad 4: Net-(J19-D-) -> Net-(R100-Pad1)
- U15 pad 6: Net-(J19-D+) -> Net-(R99-Pad1)
- U18 pad 10: Net-(U18-VSS-Pad10) -> GND
- U18 pad 100: unconnected-(U18-VDD-Pad100) -> +3.3V
- U18 pad 11: unconnected-(U18-VDD-Pad11) -> +3.3V
- U18 pad 12: unconnected-(U18-PH0-Pad12) -> Net-(U18-PH0)
- U18 pad 13: unconnected-(U18-PH1-Pad13) -> Net-(U18-PH1)
- U18 pad 14: unconnected-(U18-NRST-Pad14) -> MCU_RESET
- U18 pad 19: unconnected-(U18-VSSA-Pad19) -> GND
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Routing:
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- added copper zone on F.Cu, net +12V
- added copper zone on In2.Cu, net +12V
- added copper zone on F.Cu, net +5V
- added copper zone on F.Cu, net +5VSB
- added copper zone on F.Cu, net /POWER_INPUT/VIN
- added copper zone on F.Cu, net GND
- added copper zone on In1.Cu, net GND
- added copper zone on B.Cu, net Net-(J2-Pin_1)
- added copper zone on B.Cu, net Net-(J2-Pin_2)
- added copper zone on F.Cu, net Net-(J2-Pin_2)
- added copper zone on B.Cu, net Net-(J2-Pin_3)
- added copper zone on B.Cu, net Net-(J2-Pin_4)
- added copper zone on F.Cu, net Net-(J2-Pin_4)
- added copper zone on F.Cu, net Net-(J4-Pin_1)
- added copper zone on F.Cu, net Net-(J4-Pin_2)
- added copper zone on B.Cu, net Net-(U1-DRAIN_2)
- added copper zone on F.Cu, net Net-(U1-DRAIN_2)
- added copper zone on In1.Cu, net Net-(U1-DRAIN_2)
- added copper zone on F.Cu, net Net-(U3-VI)
- added copper zone on F.Cu, net Net-(U5-BRA)
- added copper zone on F.Cu, net Net-(U5-BRB)
Other:
- board size 118 x 126 mm -> 120 x 100 mm
- copper layers 2 -> 4

Commit message: m
Parts:
- moved C14 160.9 mm to (218.4, 236.6)
- moved C19 160.9 mm to (233.3, 234.6)
- moved C20 160.9 mm to (234.7, 232.0)
- moved C7 160.9 mm to (207.1, 232.6)
- moved C8 160.9 mm to (208.4, 247.3)
- moved C9 160.9 mm to (208.5, 250.7)
- moved L1 160.9 mm to (206.8, 241.7)
- moved R18 160.9 mm to (219.2, 236.6)
- moved U2 160.9 mm to (212.4, 234.5)
- moved U3 160.9 mm to (229.4, 228.3)
- moved C10 160.9 mm to (200.5, 235.5)
- moved C11 160.9 mm to (202.6, 235.5)
- moved C12 160.9 mm to (204.4, 235.7)
- moved C121 160.9 mm to (231.9, 253.3)
- moved C13 160.9 mm to (217.2, 231.0)
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Other:
- board size 120 x 100 mm -> 120 x 130 mm

Commit message: m
Parts:
- removed the C61 at (168.0, 37.5)
- removed the C61 at (133.3, 37.5)
- removed the C62 at (140.6, 37.4)
- removed the C62 at (175.3, 37.4)
- removed the C63 at (140.1, 39.9)
- removed the C63 at (174.8, 39.9)
- removed the C64 at (140.0, 41.5)
- removed the C64 at (174.8, 41.5)
- removed the C65 at (188.7, 46.3)
- removed the C65 at (154.0, 46.3)
- removed H1, H2, H3, H4: MountingHole, MountingHole:MountingHole_3.2mm_M3_DIN965_Pad_TopBottom
- removed J1: 0430450606, Library:0430450606
- removed the J4 at (146.2, 28.8)
- removed the J4 at (181.0, 28.8)
- removed the R56 at (188.7, 44.7)
- removed the R56 at (154.0, 44.7)
- removed the R57 at (188.7, 41.6)
- removed the R57 at (154.0, 41.6)
- removed the R58 at (175.5, 43.8)
- removed the R58 at (140.8, 43.8)
- removed the R59 at (188.7, 38.5)
- removed the R59 at (154.0, 38.5)
- removed the R60 at (154.0, 43.1)
- removed the R60 at (188.7, 43.1)
- removed the R61 at (174.0, 43.8)
- removed the R61 at (139.2, 43.8)
- removed the R62 at (154.0, 36.9)
- removed the R62 at (188.7, 36.9)
- removed the R63 at (154.0, 40.0)
- removed the R63 at (188.7, 40.0)
- removed the U7 at (146.2, 39.6)
- removed the U7 at (181.0, 39.6)
- added C61: 220uF, Capacitor_SMD:CP_Elec_8x10, F.Cu at (131.2, 25.2)
- added C61: 220uF, Capacitor_SMD:CP_Elec_8x10, F.Cu at (164.6, 25.2)
- added C62: 100nF, Capacitor_SMD:C_0603_1608Metric, F.Cu at (138.5, 25.0)
- added C62: 100nF, Capacitor_SMD:C_0603_1608Metric, F.Cu at (171.9, 25.0)
- added C63: 100nF, Capacitor_SMD:C_0603_1608Metric, F.Cu at (138.0, 27.5)
- added C63: 100nF, Capacitor_SMD:C_0603_1608Metric, F.Cu at (171.4, 27.5)
- added C64: 22nF, Capacitor_SMD:C_0603_1608Metric, F.Cu at (171.4, 29.1)
- added C64: 22nF, Capacitor_SMD:C_0603_1608Metric, F.Cu at (138.0, 29.1)
- added C65: 100nF, Capacitor_SMD:C_0603_1608Metric, F.Cu at (185.3, 34.0)
- added C65: 100nF, Capacitor_SMD:C_0603_1608Metric, F.Cu at (151.9, 33.9)
- added J4: B2B-XH-AM, Library:43650-02YY_242526, F.Cu at (177.6, 16.4)
- added J4: B2B-XH-AM, Library:43650-02YY_242526, F.Cu at (144.2, 16.4)
- added R56: 10k, Resistor_SMD:R_0603_1608Metric, F.Cu at (151.9, 32.4)
- added R56: 10k, Resistor_SMD:R_0603_1608Metric, F.Cu at (185.3, 32.4)
- added R57: 1k, Resistor_SMD:R_0603_1608Metric, F.Cu at (185.3, 29.3)
- added R57: 1k, Resistor_SMD:R_0603_1608Metric, F.Cu at (151.9, 29.2)
- added R58: 0, Resistor_SMD:R_0603_1608Metric, F.Cu at (138.7, 31.5)
- added R58: 0, Resistor_SMD:R_0603_1608Metric, F.Cu at (172.1, 31.5)
- added R59: 0, Resistor_SMD:R_0603_1608Metric, F.Cu at (151.9, 26.1)
- added R59: 0, Resistor_SMD:R_0603_1608Metric, F.Cu at (185.3, 26.2)
- added R60: 11k, Resistor_SMD:R_0603_1608Metric, F.Cu at (185.3, 30.8)
- added R60: 11k, Resistor_SMD:R_0603_1608Metric, F.Cu at (151.9, 30.8)
- added R61: 0, Resistor_SMD:R_0603_1608Metric, F.Cu at (137.2, 31.5)
- added R61: 0, Resistor_SMD:R_0603_1608Metric, F.Cu at (170.6, 31.5)
- added R62: 0, Resistor_SMD:R_0603_1608Metric, F.Cu at (185.3, 24.6)
- added R62: 0, Resistor_SMD:R_0603_1608Metric, F.Cu at (151.9, 24.6)
- added R63: 6.8k, Resistor_SMD:R_0603_1608Metric, F.Cu at (151.9, 27.7)
- added R63: 6.8k, Resistor_SMD:R_0603_1608Metric, F.Cu at (185.3, 27.7)
- added U7: DRV8876PWPR, Library:SOP65P640X120-17N, F.Cu at (144.2, 27.3)
- added U7: DRV8876PWPR, Library:SOP65P640X120-17N, F.Cu at (177.6, 27.3)
- moved C61 12.4 mm to (98.0, 25.2)
- moved C62 12.4 mm to (105.3, 25.0)
- moved C65 12.4 mm to (118.7, 33.9)
- moved R56 12.4 mm to (118.7, 32.4)
- moved R59 12.4 mm to (118.7, 26.1)
- moved R60 12.4 mm to (118.7, 30.8)
- moved R62 12.4 mm to (118.7, 24.6)
- moved C63 12.4 mm to (104.8, 27.5)
- moved C64 12.4 mm to (104.8, 29.1)
- moved J4 12.4 mm to (111.0, 16.4)
- moved R57 12.4 mm to (118.7, 29.2)
- moved R58 12.4 mm to (105.5, 31.5)
- moved R61 12.4 mm to (104.0, 31.5)
- moved R63 12.4 mm to (118.7, 27.7)
- moved U7 12.4 mm to (111.0, 27.3)
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Routing:
- removed copper zone on In2.Cu, net +12V
- removed copper zone on In1.Cu, net GND
Other:
- board size 120 x 130 mm -> 116 x 133.1 mm

Commit message: m
Parts:
- removed the C127 at (142.6, 220.3)
- removed the C127 at (112.5, 220.3)
- removed the C128 at (112.4, 222.3)
- removed the C128 at (142.6, 222.2)
- removed the C129 at (114.9, 237.1)
- removed the C129 at (145.0, 237.0)
- removed the C130 at (146.2, 226.6)
- removed the C130 at (116.0, 226.6)
- removed the C131 at (115.9, 216.8)
- removed the C131 at (146.1, 216.7)
- removed the C132 at (115.9, 218.3)
- removed the C132 at (146.1, 218.3)
- removed the C25 at (105.6, 49.0)
- removed the C25 at (175.1, 69.8)
- removed the C26 at (168.3, 63.6)
- removed the C26 at (112.4, 55.3)
- removed the C27 at (173.6, 66.6)
- removed the C27 at (107.1, 52.3)
- removed the C28 at (182.9, 49.1)
- removed the C28 at (97.8, 69.7)
- removed the C29 at (182.9, 68.1)
- removed the C29 at (97.8, 50.7)
- removed the C30 at (191.1, 47.7)
- removed the C30 at (89.6, 71.2)
- removed the C31 at (191.1, 69.6)
- removed the C31 at (89.6, 49.2)
- removed the C32 at (110.5, 67.4)
- removed the C32 at (170.2, 51.4)
- removed the C33 at (170.0, 63.6)
- removed the C33 at (110.7, 55.3)
- removed the C34 at (114.2, 62.9)
- removed the C34 at (166.5, 56.0)
- removed the C35 at (166.4, 54.2)
- removed the C35 at (114.3, 64.7)
- removed the C36 at (170.4, 53.6)
- removed the C36 at (110.3, 65.2)
- removed the C37 at (179.7, 61.1)
- removed the C37 at (101.0, 57.7)
- removed the C38 at (172.2, 62.8)
- removed the C38 at (108.4, 56.0)
- removed the C39 at (101.0, 62.5)
- removed the C39 at (179.7, 56.3)
- removed the C40 at (174.3, 51.9)
- removed the C40 at (106.4, 67.0)
- removed the C41 at (105.5, 65.0)
- removed the C41 at (175.1, 53.9)
- removed the C42 at (105.5, 55.3)
- removed the C42 at (175.1, 63.5)
- removed the C61 at (131.2, 25.2)
- removed the C61 at (98.0, 25.2)
- removed the C61 at (164.6, 25.2)
- removed the C62 at (105.3, 25.0)
- removed the C62 at (138.5, 25.0)
- removed the C62 at (171.9, 25.0)
- removed the C63 at (104.8, 27.5)
- removed the C63 at (138.0, 27.5)
- removed the C63 at (171.4, 27.5)
- removed the C64 at (171.4, 29.1)
- removed the C64 at (138.0, 29.1)
- removed the C64 at (104.8, 29.1)
- removed the C65 at (118.7, 33.9)
- removed the C65 at (185.3, 34.0)
- removed the C65 at (151.9, 33.9)
- removed the D4 at (162.5, 61.0)
- removed the D4 at (118.2, 57.9)
- removed the D7 at (152.4, 222.6)
- removed the D7 at (122.2, 222.6)
- removed the D9 at (147.6, 232.4)
- removed the D9 at (117.5, 232.5)
- removed IC1: TRS3122ERGER, Library:QFN50P400X400X100-25N-D
- removed the J2 at (93.8, 60.2)
- removed the J2 at (186.9, 58.6)
- removed the J21 at (103.1, 239.5)
- removed the J21 at (133.2, 239.4)
- removed the J4 at (177.6, 16.4)
- removed the J4 at (144.2, 16.4)
- removed the J4 at (111.0, 16.4)
- removed the Q3 at (121.3, 219.8)
- removed the Q3 at (151.5, 219.7)
- removed the R108 at (118.3, 219.2)
- removed the R108 at (148.4, 219.2)
- removed the R109 at (148.4, 222.3)
- removed the R109 at (118.3, 222.3)
- removed the R110 at (149.2, 216.8)
- removed the R110 at (119.0, 216.8)
- removed the R111 at (119.8, 222.3)
- removed the R111 at (150.0, 222.3)
- removed the R112 at (141.3, 221.2)
- removed the R112 at (111.2, 221.3)
- removed the R113 at (140.5, 223.7)
- removed the R113 at (110.3, 223.7)
- removed the R114 at (110.3, 225.3)
- removed the R114 at (140.5, 225.2)
- removed the R115 at (153.4, 216.9)
- removed the R115 at (123.2, 217.0)
- removed the R116 at (154.1, 219.3)
- removed the R116 at (123.9, 219.3)
- removed the R22 at (105.5, 52.3)
- removed the R22 at (175.1, 66.6)
- removed the R23 at (112.7, 51.8)
- removed the R23 at (168.0, 67.1)
- removed the R24 at (171.1, 69.7)
- removed the R24 at (109.6, 49.1)
- removed the R25 at (165.8, 51.6)
- removed the R25 at (114.9, 67.2)
- removed the R26 at (162.4, 57.5)
- removed the R26 at (118.2, 61.3)
- removed the R27 at (162.4, 59.3)
- removed the R27 at (118.2, 59.6)
- removed the R28 at (162.4, 62.7)
- removed the R28 at (118.2, 56.2)
- removed the R29 at (113.4, 67.2)
- removed the R29 at (167.3, 51.6)
- removed the R30 at (165.6, 57.5)
- removed the R30 at (115.1, 61.3)
- removed the R31 at (115.1, 59.6)
- removed the R31 at (165.6, 59.3)
- removed the R32 at (109.6, 52.3)
- removed the R32 at (171.1, 66.5)
- removed the R33 at (115.1, 56.2)
- removed the R33 at (165.6, 62.7)
- removed the R34 at (115.1, 57.9)
- removed the R34 at (165.6, 61.0)
- removed the R35 at (177.5, 53.7)
- removed the R35 at (103.2, 65.2)
- removed the R36 at (177.5, 63.7)
- removed the R36 at (103.2, 55.1)
- removed the R37 at (172.5, 50.8)
- removed the R37 at (108.2, 68.1)
- removed the R38 at (171.1, 68.1)
- removed the R38 at (109.6, 50.7)
- removed the R56 at (151.9, 32.4)
- removed the R56 at (185.3, 32.4)
- removed the R56 at (118.7, 32.4)
- removed the R57 at (118.7, 29.2)
- removed the R57 at (185.3, 29.3)
- removed the R57 at (151.9, 29.2)
- removed the R58 at (138.7, 31.5)
- removed the R58 at (172.1, 31.5)
- removed the R58 at (105.5, 31.5)
- removed the R59 at (118.7, 26.1)
- removed the R59 at (151.9, 26.1)
- removed the R59 at (185.3, 26.2)
- removed the R60 at (185.3, 30.8)
- removed the R60 at (151.9, 30.8)
- removed the R60 at (118.7, 30.8)
- removed the R61 at (104.0, 31.5)
- removed the R61 at (137.2, 31.5)
- removed the R61 at (170.6, 31.5)
- removed the R62 at (185.3, 24.6)
- removed the R62 at (118.7, 24.6)
- removed the R62 at (151.9, 24.6)
- removed the R63 at (118.7, 27.7)
- removed the R63 at (151.9, 27.7)
- removed the R63 at (185.3, 27.7)
- removed R93: 22, Resistor_SMD:R_0603_1608Metric
- removed REF** (x2): TSSOP-16_4.4x5mm_P0.65mm, Package_SO:TSSOP-16_4.4x5mm_P0.65mm
- removed the U20 at (145.4, 221.3)
- removed the U20 at (115.2, 221.4)
- removed the U5 at (170.9, 58.7)
- removed the U5 at (109.8, 60.2)
- removed the U7 at (111.0, 27.3)
- removed the U7 at (144.2, 27.3)
- removed the U7 at (177.6, 27.3)
- added C106: 220uF, Capacitor_SMD:CP_Elec_8x10, F.Cu at (241.3, 47.5)
- added C123: 100nF, Capacitor_SMD:C_0603_1608Metric, F.Cu at (184.8, -36.0)
- added C124: 100nF, Capacitor_SMD:C_0603_1608Metric, F.Cu at (184.8, -33.5)
- added C125: 100nF, Capacitor_SMD:C_0603_1608Metric, F.Cu at (101.3, -37.0)
- added C126: 100nF, Capacitor_SMD:C_0603_1608Metric, F.Cu at (106.5, -37.0)
- added C127: 1uF, Capacitor_SMD:C_0603_1608Metric, F.Cu at (184.8, -26.0)
- added C128: 100nF, Capacitor_SMD:C_0603_1608Metric, F.Cu at (188.8, -51.1)
- added C129: 100nF, Capacitor_SMD:C_0603_1608Metric, F.Cu at (188.8, -48.6)
- added C130: 100nF, Capacitor_SMD:C_0603_1608Metric, F.Cu at (112.4, -37.0)
- added C131: 100nF, Capacitor_SMD:C_0603_1608Metric, F.Cu at (117.6, -37.0)
- added C132: 100nF, Capacitor_SMD:C_0603_1608Metric, F.Cu at (188.8, -41.0)
- added C139: 1uF, Capacitor_SMD:C_1206_3216Metric, F.Cu at (-52.8, 120.2)
- added C140: 100nF, Capacitor_SMD:C_0603_1608Metric, F.Cu at (-72.1, 111.7)
- added C141: 22nF, Capacitor_SMD:C_0603_1608Metric, F.Cu at (-72.1, 114.2)
- added C142: 3.3nF, Capacitor_SMD:C_0402_1005Metric, F.Cu at (-46.2, 115.9)
- added C143: 100nF, Capacitor_SMD:C_0603_1608Metric, F.Cu at (-72.1, 116.7)
- added C144: 100nF, Capacitor_SMD:C_0603_1608Metric, F.Cu at (-72.1, 119.2)
- added C145: 10uF, Capacitor_SMD:C_1210_3225Metric, F.Cu at (-20.4, 124.0)
- added C146: 47uF, Capacitor_SMD:CP_Elec_6.3x7.7, F.Cu at (-24.5, 114.5)
- added C147: 1uF, Capacitor_SMD:C_1206_3216Metric, F.Cu at (-20.4, 120.2)
- added C148: 100nF, Capacitor_SMD:C_0603_1608Metric, F.Cu at (-39.8, 111.7)
- added C149: 22nF, Capacitor_SMD:C_0603_1608Metric, F.Cu at (-39.8, 114.2)
- added C150: 3.3nF, Capacitor_SMD:C_0402_1005Metric, F.Cu at (-13.8, 115.9)
- added C151: 100nF, Capacitor_SMD:C_0603_1608Metric, F.Cu at (-39.8, 116.7)
- added C152: 100nF, Capacitor_SMD:C_0603_1608Metric, F.Cu at (-39.8, 119.2)
- added C153: 10uF, Capacitor_SMD:C_1210_3225Metric, F.Cu at (55.7, 100.6)
- added C154: 47uF, Capacitor_SMD:CP_Elec_6.3x7.7, F.Cu at (46.2, 104.7)
- added C155: 1uF, Capacitor_SMD:C_1206_3216Metric, F.Cu at (51.9, 100.6)
- added C156: 100nF, Capacitor_SMD:C_0603_1608Metric, F.Cu at (43.3, 119.9)
- added C157: 22nF, Capacitor_SMD:C_0603_1608Metric, F.Cu at (45.9, 119.9)
- added C158: 3.3nF, Capacitor_SMD:C_0402_1005Metric, F.Cu at (47.5, 94.0)
- added C159: 100nF, Capacitor_SMD:C_0603_1608Metric, F.Cu at (48.4, 119.9)
- added C160: 100nF, Capacitor_SMD:C_0603_1608Metric, F.Cu at (50.9, 119.9)
- added C25: 22uF, Capacitor_Tantalum_SMD:CP_EIA-3528-21_Kemet-B, F.Cu at (221.2, 122.6)
- added C26: 4.7uF, Capacitor_SMD:C_0603_1608Metric, F.Cu at (206.5, 117.3)
- added C27: 100nF, Capacitor_SMD:C_0603_1608Metric, F.Cu at (206.5, 119.8)
- added C28: 4.7uF, Capacitor_SMD:C_0805_2012Metric, F.Cu at (285.0, 48.7)
- added C29: 4.7uF, Capacitor_SMD:C_0805_2012Metric, F.Cu at (285.0, 51.7)
- added C30: 100nF, Capacitor_SMD:C_0603_1608Metric, F.Cu at (309.1, 24.1)
- added C31: 100nF, Capacitor_SMD:C_0603_1608Metric, F.Cu at (309.1, 26.6)
- added C32: 100nF, Capacitor_SMD:C_0603_1608Metric, F.Cu at (309.1, 29.1)
- added C33: 100nF, Capacitor_SMD:C_0603_1608Metric, F.Cu at (309.1, 31.6)
- added C34: 100nF, Capacitor_SMD:C_0603_1608Metric, F.Cu at (309.1, 34.2)
- added C35: 100nF, Capacitor_SMD:C_0603_1608Metric, F.Cu at (309.1, 36.7)
- added C36: 100nF, Capacitor_SMD:C_0603_1608Metric, F.Cu at (309.1, 39.2)
- added C37: 100nF, Capacitor_SMD:C_0603_1608Metric, F.Cu at (309.1, 41.7)
- added C38: 100nF, Capacitor_SMD:C_0603_1608Metric, F.Cu at (309.1, 44.2)
- added C39: 100nF, Capacitor_SMD:C_0603_1608Metric, F.Cu at (313.1, 24.1)
- added C40: 100nF, Capacitor_SMD:C_0603_1608Metric, F.Cu at (313.1, 26.6)
- added C41: 1uF, Capacitor_SMD:C_0603_1608Metric, F.Cu at (313.1, 29.1)
- added C42: 100nF, Capacitor_SMD:C_0603_1608Metric, F.Cu at (313.1, 31.6)
- added C61: 100nF, Capacitor_SMD:C_0603_1608Metric, F.Cu at (149.3, 120.7)
- added C62: 100nF, Capacitor_SMD:C_0603_1608Metric, F.Cu at (130.8, 178.5)
- added C63: 100nF, Capacitor_SMD:C_0603_1608Metric, F.Cu at (130.8, 181.0)
- added C64: 1uF, Capacitor_SMD:C_1210_3225Metric, F.Cu at (206.0, 111.6)
- added C65: 100nF, Capacitor_SMD:C_0603_1608Metric, F.Cu at (205.1, 81.7)
- added C98: 100nF, Capacitor_SMD:C_0603_1608Metric, F.Cu at (313.7, 95.6)
- added D11: SP0502BAHT, Package_TO_SOT_SMD:SOT-23, F.Cu at (126.3, -36.5)
- added D12: SP0502BAHT, Package_TO_SOT_SMD:SOT-23, F.Cu at (137.3, -36.5)
- added D13: B330A-13-F, Diode_SMD:D_SMA, F.Cu at (-47.8, 94.5)
- added D14: SMAJ15A, Diode_SMD:D_SMA, F.Cu at (-47.8, 99.0)
- added D15: GREEN, LED_SMD:LED_0603_1608Metric, F.Cu at (-49.6, 116.2)
- added D16: SMAJ30CA, Diode_SMD:D_SMA, F.Cu at (-47.8, 103.6)
- added D17: SMAJ30CA, Diode_SMD:D_SMA, F.Cu at (-47.8, 108.1)
- added D18: B330A-13-F, Diode_SMD:D_SMA, F.Cu at (-15.5, 94.5)
- added D19: SMAJ15A, Diode_SMD:D_SMA, F.Cu at (-15.5, 99.0)
- added D20: GREEN, LED_SMD:LED_0603_1608Metric, F.Cu at (-17.3, 116.2)
- added D21: SMAJ30CA, Diode_SMD:D_SMA, F.Cu at (-15.5, 103.6)
- added D22: SMAJ30CA, Diode_SMD:D_SMA, F.Cu at (-15.5, 108.1)
- added D23: B330A-13-F, Diode_SMD:D_SMA, F.Cu at (26.1, 95.6)
- added D24: SMAJ15A, Diode_SMD:D_SMA, F.Cu at (30.7, 95.6)
- added D25: GREEN, LED_SMD:LED_0603_1608Metric, F.Cu at (47.8, 97.4)
- added D26: SMAJ30CA, Diode_SMD:D_SMA, F.Cu at (35.2, 95.6)
- added D27: SMAJ30CA, Diode_SMD:D_SMA, F.Cu at (39.8, 95.6)
- added D4: SMF5V0A, Diode_SMD:D_SMF, F.Cu at (64.3, 197.8)
- added D6: RED, LED_SMD:LED_0603_1608Metric, F.Cu at (210.8, 110.8)
- added D7: RED, LED_SMD:LED_0603_1608Metric, F.Cu at (306.4, 101.4)
- added D9: SP0502BAHT, Package_TO_SOT_SMD:SOT-23, F.Cu at (103.9, -36.4)
- added H1: MountingHole_Pad, MountingHole:MountingHole_3.2mm_M3_DIN965_Pad_TopBottom, F.Cu at (194.9, 119.6)
- added H2: MountingHole_Pad, MountingHole:MountingHole_3.2mm_M3_DIN965_Pad_TopBottom, F.Cu at (194.9, 126.8)
- added H3: MountingHole_Pad, MountingHole:MountingHole_3.2mm_M3_DIN965_Pad_TopBottom, F.Cu at (74.6, 151.2)
- added H4: MountingHole_Pad, MountingHole:MountingHole_3.2mm_M3_DIN965_Pad_TopBottom, F.Cu at (174.8, 151.2)
- added J1: 172447-0006, Library:172447-YY06, B.Cu at (97.3, 154.9)
- added J16: BM06B-GHS-TBT, Library:BM06BGHSTBTLFSN, F.Cu at (189.8, -10.2)
- added J19: BM06B-GHS-TBT, Library:BM06BGHSTBTLFSN, F.Cu at (152.9, -30.8)
- added J2: Conn_01x10, Library:BM10BGHSTBT, F.Cu at (316.6, 50.1)
- added J21: 43045-0810, Connector_Molex:Molex_Micro-Fit_3.0_43045-0810_2x04-1MP_P3.00mm_Horizontal, F.Cu at (-30.7, 105.6)
- added J4: USB_B, Library:UJ2BV1TH, B.Cu at (152.4, 149.2)
- added L3: BLM21PG221SN1D, Inductor_SMD:L_0805_2012Metric, F.Cu at (150.1, 144.2)
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Connections:
- C10 pad 1: +12V -> Net-(U2-BOOT)
- C10 pad 2: GND -> Net-(U2-PH)
- C100 pad 1: GND -> +12V
- C100 pad 2: +3.3V -> GND
- C101 pad 1: GND -> +12V
- C101 pad 2: +3.3V -> GND
- C102 pad 1: GND -> Net-(U12-VCP)
- C102 pad 2: +3.3V -> +12V
- C103 pad 1: GND -> Net-(U12-CPL)
- C103 pad 2: +3.3V -> Net-(U12-CPH)
- C104 pad 2: +3.3V -> /DC_DRIVERS/J_FAULT
- C105 pad 1: GND -> +12V
- C105 pad 2: +3.3V -> GND
- C107 pad 1: GND -> +12V
- C107 pad 2: VDDA -> GND
- C108 pad 1: GND -> +12V
- C108 pad 2: VDDA -> GND
- C109 pad 1: GND -> Net-(U13-VCP)
- C109 pad 2: +3.3V -> +12V
- C11 pad 1: +12V -> +5V
- C110 pad 1: GND -> Net-(U13-CPL)
- C110 pad 2: EXP_GPIO_6 -> Net-(U13-CPH)
- C111 pad 2: EXP_GPIO_5 -> /DC_DRIVERS/Z_FAULT
- C112 pad 1: GND -> +12V
- C112 pad 2: EXP_GPIO_4 -> GND
- C113 pad 1: GND -> +12V
- C113 pad 2: EXP_GPIO_3 -> GND
- C114 pad 1: GND -> Net-(U14-VCP)
- C114 pad 2: EXP_GPIO_2 -> +12V
- C115 pad 1: GND -> Net-(U14-CPL)
- C115 pad 2: EXP_GPIO_1 -> Net-(U14-CPH)
- C116 pad 2: MCU_RESET -> /DC_DRIVERS/F_FAULT
- C117 pad 2: Net-(U18-PH1) -> +3.3V
- C118 pad 2: Net-(U18-PH0) -> +5VSB
- C119 pad 2: Net-(U18-VCAP_1) -> Net-(J12-Pin_2)
- C12 pad 1: +12V -> +5V
- C120 pad 2: Net-(U18-VCAP_2) -> Net-(J12-Pin_1)
- C121 pad 1: Net-(U1-EN) -> GND
- C121 pad 2: GND -> +3.3V
- C122 pad 2: USB_VBUS -> +3.3V
- C13 pad 1: Net-(U2-SS) -> +12V
- C133 pad 2: Net-(U21-IN) -> Net-(J17-Pin_2)
- C134 pad 2: Net-(U21-IN) -> Net-(J17-Pin_1)
- C135 pad 2: Net-(U21-ITIMER_1) -> +3.3V
- C136 pad 2: Net-(U21-DVDT_1) -> Net-(J18-Pin_1)
- C137 pad 2: Net-(D10-A1) -> /ACC1/ACC1_+12V
- C138 pad 1: Net-(D10-A1) -> /ACC1/ACC1_+12V
- C14 pad 1: Net-(U2-COMP) -> +12V
- C15 pad 1: Net-(C15-Pad1) -> +12V
- C16 pad 1: +5V -> Net-(U2-SS)
- C17 pad 1: +5V -> Net-(U2-COMP)
- C18 pad 1: Net-(U3-VI) -> Net-(C18-Pad1)
- C18 pad 2: /MCU/12V_PRES -> GND
- C19 pad 1: Net-(U3-VI) -> +5V
- C20 pad 1: Net-(U3-VI) -> +5V
- C21 pad 1: +3.3V -> Net-(U3-VI)
- C21 pad 2: GND -> Net-(U4-ST)
- C22 pad 1: +3.3V -> Net-(U3-VI)
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Routing:
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- added copper zone on In2.Cu, net +12V
- added copper zone on B.Cu, net GND
- added copper zone on In1.Cu, net GND
- added copper zone on B.Cu, net GNDD
- added copper zone on F.Cu, net GNDD
- added copper zone on In1.Cu, net GNDD
- added copper zone on In2.Cu, net GNDD
- removed copper zone on F.Cu, net +12V
- removed copper zone on F.Cu, net +5V
- removed copper zone on F.Cu, net +5VSB
- removed copper zone on F.Cu, net /POWER_INPUT/VIN
- removed copper zone on B.Cu, net Net-(J2-Pin_1)
- removed copper zone on F.Cu, net Net-(J2-Pin_1)
- removed copper zone on B.Cu, net Net-(J2-Pin_2)
- removed copper zone on F.Cu, net Net-(J2-Pin_2)
- removed copper zone on B.Cu, net Net-(J2-Pin_3)
- removed copper zone on F.Cu, net Net-(J2-Pin_3)
- removed copper zone on B.Cu, net Net-(J2-Pin_4)
- removed copper zone on F.Cu, net Net-(J2-Pin_4)
- removed copper zone on F.Cu, net Net-(J4-Pin_1)
- removed copper zone on F.Cu, net Net-(J4-Pin_2)
- removed copper zone on B.Cu, net Net-(U1-DRAIN_2)
- removed copper zone on F.Cu, net Net-(U1-DRAIN_2)
- removed copper zone on In1.Cu, net Net-(U1-DRAIN_2)
- removed copper zone on F.Cu, net Net-(U3-VI)
- removed copper zone on F.Cu, net Net-(U5-BRA)
- removed copper zone on F.Cu, net Net-(U5-BRB)

Commit message: init
Parts:
- added R203: 100, Resistor_SMD:R_0603_1608Metric, F.Cu at (-98.7, 71.5)
- added R204: 100, Resistor_SMD:R_0603_1608Metric, F.Cu at (-98.7, 74.0)
- added R205: 100, Resistor_SMD:R_0603_1608Metric, F.Cu at (-98.7, 76.5)
- added R206: 10k, Resistor_SMD:R_0603_1608Metric, F.Cu at (-98.7, 79.1)
- added R207: 100, Resistor_SMD:R_0603_1608Metric, F.Cu at (-98.7, 109.3)
- added R208: 100, Resistor_SMD:R_0603_1608Metric, F.Cu at (-98.7, 111.8)
- added R209: 100, Resistor_SMD:R_0603_1608Metric, F.Cu at (-98.7, 114.3)
- added R210: 10k, Resistor_SMD:R_0603_1608Metric, F.Cu at (-98.7, 116.8)
- added R211: 100, Resistor_SMD:R_0603_1608Metric, F.Cu at (54.5, 95.3)
- added R212: 100, Resistor_SMD:R_0603_1608Metric, F.Cu at (54.5, 92.1)
- added R213: 100, Resistor_SMD:R_0603_1608Metric, F.Cu at (54.6, 90.5)
- added R214: 10k, Resistor_SMD:R_0603_1608Metric, F.Cu at (48.8, 88.8)
- added R215: 120, Resistor_SMD:R_0603_1608Metric, F.Cu at (-98.7, 81.6)
- added R216: 120, Resistor_SMD:R_0603_1608Metric, F.Cu at (-98.7, 119.4)
- added R217: 120, Resistor_SMD:R_0603_1608Metric, F.Cu at (46.4, 92.7)
- moved U17 90.2 mm to (132.5, -73.6), turned to -90 degrees
- moved U16 90.0 mm to (128.8, -73.6), turned to 90 degrees
- moved U19 86.8 mm to (148.2, -74.0), turned to -90 degrees
- moved U18 85.4 mm to (144.5, -73.9), turned to 90 degrees
- moved C150 81.8 mm to (-95.2, 123.7)
- moved J14 73.3 mm to (130.6, -62.8)
- moved R125 73.3 mm to (128.7, -69.0), turned to 90 degrees
- moved U22 72.6 mm to (-87.4, 119.0)
- moved D20 71.2 mm to (-88.1, 123.0)
- moved R127 71.0 mm to (134.5, -69.0), turned to 90 degrees
- moved C124 70.9 mm to (126.2, -73.6), turned to 90 degrees
- moved C148 70.9 mm to (-110.7, 109.3)
- moved C149 70.9 mm to (-110.7, 111.8)
- moved C151 70.9 mm to (-110.7, 114.3)
- moved C152 70.9 mm to (-110.7, 116.8)
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Connections:
- net /ACC1/ACC1_DIR renamed Net-(U21-DE)
- net /ACC1/ACC1_RX renamed Net-(U21-R)
- net /ACC2/ACC2_DIR renamed Net-(U23-DE)
- net /ACC2/ACC2_RX renamed Net-(U23-R)
- net /ACC3/ACC3_DIR renamed Net-(U25-DE)
- net /ACC3/ACC3_RX renamed Net-(U25-R)
- R129 pad 2: Net-(U17-1Y) -> Net-(U17-2Y)
- R130 pad 2: Net-(U17-2Y) -> Net-(U17-1Y)
- R142 pad 2: Net-(U19-1Y) -> Net-(U19-2Y)
- R143 pad 2: Net-(U19-2Y) -> Net-(U19-1Y)
- U17 pad 1: /LIM_ENC/XY_ENC_CLK -> /LIM_ENC/X_ENC_CS
- U17 pad 3: /LIM_ENC/X_ENC_CS -> /LIM_ENC/XY_ENC_CLK
- U19 pad 1: /LIM_ENC/XY_ENC_CLK -> /LIM_ENC/Y_ENC_CS
- U19 pad 3: /LIM_ENC/Y_ENC_CS -> /LIM_ENC/XY_ENC_CLK
- U21 pad 5: /ACC1/ACC1_TX -> Net-(U21-D)
- U21 pad 7: +3.3V -> Net-(U21-SLR)
- U23 pad 5: /ACC2/ACC2_TX -> Net-(U23-D)
- U23 pad 7: +3.3V -> Net-(U23-SLR)
- U25 pad 5: /ACC3/ACC3_TX -> Net-(U25-D)
- U25 pad 7: +3.3V -> Net-(U25-SLR)
- U25 pad 8: Net-(D26-A2) -> Net-(D27-A2)
- U25 pad 9: Net-(D27-A2) -> Net-(D26-A2)
Routing:
- net /LIM_ENC/Y_ENC_INDEX_INPUT: track 0.00 -> 15.9 mm, vias 0 -> 2
- net /LIM_ENC/X_ENC_INDEX_INPUT: track 0.00 -> 10.0 mm, vias 0 -> 2
- net /LIM_ENC/Y_ENC_DO_INPUT: track 0.00 -> 8.39 mm
- net /LIM_ENC/X_ENC_DO_INPUT: track 0.00 -> 8.39 mm
- net GND: track 28.2 -> 36.2 mm, vias 25 -> 33
- net +3.3V: track 16.9 -> 24.9 mm, vias 4 -> 12
- net /LIM_ENC/Y_ENC_CS_OUTPUT: track 0.00 -> 5.83 mm
- net /LIM_ENC/X_ENC_CS_OUTPUT: track 0.00 -> 5.83 mm
- net /LIM_ENC/Y_ENC_CLK_OUTPUT: track 0.00 -> 3.46 mm
- net /LIM_ENC/X_ENC_CLK_OUTPUT: track 0.00 -> 3.46 mm
- net Net-(U19-1Y): track 0.00 -> 3.08 mm
- net Net-(U17-1Y): track 0.00 -> 3.08 mm
- net Net-(U19-2Y): track 0.00 -> 2.98 mm
- net Net-(U17-2Y): track 0.00 -> 2.98 mm
