File: hardware/Ziess-Microsope-Controller_Main_board/Ziess-Microsope-Controller_Main_board.kicad_pcb (KiCad board)
At the start: 4 copper layers, 116 x 133.1 mm, 466 parts, among them J1 172447-0006, J10 43650-0224, J11 BM04B-GHS-TBT, J12 BM03B-GHS-TBT, J13 BM03B-GHS-TBT, J14 BM06B-GHS-TBT, J15 BM03B-GHS-TBT, J16 BM06B-GHS-TBT, J17 BM03B-GHS-TBT, J18 BM03B-GHS-TBT, J19 BM06B-GHS-TBT, J2 Conn_01x10, J20 43045-0810, J21 43045-0810, J22 43045-0810, J3 TC2030, J4 USB_B, J5 U.FL-R-SMT-1_10, J6 43045-0418, J7 43045-0418, J8 43650-0224, J9 43650-0224, Q1 BSS84, Q2 2N7002, Q3 2N7002, Q4 2N7002, Q5 2N7002, SW1 RESET, SW2 SW_Push, SW3 CJS1201A, U1 TPS24751RUVR, U10 TMC2209-LA, U11 TMC2209-LA, U12 DRV8876PWPR, U13 DRV8876PWPR, U14 DRV8876PWPR, U15 SN74LVC2G17DBV, U16 SN74LVC2G17DBV, U17 SN74LVC2G17DBV, U18 SN74LVC2G17DBV, U19 SN74LVC2G17DBV, U2 TPS54336ADDA, U20 TPS259472LRPWR, U21 THVD2450VDRCR, U22 TPS259472LRPWR, U23 THVD2450VDRCR, U24 TPS259472LRPWR, U25 THVD2450VDRCR, U3 AMS1117-3.3, U4 TPS2116DRL, U5 STM32F765ZGTx, U6 ADUM3160, U7 USBLC6-2SC6, U8 74AHCT1G125, U9 74LVC1G17, Y1 Crystal_Small

Commit message: m
Parts:
- removed C137, C145: 10uF, Capacitor_SMD:C_1210_3225Metric
- removed C138, C146: 47uF, Capacitor_SMD:CP_Elec_6.3x7.7
- removed C139, C147: 1uF, Capacitor_SMD:C_1206_3216Metric
- removed C140, C143, C144, C148, C151, C152: 100nF, Capacitor_SMD:C_0603_1608Metric
- removed C141, C149: 22nF, Capacitor_SMD:C_0603_1608Metric
- removed C142, C150: 3.3nF, Capacitor_SMD:C_0402_1005Metric
- removed D13, D18: B330A-13-F, Diode_SMD:D_SMA
- removed D14, D19: SMAJ15A, Diode_SMD:D_SMA
- removed D15, D20: GREEN, LED_SMD:LED_0603_1608Metric
- removed D16, D17, D21, D22: SMAJ30CA, Diode_SMD:D_SMA
- removed J20, J21: 43045-0810, Connector_Molex:Molex_Micro-Fit_3.0_43045-0810_2x04-1MP_P3.00mm_Horizontal
- removed Q3, Q4: 2N7002, Package_TO_SOT_SMD:SOT-23
- removed R151, R168: 470k, Resistor_SMD:R_0603_1608Metric
- removed R152, R169: 82k, Resistor_SMD:R_0603_1608Metric
- removed R153, R156, R158, R159, R160, R162, R163, R164, R165, R166, R167, R170, R173, R175, R176, R177, R179, R180, R181, R182, R183, R184, R206, R210: 10k, Resistor_SMD:R_0603_1608Metric
- removed R154, R171, R203, R204, R205, R207, R208, R209: 100, Resistor_SMD:R_0603_1608Metric
- removed R155, R172: 1.5k, Resistor_SMD:R_0603_1608Metric
- removed R157, R174: 390k, Resistor_SMD:R_0603_1608Metric
- removed R161, R178: 1.65k, Resistor_SMD:R_0603_1608Metric
- removed R215, R216: 120, Resistor_SMD:R_0603_1608Metric
- removed U20, U22: TPS259472LRPWR, Library:TPS259472LRPWR
- removed U21, U23: THVD2450VDRCR, Library:THVD2450VDRCR
- added JP1: SolderJumper_3_Bridged12, Jumper:SolderJumper-3_P1.3mm_Bridged123_Pad1.0x1.5mm, F.Cu at (98.5, 44.9)
- added TP1: TestPoint, TestPoint:TestPoint_Pad_D1.0mm, F.Cu at (91.5, 36.6)
- added TP1: TestPoint, TestPoint:TestPoint_Pad_D1.0mm, F.Cu at (91.5, 42.1)
- added TP1: TestPoint, TestPoint:TestPoint_Pad_D1.0mm, F.Cu at (101.1, 34.5)
- added TP2: TestPoint, TestPoint:TestPoint_Pad_D1.0mm, F.Cu at (96.2, 47.4)
- added TP3: TestPoint, TestPoint:TestPoint_Pad_D1.0mm, F.Cu at (72.0, 57.0)
- added TP4: TestPoint, TestPoint:TestPoint_Pad_D1.0mm, F.Cu at (72.0, 60.0)
- C158: footprint Capacitor_SMD:C_0402_1005Metric -> Capacitor_SMD:C_0603_1608Metric
- moved C83 160.4 mm to (158.3, 43.6)
- moved C84 160.4 mm to (158.3, 46.1)
- moved C85 160.4 mm to (172.5, 45.9)
- moved C86 160.4 mm to (172.5, 52.8)
- moved C89 160.4 mm to (158.3, 48.7)
- moved C90 160.4 mm to (158.3, 51.2)
- moved C91 160.4 mm to (158.3, 53.7)
- moved C95 160.4 mm to (153.3, 51.0)
- moved C98 160.4 mm to (158.3, 56.2)
- moved C99 160.4 mm to (158.3, 58.7)
- moved J7 160.4 mm to (164.4, 35.4)
- moved R79 160.4 mm to (162.3, 48.7)
- moved R86 160.4 mm to (166.3, 48.7)
- moved R90 160.4 mm to (148.1, 50.2)
- moved R91 160.4 mm to (148.1, 54.4)
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Connections:
- R214 pad 2: +3.3V -> Net-(JP1-C)
Routing:
- net /ACC3/ACC3_PRESENT: track 0.00 -> 19.2 mm
- net +3.3V: track 24.9 -> 35.6 mm, vias 12 -> 16
- net Net-(U24-EN/UVLO_1): track 0.00 -> 10.7 mm
- net Net-(J22-Pin_6): track 0.00 -> 10.7 mm
- net Net-(D26-A2): track 0.00 -> 9.70 mm
- net Net-(D27-A2): track 0.00 -> 9.48 mm
- net /ACC3/ACC3_IMON: track 0.00 -> 7.87 mm
- net /ACC3/ACC3_PWR_FLG: track 0.00 -> 6.95 mm
- net Net-(Q5-G): track 0.00 -> 6.10 mm, vias 0 -> 1
- net Net-(U24-PGTH/_~{FLT_1}): track 0.00 -> 5.60 mm
- net Net-(U25-DE): track 0.00 -> 5.46 mm
- net Net-(D25-A): track 0.00 -> 4.78 mm
- net Net-(J22-Pin_4): track 0.00 -> 4.67 mm
- net /ACC3/ACC3_TX: track 0.00 -> 4.37 mm
- net Net-(U25-R): track 0.00 -> 4.14 mm
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
Commit message: init
Parts:
- removed J13: BM03B-GHS-TBT, Library:BM03BGHSTBTLFSN
- added C137: 10uF, Capacitor_SMD:C_1210_3225Metric, F.Cu at (28.8, 19.8)
- added C138: 47uF, Capacitor_SMD:CP_Elec_6.3x7.7, F.Cu at (20.8, 21.8)
- added C139: 1uF, Capacitor_SMD:C_1206_3216Metric, F.Cu at (28.8, 23.6)
- added C140: 100nF, Capacitor_SMD:C_0603_1608Metric, F.Cu at (1.50, 19.0)
- added C141: 22nF, Capacitor_SMD:C_0603_1608Metric, F.Cu at (1.50, 21.5)
- added C142: 3.3nF, Capacitor_SMD:C_0402_1005Metric, F.Cu at (17.0, 33.4)
- added C143: 100nF, Capacitor_SMD:C_0603_1608Metric, F.Cu at (1.50, 24.0)
- added C144: 100nF, Capacitor_SMD:C_0603_1608Metric, F.Cu at (1.50, 26.5)
- added C145: 10uF, Capacitor_SMD:C_1210_3225Metric, F.Cu at (63.8, 19.8)
- added C146: 47uF, Capacitor_SMD:CP_Elec_6.3x7.7, F.Cu at (55.7, 21.8)
- added C147: 1uF, Capacitor_SMD:C_1206_3216Metric, F.Cu at (63.8, 23.6)
- added C148: 100nF, Capacitor_SMD:C_0603_1608Metric, F.Cu at (36.5, 19.0)
- added C149: 22nF, Capacitor_SMD:C_0603_1608Metric, F.Cu at (36.5, 21.5)
- added C150: 3.3nF, Capacitor_SMD:C_0402_1005Metric, F.Cu at (51.9, 33.4)
- added C151: 100nF, Capacitor_SMD:C_0603_1608Metric, F.Cu at (36.5, 24.0)
- added C152: 100nF, Capacitor_SMD:C_0603_1608Metric, F.Cu at (36.5, 26.5)
- added D13: B330A-13-F, Diode_SMD:D_SMA, F.Cu at (25.8, 1.77)
- added D14: SMAJ15A, Diode_SMD:D_SMA, F.Cu at (25.8, 6.33)
- added D15: GREEN, LED_SMD:LED_0603_1608Metric, F.Cu at (24.1, 32.7)
- added D16: SMAJ30CA, Diode_SMD:D_SMA, F.Cu at (25.8, 10.9)
- added D17: SMAJ30CA, Diode_SMD:D_SMA, F.Cu at (25.8, 15.4)
- added D18: B330A-13-F, Diode_SMD:D_SMA, F.Cu at (60.8, 1.77)
- added D19: SMAJ15A, Diode_SMD:D_SMA, F.Cu at (60.8, 6.33)
- added D20: GREEN, LED_SMD:LED_0603_1608Metric, F.Cu at (59.0, 32.7)
- added D21: SMAJ30CA, Diode_SMD:D_SMA, F.Cu at (60.8, 10.9)
- added D22: SMAJ30CA, Diode_SMD:D_SMA, F.Cu at (60.8, 15.4)
- added H1: MountingHole_Pad, MountingHole:MountingHole_3.2mm_M3_DIN965_Pad_TopBottom, F.Cu at (207.1, 199.7)
- added J20: 43045-0810, Connector_Molex:Molex_Micro-Fit_3.0_43045-0810_2x04-1MP_P3.00mm_Horizontal, F.Cu at (10.6, 12.9)
- added J21: 43045-0810, Connector_Molex:Molex_Micro-Fit_3.0_43045-0810_2x04-1MP_P3.00mm_Horizontal, F.Cu at (45.6, 12.9)
- added Q3: 2N7002, Package_TO_SOT_SMD:SOT-23, F.Cu at (30.0, 28.1)
- added Q4: 2N7002, Package_TO_SOT_SMD:SOT-23, F.Cu at (64.9, 28.1)
- added R151: 470k, Resistor_SMD:R_0603_1608Metric, F.Cu at (1.50, 29.0)
- added R152: 82k, Resistor_SMD:R_0603_1608Metric, F.Cu at (1.50, 31.5)
- added R153: 10k, Resistor_SMD:R_0603_1608Metric, F.Cu at (1.50, 34.0)
- added R154: 100, Resistor_SMD:R_0603_1608Metric, F.Cu at (5.51, 19.0)
- added R155: 1.5k, Resistor_SMD:R_0603_1608Metric, F.Cu at (5.51, 21.5)
- added R156: 10k, Resistor_SMD:R_0603_1608Metric, F.Cu at (5.51, 24.0)
- added R157: 390k, Resistor_SMD:R_0603_1608Metric, F.Cu at (5.51, 26.5)
- added R158: 10k, Resistor_SMD:R_0603_1608Metric, F.Cu at (5.51, 29.0)
- added R159: 10k, Resistor_SMD:R_0603_1608Metric, F.Cu at (5.51, 31.5)
- added R160: 10k, Resistor_SMD:R_0603_1608Metric, F.Cu at (5.51, 34.0)
- added R161: 1.65k, Resistor_SMD:R_0603_1608Metric, F.Cu at (9.53, 19.0)
- added R162: 10k, Resistor_SMD:R_0603_1608Metric, F.Cu at (9.53, 21.5)
- added R163: 10k, Resistor_SMD:R_0603_1608Metric, F.Cu at (9.53, 24.0)
- added R164: 10k, Resistor_SMD:R_0603_1608Metric, F.Cu at (9.53, 26.5)
- added R165: 10k, Resistor_SMD:R_0603_1608Metric, F.Cu at (9.53, 29.0)
- added R166: 10k, Resistor_SMD:R_0603_1608Metric, F.Cu at (9.53, 31.5)
- added R167: 10k, Resistor_SMD:R_0603_1608Metric, F.Cu at (9.53, 34.0)
- added R168: 470k, Resistor_SMD:R_0603_1608Metric, F.Cu at (36.5, 29.0)
- added R169: 82k, Resistor_SMD:R_0603_1608Metric, F.Cu at (36.5, 31.5)
- added R170: 10k, Resistor_SMD:R_0603_1608Metric, F.Cu at (36.5, 34.0)
- added R171: 100, Resistor_SMD:R_0603_1608Metric, F.Cu at (40.5, 19.0)
- added R172: 1.5k, Resistor_SMD:R_0603_1608Metric, F.Cu at (40.5, 21.5)
- added R173: 10k, Resistor_SMD:R_0603_1608Metric, F.Cu at (40.5, 24.0)
- added R174: 390k, Resistor_SMD:R_0603_1608Metric, F.Cu at (40.5, 26.5)
- added R175: 10k, Resistor_SMD:R_0603_1608Metric, F.Cu at (40.5, 29.0)
- added R176: 10k, Resistor_SMD:R_0603_1608Metric, F.Cu at (40.5, 31.5)
- added R177: 10k, Resistor_SMD:R_0603_1608Metric, F.Cu at (40.5, 34.0)
- added R178: 1.65k, Resistor_SMD:R_0603_1608Metric, F.Cu at (44.5, 19.0)
- added R179: 10k, Resistor_SMD:R_0603_1608Metric, F.Cu at (44.5, 21.5)
- added R180: 10k, Resistor_SMD:R_0603_1608Metric, F.Cu at (44.5, 24.0)
- added R181: 10k, Resistor_SMD:R_0603_1608Metric, F.Cu at (44.5, 26.5)
- added R182: 10k, Resistor_SMD:R_0603_1608Metric, F.Cu at (44.5, 29.0)
- added R183: 10k, Resistor_SMD:R_0603_1608Metric, F.Cu at (44.5, 31.5)
- added R184: 10k, Resistor_SMD:R_0603_1608Metric, F.Cu at (44.5, 34.0)
- added R203: 100, Resistor_SMD:R_0603_1608Metric, F.Cu at (13.5, 19.0)
- added R204: 100, Resistor_SMD:R_0603_1608Metric, F.Cu at (13.5, 21.5)
- added R205: 100, Resistor_SMD:R_0603_1608Metric, F.Cu at (13.5, 24.0)
- added R206: 10k, Resistor_SMD:R_0603_1608Metric, F.Cu at (13.5, 26.5)
- added R207: 100, Resistor_SMD:R_0603_1608Metric, F.Cu at (48.5, 19.0)
- added R208: 100, Resistor_SMD:R_0603_1608Metric, F.Cu at (48.5, 21.5)
- added R209: 100, Resistor_SMD:R_0603_1608Metric, F.Cu at (48.5, 24.0)
- added R210: 10k, Resistor_SMD:R_0603_1608Metric, F.Cu at (48.5, 26.5)
- added R215: 120, Resistor_SMD:R_0603_1608Metric, F.Cu at (13.5, 29.0)
- added R216: 120, Resistor_SMD:R_0603_1608Metric, F.Cu at (48.5, 29.0)
- added TP5: TestPoint, TestPoint:TestPoint_Pad_D1.0mm, F.Cu at (36.0, 38.8)
- added U20: TPS259472LRPWR, Library:TPS259472LRPWR, F.Cu at (24.8, 28.6)
- added U21: THVD2450VDRCR, Library:THVD2450VDRCR, F.Cu at (18.8, 29.1)
- added U22: TPS259472LRPWR, Library:TPS259472LRPWR, F.Cu at (59.7, 28.6)
- added U23: THVD2450VDRCR, Library:THVD2450VDRCR, F.Cu at (53.7, 29.1)
- C117, C118, C119, C120, C121, C122, C123, C124, C125, C126, C127, C128, C129, C130, C131, C132, C133, C134, C135, C136: footprint Capacitor_SMD:C_0603_1608Metric -> Capacitor_SMD:C_0402_1005Metric
- J12: value BM03B-GHS-TBT -> BM06B-GHS-TBT; footprint Library:BM03BGHSTBTLFSN -> Library:BM06BGHSTBTLFSN
- R116, R117, R118, R119, R120, R121, R122, R123, R124, R125, R126, R127, R128, R129, R130, R131, R132, R133, R134, R135, R136, R137, R138, R139, R140, R141, R142, R143, R144, R145, R146, R147, R148, R149, R150: footprint Resistor_SMD:R_0603_1608Metric -> Resistor_SMD:R_0402_1005Metric
- moved R120 230.3 mm to (168.2, 129.5), turned to -90 degrees
- moved R119 229.9 mm to (170.5, 131.5), turned to 180 degrees
- moved C120 229.3 mm to (170.5, 129.9), turned to 0 degrees
- moved R121 228.2 mm to (168.2, 125.1), turned to 90 degrees
- moved D8 227.6 mm to (170.0, 127.3), turned to 180 degrees
- moved C119 227.5 mm to (170.5, 124.7), turned to 0 degrees
- moved R118 227.0 mm to (170.5, 123.2), turned to 180 degrees
- moved J12 222.3 mm to (176.7, 122.4), turned to 90 degrees
- moved R124 215.9 mm to (168.2, 119.7), turned to -90 degrees
- moved R123 215.5 mm to (170.5, 121.6), turned to 180 degrees
- moved C126 214.9 mm to (170.5, 120.1), turned to 0 degrees
- moved R128 213.7 mm to (168.2, 115.3), turned to 90 degrees
- moved D9 213.1 mm to (170.0, 117.5), turned to 180 degrees
- moved C125 212.9 mm to (170.5, 114.9), turned to 0 degrees
- moved R122 212.4 mm to (170.5, 113.3), turned to 180 degrees
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Connections:
- C119 pad 2: Net-(J12-Pin_2) -> Net-(J12-Pin_5)
- C120 pad 2: Net-(J12-Pin_1) -> Net-(J12-Pin_6)
- C125 pad 2: Net-(J13-Pin_2) -> Net-(J12-Pin_2)
- C126 pad 2: Net-(J13-Pin_1) -> Net-(J12-Pin_3)
- D8 pad 1: Net-(J12-Pin_1) -> Net-(J12-Pin_6)
- D8 pad 2: Net-(J12-Pin_2) -> Net-(J12-Pin_5)
- D9 pad 1: Net-(J13-Pin_1) -> Net-(J12-Pin_3)
- D9 pad 2: Net-(J13-Pin_2) -> Net-(J12-Pin_2)
- J12 pad 1: Net-(J12-Pin_1) -> GND
- J12 pad 3: GND -> Net-(J12-Pin_3)
- J12 pad 4: (no net) -> GND
- J12 pad 5: (no net) -> Net-(J12-Pin_5)
- R118 pad 1: Net-(J12-Pin_2) -> Net-(J12-Pin_5)
- R119 pad 1: Net-(J12-Pin_1) -> Net-(J12-Pin_6)
- R120 pad 1: Net-(J12-Pin_1) -> Net-(J12-Pin_6)
- R121 pad 1: Net-(J12-Pin_2) -> Net-(J12-Pin_5)
- R122 pad 1: Net-(J13-Pin_2) -> Net-(J12-Pin_2)
- R123 pad 1: Net-(J13-Pin_1) -> Net-(J12-Pin_3)
- R124 pad 1: Net-(J13-Pin_1) -> Net-(J12-Pin_3)
- R128 pad 1: Net-(J13-Pin_2) -> Net-(J12-Pin_2)
Routing:
- net GND: track 36.4 -> 0.25 mm, vias 33 -> 0
- net /LIM_ENC/Y_ENC_INDEX_INPUT: track 15.9 -> 0.00 mm, vias 2 -> 0
- net +3.3V: track 35.6 -> 20.7 mm, vias 16 -> 6
- net /LIM_ENC/X_ENC_INDEX_INPUT: track 10.0 -> 0.00 mm, vias 2 -> 0
- net Net-(J15-Pin_1): track 9.83 -> 0.00 mm
- net Net-(J12-Pin_1): track 9.83 -> 0.00 mm
- net Net-(J13-Pin_1): track 9.83 -> 0.00 mm
- net Net-(J17-Pin_1): track 9.83 -> 0.00 mm
- net Net-(J15-Pin_2): track 9.77 -> 0.00 mm
- net Net-(J12-Pin_2): track 9.77 -> 0.00 mm
- net Net-(J17-Pin_2): track 9.77 -> 0.00 mm
- net Net-(J13-Pin_2): track 9.77 -> 0.00 mm
- net Net-(J18-Pin_1): track 9.14 -> 0.00 mm
- net /LIM_ENC/Y_ENC_DO_INPUT: track 8.39 -> 0.00 mm
- net /LIM_ENC/X_ENC_DO_INPUT: track 8.39 -> 0.00 mm
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