File: hardware/Ziess-Microsope-Controller_Main_board/DC_DRIVERS.kicad_sch (KiCad schematic)
At the start: 46 parts, among them J4 B2B-XH-AM, J5 B2B-XH-AM, J6 B2B-XH-AM, U7 DRV8876PWPR, U8 DRV8876PWPR, U9 DRV8876PWPR

Commit message: init
Other:
- note added: "25V"
Changed lines of the file:
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@@
 	(generator_version "10.0")
 	(paper "A4")
+	(text "25V"
+		(exclude_from_sim no)
+		(at 167.132 71.374 0)
+		(effects
+			(font
+				(size 1.27 1.27)
+			)
+		)
+	)
+	(text "25V"
+		(exclude_from_sim no)
+		(at 56.134 30.734 0)
+		(effects
+			(font
+				(size 1.27 1.27)
+			)
+		)
+	)
+	(text "25V"
+		(exclude_from_sim no)
+		(at 64.262 132.334 0)
+		(effects
+			(font
+				(size 1.27 1.27)
+			)
+		)
+	)
 	(junction
 		(at 154.94 116.84)

Commit message: m
Parts:
- J10: renamed from J6; value B2B-XH-AM -> 43650-0224
- J8: renamed from J4; value B2B-XH-AM -> 43650-0224
- J9: renamed from J5; value B2B-XH-AM -> 43650-0224
- renumbered C61 to C100, C62 to C101, C63 to C102, C64 to C103, C65 to C104, C66 to C105, C67 to C106, C68 to C107, C69 to C108, C70 to C109, C71 to C110, C72 to C111, C73 to C112, C74 to C113, C75 to C114, C76 to C115, C77 to C116, R62 to R100, R63 to R101, R64 to R102, R65 to R103, R66 to R104, R67 to R105, R68 to R106, R69 to R107, R70 to R108, R71 to R109, R72 to R110, R73 to R111, R74 to R112, R75 to R113, R76 to R114, R77 to R115, R56 to R94, R57 to R95, R58 to R96, R59 to R97, R60 to R98, R61 to R99, U7 to U12, U8 to U13, U9 to U14
