File: hardware/Ziess-Microsope-Controller_Main_board/POWER_INPUT.kicad_sch (KiCad schematic)
At the start: 28 parts, among them J1 0430450606, Q1 BSS84, Q2 2N7002, SW1 RESET, U1 TPS24751RUVR

Commit message: m
Parts:
- C6: value 33nF -> 100nF
- J1: value 0430450606 -> 172447-0006; footprint Library:0430450606 -> Library:172447-YY06
- R2, R3: value 1.5k -> 6.8k
- R5: value 15k -> 130k
- R7: value 130k -> 15k
Changed lines of the file:
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@@
 			)
 		)
-		(property "Value" "1.5k"
+		(property "Value" "6.8k"
 			(at 150.495 41.275 90)
 			(show_name no)
@@
 		(in_pos_files yes)
 		(dnp no)
-		(fields_autoplaced yes)
 		(property "Reference" "R8"
-			(at 129.54 106.6799 0)
+			(at 128.778 106.934 0)
 			(show_name no)
 			(do_not_autoplace no)
@@
 		)
 		(property "Value" "47k"
-			(at 129.54 109.2199 0)
+			(at 128.524 108.966 0)
 			(show_name no)
 			(do_not_autoplace no)
@@
 		(in_pos_files yes)
 		(dnp no)
-		(fields_autoplaced yes)
 		(property "Reference" "R6"
-			(at 117.475 81.2799 0)
+			(at 116.84 81.788 0)
 			(show_name no)
 			(do_not_autoplace no)
@@
 		)
 		(property "Value" "10k"
-			(at 117.475 83.8199 0)
+			(at 116.84 83.566 0)
 			(show_name no)
 			(do_not_autoplace no)
@@
 		(in_pos_files yes)
 		(dnp no)
-		(fields_autoplaced yes)
 		(property "Reference" "C6"
-			(at 142.24 106.6862 0)
-			(show_name no)
-			(do_not_autoplace no)
-			(effects
-				(font
-					(size 1.27 1.27)
-				)
-				(justify left)
-			)
-		)
-		(property "Value" "33nF"
-			(at 142.24 109.2262 0)
+			(at 141.986 106.934 0)
+			(show_name no)
+			(do_not_autoplace no)
+			(effects
+				(font
+					(size 1.27 1.27)
+				)
+				(justify left)
+			)
+		)
+		(property "Value" "100nF"
+			(at 141.986 108.712 0)
 			(show_name no)
 			(do_not_autoplace no)
@@
 		(in_pos_files yes)
 		(dnp no)
-		(fields_autoplaced yes)
 		(property "Reference" "R4"
-			(at 134.62 48.2599 0)
+			(at 133.604 48.514 0)
 			(show_name no)
 			(do_not_autoplace no)
@@
 		)
 		(property "Value" "36"
-			(at 134.62 50.7999 0)
+			(at 133.604 50.546 0)
 			(show_name no)
 			(do_not_autoplace no)
@@
 			)
 		)
-		(property "Value" "1.5k"
+		(property "Value" "6.8k"
 			(at 155.575 47.625 90)
 			(show_name no)
@@
 		(in_pos_files yes)
 		(dnp no)
-		(fields_autoplaced yes)
 		(property "Reference" "R5"
-			(at 117.475 54.6099 0)
-			(show_name no)
-			(do_not_autoplace no)
-			(effects
-				(font
-					(size 1.27 1.27)
-				)
-				(justify left)
-			)
-		)
-		(property "Value" "15k"
-			(at 117.475 57.1499 0)
+			(at 117.094 55.372 0)
+			(show_name no)
+			(do_not_autoplace no)
+			(effects
+				(font
+					(size 1.27 1.27)
+				)
+				(justify left)
+			)
+		)
+		(property "Value" "130k"
+			(at 116.84 57.15 0)
 			(show_name no)
 			(do_not_autoplace no)
@@
 			)
 		)
-		(property "Value" "0430450606"
+		(property "Value" "172447-0006"
 			(at 26.416 76.454 0)
 			(show_name no)
@@
 			)
 		)
-		(property "Footprint" "Library:0430450606"
+		(property "Footprint" "Library:172447-YY06"
 			(at 26.67 68.58 0)
 			(hide yes)
@@
 		(in_pos_files yes)
 		(dnp no)
-		(fields_autoplaced yes)
 		(property "Reference" "R7"
-			(at 117.475 106.6799 0)
-			(show_name no)
-			(do_not_autoplace no)
-			(effects
-				(font
-					(size 1.27 1.27)
-				)
-				(justify left)
-			)
-		)
-		(property "Value" "130k"
-			(at 117.475 109.2199 0)
+			(at 117.094 107.188 0)
+			(show_name no)
+			(do_not_autoplace no)
+			(effects
+				(font
+					(size 1.27 1.27)
+				)
+				(justify left)
+			)
+		)
+		(property "Value" "15k"
+			(at 116.84 108.966 0)
 			(show_name no)
 			(do_not_autoplace no)
@@
 		(dnp no)
 		(property "Reference" "R9"
-			(at 178.435 108.585 0)
+			(at 178.054 108.458 0)
 			(show_name no)
 			(do_not_autoplace no)
@@
 		)
 		(property "Value" "1.3k"
-			(at 180.975 110.49 0)
-			(show_name no)
-			(do_not_autoplace no)
+			(at 179.578 110.236 0)
+			(show_name no)
+			(do_not_autoplace no)

Commit message: m
Parts:
- added C151: 100nF, Capacitor_SMD:C_0805_2012Metric, symbol Device:C_Small
- added C152: 10uF, Capacitor_SMD:C_0805_2012Metric, symbol Device:C_Small
- added D22: SMF5V0A, Diode_SMD:D_SMF, symbol Diode:SMF5V0A
- added R100: 100k, Resistor_SMD:R_0603_1608Metric, symbol Device:R_Small
- added R96: 10k, Resistor_SMD:R_0603_1608Metric, symbol Device:R_Small
- added R99: 22k, Resistor_SMD:R_0603_1608Metric, symbol Device:R_Small
- C2: footprint Capacitor_SMD:C_0805_2012Metric -> Capacitor_SMD:C_1210_3225Metric
- R2, R3: value 6.8k -> 10k
- R4: value 36 -> 51.1
- R8: value 47k -> 57.6k
- R9: value 1.3k -> 1.78k
Connections:
- net +12V: now also R100.1
- net +5VSB: now also C151.1, C152.1, D22.1 (A1)
- net GND: now also C151.2, C152.2, D22.2 (A2), R99.2
- net INPUT_IMON: now also R96.2; no longer R9.1, U1.2 (IMON)
- new net: R9.1, R96.1, U1.2 (IMON)
- new net 12V_SENSE: R100.2, R99.1
Other:
- moved on the sheet: C2, D3, J1, Q1, Q2, R10, R11, R12, R137, SW1

Commit message: m
Parts:
- renumbered C151 to C6, C152 to C7, C121 to C8, C6 to C9, D22 to D4, R99 to R1, R7 to R10, R8 to R11, R9 to R12, R10 to R13, R11 to R14, R137 to R15, R12 to R16, R100 to R2, R1 to R3, R2 to R4, R3 to R5, R4 to R6, R5 to R7, R6 to R8, R96 to R9
