File: hardware/Ziess-Microsope-Controller_Main_board/USB_SYNC.kicad_sch (KiCad schematic)
At the start: 29 parts, among them J18 CONBNC001, J19 USB_B, U15 USBLC6-2SC6, U16 74LVC1G17, U17 74AHCT1G125, U19 ADUM3160

Commit message: m
Parts:
- J5: renamed from J18; value CONBNC001 -> U.FL-R-SMT-1_10; footprint Library:CONBNC001 -> Library:U.FL-R-SMT-1_10_
- renumbered C124 to C57, C125 to C58, C126 to C59, C139 to C60, C123 to C61, C106 to C62, C99 to C63, D21 to D5, J19 to J4, R149 to R46, R151 to R47, R155 to R48, R148 to R49, R156 to R50, R154 to R51, R153 to R52, R107 to R53, R188 to R54, R101 to R55, R105 to R56, R189 to R57, R146 to R58, R147 to R59, U19 to U6, U15 to U7, U17 to U8, U16 to U9
Connections:
- net at U7.1 (I/O1): now also R48.2; no longer J4.3 (D+)
- net at U7.3 (I/O2): now also R50.2; no longer J4.2 (D-)
- net at U7.4 (I/O2): now also J4.2 (D-); no longer R50.2
- net at U7.6 (I/O1): now also J4.3 (D+); no longer R48.2
