File: hardware/Ziess-Microsope-Controller_Main_board/Y_DRIVER.kicad_sch (KiCad schematic)
At the start: 38 parts, among them J3 B4B-XH-AM, U6 TMC2209-LA

Commit message: init
Parts:
- J3: value B4B-XH-AM -> 43045-0418
- R44: now fitted; now in the parts list
- R45, R48: now not fitted; now left out of the parts list
- R52, R53: footprint Resistor_SMD:R_0603_1608Metric -> Resistor_SMD:R_2010_5025Metric
Changed lines of the file:
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@@
 	(text "2010"
 		(exclude_from_sim no)
-		(at 181.61 127 0)
+		(at 181.864 128.016 0)
 		(effects
 			(font
@@
 			)
 		)
-		(property "Value" "B4B-XH-AM"
+		(property "Value" "43045-0418"
 			(at 234.95 101.6 0)
 			(show_name no)
@@
 		(body_style 1)
 		(exclude_from_sim no)
-		(in_bom yes)
+		(in_bom no)
 		(on_board yes)
 		(in_pos_files yes)
-		(dnp no)
+		(dnp yes)
 		(property "Reference" "R48"
 			(at 72.39 90.805 0)
@@
 		(body_style 1)
 		(exclude_from_sim no)
-		(in_bom no)
+		(in_bom yes)
 		(on_board yes)
 		(in_pos_files yes)
-		(dnp yes)
+		(dnp no)
 		(property "Reference" "R44"
 			(at 72.39 79.375 0)
@@
 			)
 		)
-		(property "Footprint" "Resistor_SMD:R_0603_1608Metric"
+		(property "Footprint" "Resistor_SMD:R_2010_5025Metric"
 			(at 185.42 113.03 0)
 			(hide yes)
@@
 		(body_style 1)
 		(exclude_from_sim no)
-		(in_bom yes)
+		(in_bom no)
 		(on_board yes)
 		(in_pos_files yes)
-		(dnp no)
+		(dnp yes)
 		(property "Reference" "R45"
 			(at 102.235 80.645 90)
@@
 			)
 		)
-		(property "Footprint" "Resistor_SMD:R_0603_1608Metric"
+		(property "Footprint" "Resistor_SMD:R_2010_5025Metric"
 			(at 175.26 113.03 0)
 			(hide yes)

Commit message: m
Parts:
- renumbered C43 to C82, C44 to C83, C45 to C84, C46 to C85, C47 to C86, C48 to C87, C49 to C88, C50 to C89, C51 to C90, C52 to C91, C53 to C92, C54 to C93, C55 to C94, C56 to C95, C57 to C96, C58 to C97, C59 to C98, C60 to C99, D5 to D7, J3 to J7, R39 to R77, R40 to R78, R41 to R79, R42 to R80, R43 to R81, R44 to R82, R45 to R83, R46 to R84, R47 to R85, R48 to R86, R49 to R87, R50 to R88, R51 to R89, R52 to R90, R53 to R91, R54 to R92, R55 to R93, U6 to U11
