File: hardware/Ziess-Microsope-Controller_Main_board/ACC1.kicad_sch (KiCad schematic)
At the start: 34 parts, among them J21 Conn_01x08_Shielded, Q3 2N7002, U20 TPS259472LRPWR, U21 THVD2450VDRCR

Commit message: m
Parts:
- removed J21: Conn_01x08_Shielded, Library:MD80SV, symbol Connector_Generic_Shielded:Conn_01x08_Shielded
- added J20: 43045-0810, Connector_Molex:Molex_Micro-Fit_3.0_43045-0810_2x04-1MP_P3.00mm_Horizontal, symbol Connector_Generic:Conn_01x08
- renumbered C129 to C137, C98 to C138, C132 to C139, C131 to C140, C128 to C141, C127 to C142, C133 to C143, C134 to C144, D9 to D13, D10 to D14, D7 to D15, D8 to D16, D6 to D17, R108 to R151, R113 to R152, R144 to R153, R110 to R154, R116 to R155, R109 to R156, R111 to R157, R143 to R158, R115 to R159, R114 to R160, R112 to R161, R142 to R162, R141 to R163, R138 to R164, R139 to R165, R140 to R166, R136 to R167
Connections:
- net ACC1_+12V: now also J20.1 (Pin_1), J20.2 (Pin_2)
- net GND: now also D16.1 (A1), D17.1 (A1), R167.1, J20.3 (Pin_3), J20.5 (Pin_5)
- net at R163.1, R165.1: now also J20.4 (Pin_4)
- net at D16.2 (A2), U21.8 (A): now also J20.7 (Pin_7)
- net at D17.2 (A2), U21.9 (B): now also J20.8 (Pin_8)
- net at R162.1, R166.1: now also J20.6 (Pin_6)
- net ACC3_DIR renamed ACC1_DIR
- net ACC3_IMON renamed ACC1_IMON
- net ACC3_PG renamed ACC1_PG
- net ACC3_PRESENT renamed ACC1_PRESENT
- net ACC3_PWR_EN renamed ACC1_PWR_EN
- net ACC3_PWR_FLG renamed ACC1_PWR_FLG
- net ACC3_RX renamed ACC1_RX
- net ACC3_TX renamed ACC1_TX

Commit message: init
Parts:
- added R203, R204, R205: 100, Resistor_SMD:R_0603_1608Metric, symbol Device:R_Small
- added R206: 10k, Resistor_SMD:R_0603_1608Metric, symbol Device:R_Small
- added R215: 120, Resistor_SMD:R_0603_1608Metric, symbol Device:R_Small
Connections:
- net +3.3V: now also R206.2; no longer U21.7 (SLR)
- net ACC1_DIR: now also R204.1; no longer R167.2, U21.3 (DE), U21.4 (~{RE})
- net ACC1_RX: now also R203.1; no longer R164.1, U21.2 (R)
- net ACC1_TX: now also R205.1; no longer U21.5 (D)
- net at D16.2 (A2), J20.7 (Pin_7), U21.8 (A): now also R215.2
- net at D17.2 (A2), J20.8 (Pin_8), U21.9 (B): now also R215.1
- new net: R164.1, R203.2, U21.2 (R)
- new net: R205.2, U21.5 (D)
- new net: R167.2, R204.2, U21.3 (DE), U21.4 (~{RE})
- new net: R206.1, U21.7 (SLR)
