File: hardware/Ziess-Microsope-Controller_Main_board/ACC2.kicad_sch (KiCad schematic)
At the start: 34 parts, among them J22 Conn_01x08_Shielded, Q4 2N7002, U22 TPS259472LRPWR, U23 THVD2450VDRCR

Commit message: m
Parts:
- removed C130: 22nF, Capacitor_SMD:C_0603_1608Metric, symbol Device:C_Small
- removed C135: 1uF, Capacitor_SMD:C_1206_3216Metric, symbol Device:C_Small
- removed C136, C138, C140: 100nF, Capacitor_SMD:C_0603_1608Metric, symbol Device:C_Small
- removed C137: 3.3nF, Capacitor_SMD:C_0402_1005Metric, symbol Device:C_Small
- removed C141: 10uF, Capacitor_SMD:C_1210_3225Metric, symbol Device:C_Small
- removed C142: 47uF, Capacitor_SMD:CP_Elec_6.3x7.7, symbol Device:C_Polarized_Small
- removed D11, D12: SMAJ30CA, Diode_SMD:D_SMA, symbol Diode:SMAJ30CA
- removed D13: GREEN, LED_SMD:LED_0603_1608Metric, symbol Device:LED
- removed D14: B330A-13-F, Diode_SMD:D_SMA, symbol Diode:B330
- removed D15: SMAJ15A, Diode_SMD:D_SMA, symbol Diode:SMAJ15A
- removed J22: Conn_01x08_Shielded, Library:MD80SV, symbol Connector_Generic_Shielded:Conn_01x08_Shielded
- removed R145: 100, Resistor_SMD:R_0603_1608Metric, symbol Device:R_Small
- removed R150, R158, R159, R162, R163, R164, R165, R166, R167: 10k, Resistor_SMD:R_0603_1608Metric, symbol Device:R_Small
- removed R152: 470k, Resistor_SMD:R_0603_1608Metric, symbol Device:R_Small
- removed R157: 390k, Resistor_SMD:R_0603_1608Metric, symbol Device:R_Small
- removed R160: 1.65k, Resistor_SMD:R_0603_1608Metric, symbol Device:R_Small
- removed R161: 82k, Resistor_SMD:R_0603_1608Metric, symbol Device:R_Small
- added C145: 10uF, Capacitor_SMD:C_1210_3225Metric, symbol Device:C_Small
- added C146: 47uF, Capacitor_SMD:CP_Elec_6.3x7.7, symbol Device:C_Polarized_Small
- added C147: 1uF, Capacitor_SMD:C_1206_3216Metric, symbol Device:C_Small
- added C148, C151, C152: 100nF, Capacitor_SMD:C_0603_1608Metric, symbol Device:C_Small
- added C149: 22nF, Capacitor_SMD:C_0603_1608Metric, symbol Device:C_Small
- added C150: 3.3nF, Capacitor_SMD:C_0402_1005Metric, symbol Device:C_Small
- added D18: B330A-13-F, Diode_SMD:D_SMA, symbol Diode:B330
- added D19: SMAJ15A, Diode_SMD:D_SMA, symbol Diode:SMAJ15A
- added D20: GREEN, LED_SMD:LED_0603_1608Metric, symbol Device:LED
- added D21, D22: SMAJ30CA, Diode_SMD:D_SMA, symbol Diode:SMAJ30CA
- added J21: 43045-0810, Connector_Molex:Molex_Micro-Fit_3.0_43045-0810_2x04-1MP_P3.00mm_Horizontal, symbol Connector_Generic:Conn_01x08
- added R171: 100, Resistor_SMD:R_0603_1608Metric, symbol Device:R_Small
- added R172: 1.5k, Resistor_SMD:R_0603_1608Metric, symbol Device:R_Small
- added R173, R175, R176, R177, R179, R180, R181, R182, R183, R184: 10k, Resistor_SMD:R_0603_1608Metric, symbol Device:R_Small
- added R174: 390k, Resistor_SMD:R_0603_1608Metric, symbol Device:R_Small
- added R178: 1.65k, Resistor_SMD:R_0603_1608Metric, symbol Device:R_Small
- R168: value 10k -> 470k; now not fitted; now left out of the parts list
- R169: value 10k -> 82k
- R170: value 1.5k -> 10k
Connections:
- net ACC3_PG is gone; now on net +12V: R168.2
- net +12V: now also C147.2, C148.2
- net +3.3V: now also C151.2, C152.2, R172.2, R176.2, R179.2, R180.2, R181.2; no longer R169.2, R170.2
- net GND: now also C145.1, C146.2, C147.1, C148.1, C149.1, C150.1, C151.1, C152.1, D18.2 (A), D19.2 (A2), D21.1 (A1), D22.1 (A1), J21.3 (Pin_3), J21.5 (Pin_5), R173.1, R174.1, R177.1, R178.1, R184.1
- net at U22.1 (EN/UVLO_1), U22.11 (EN/UVLO_2): now also R168.1, R171.1, R173.2
- net at U22.10 (ITIMER_1), U22.14 (ITIMER_2): now also C149.2
- net at U22.12 (PGTH/_~{FLT_2}), U22.4 (PGTH/_~{FLT_1}): now also R169.2, R177.2
- net at U22.13 (DVDT_2), U22.7 (DVDT_1): now also C150.2
- net at U22.2 (OVLO/_OVCSEL): now also R174.2
- net at Q4.1 (G), U22.3 (PG/_AUXOFF): now also R170.1, R176.1; no longer R168.1, R169.1
- net at U22.9 (ILM): now also R175.2, R178.2
- net at Q4.3 (D): now also D20.1 (K)
- net at U23.8 (A): now also D21.2 (A2), J21.7 (Pin_7)
- net at U23.9 (B): now also D22.2 (A2), J21.8 (Pin_8)
- net ACC1_+12V renamed ACC2_+12V
- net ACC2_+12V: now also R169.1, C145.2, C146.1, D18.1 (K), D19.1 (A1), J21.1 (Pin_1), J21.2 (Pin_2)
- net ACC3_DIR renamed ACC2_DIR
- net ACC2_DIR: now also R184.2
- net ACC3_RX renamed ACC2_RX
- net ACC2_RX: now also R181.1
- net ACC3_TX renamed ACC2_TX
- new net: J21.6 (Pin_6), R179.1, R183.1
- new net: J21.4 (Pin_4), R180.1, R182.1
- new net: D20.2 (A), R172.1
- new net ACC2_IMON: R175.1
- new net ACC2_PG: R170.2
- new net ACC2_PRESENT: R182.2
- new net ACC2_PWR_EN: R171.2
- new net ACC2_PWR_FLG: R183.2

Commit message: init
Parts:
- added R207, R208, R209: 100, Resistor_SMD:R_0603_1608Metric, symbol Device:R_Small
- added R210: 10k, Resistor_SMD:R_0603_1608Metric, symbol Device:R_Small
- added R216: 120, Resistor_SMD:R_0603_1608Metric, symbol Device:R_Small
Connections:
- net +3.3V: now also R210.2; no longer U23.7 (SLR)
- net ACC2_DIR: now also R208.1; no longer R184.2, U23.3 (DE), U23.4 (~{RE})
- net ACC2_RX: now also R207.1; no longer R181.1, U23.2 (R)
- net ACC2_TX: now also R209.1; no longer U23.5 (D)
- net at D22.2 (A2), J21.8 (Pin_8), U23.9 (B): now also R216.1
- net at D21.2 (A2), J21.7 (Pin_7), U23.8 (A): now also R216.2
- new net: R181.1, R207.2, U23.2 (R)
- new net: R209.2, U23.5 (D)
- new net: R210.1, U23.7 (SLR)
- new net: R184.2, R208.2, U23.3 (DE), U23.4 (~{RE})
