File: hardware/Ziess-Microsope-Controller_Main_board/ACC3.kicad_sch (KiCad schematic)
At the start: 34 parts, among them J23 Conn_01x08_Shielded, Q5 2N7002, U24 TPS259472LRPWR, U25 THVD2450VDRCR

Commit message: m
Parts:
- removed C143: 1uF, Capacitor_SMD:C_1206_3216Metric, symbol Device:C_Small
- removed C144, C147, C148: 100nF, Capacitor_SMD:C_0603_1608Metric, symbol Device:C_Small
- removed C145: 22nF, Capacitor_SMD:C_0603_1608Metric, symbol Device:C_Small
- removed C146: 3.3nF, Capacitor_SMD:C_0402_1005Metric, symbol Device:C_Small
- removed C149: 10uF, Capacitor_SMD:C_1210_3225Metric, symbol Device:C_Small
- removed C150: 47uF, Capacitor_SMD:CP_Elec_6.3x7.7, symbol Device:C_Polarized_Small
- removed D16, D17: SMAJ30CA, Diode_SMD:D_SMA, symbol Diode:SMAJ30CA
- removed D18: GREEN, LED_SMD:LED_0603_1608Metric, symbol Device:LED
- removed D19: B330A-13-F, Diode_SMD:D_SMA, symbol Diode:B330
- removed D20: SMAJ15A, Diode_SMD:D_SMA, symbol Diode:SMAJ15A
- removed J23: Conn_01x08_Shielded, Library:MD80SV, symbol Connector_Generic_Shielded:Conn_01x08_Shielded
- removed R171: 100, Resistor_SMD:R_0603_1608Metric, symbol Device:R_Small
- removed R172, R175, R176, R179, R180, R181, R182, R183, R184: 10k, Resistor_SMD:R_0603_1608Metric, symbol Device:R_Small
- removed R173: 470k, Resistor_SMD:R_0603_1608Metric, symbol Device:R_Small
- removed R174: 390k, Resistor_SMD:R_0603_1608Metric, symbol Device:R_Small
- removed R177: 1.65k, Resistor_SMD:R_0603_1608Metric, symbol Device:R_Small
- removed R178: 82k, Resistor_SMD:R_0603_1608Metric, symbol Device:R_Small
- added C153: 10uF, Capacitor_SMD:C_1210_3225Metric, symbol Device:C_Small
- added C154: 47uF, Capacitor_SMD:CP_Elec_6.3x7.7, symbol Device:C_Polarized_Small
- added C155: 1uF, Capacitor_SMD:C_1206_3216Metric, symbol Device:C_Small
- added C156, C159, C160: 100nF, Capacitor_SMD:C_0603_1608Metric, symbol Device:C_Small
- added C157: 22nF, Capacitor_SMD:C_0603_1608Metric, symbol Device:C_Small
- added C158: 3.3nF, Capacitor_SMD:C_0402_1005Metric, symbol Device:C_Small
- added D23: B330A-13-F, Diode_SMD:D_SMA, symbol Diode:B330
- added D24: SMAJ15A, Diode_SMD:D_SMA, symbol Diode:SMAJ15A
- added D25: GREEN, LED_SMD:LED_0603_1608Metric, symbol Device:LED
- added D26, D27: SMAJ30CA, Diode_SMD:D_SMA, symbol Diode:SMAJ30CA
- added J22: 43045-0810, Connector_Molex:Molex_Micro-Fit_3.0_43045-0810_2x04-1MP_P3.00mm_Horizontal, symbol Connector_Generic:Conn_01x08
- added R188: 100, Resistor_SMD:R_0603_1608Metric, symbol Device:R_Small
- added R189: 1.5k, Resistor_SMD:R_0603_1608Metric, symbol Device:R_Small
- added R190, R192, R193, R194, R196, R197, R198, R199, R200, R201: 10k, Resistor_SMD:R_0603_1608Metric, symbol Device:R_Small
- added R191: 390k, Resistor_SMD:R_0603_1608Metric, symbol Device:R_Small
- added R195: 1.65k, Resistor_SMD:R_0603_1608Metric, symbol Device:R_Small
- R185: value 10k -> 470k; now not fitted; now left out of the parts list
- R186: value 10k -> 82k
- R187: value 1.5k -> 10k
Connections:
- net +12V: now also R185.2, C155.2, C156.2
- net +3.3V: now also C159.2, C160.2, R189.2, R193.2, R196.2, R197.2, R198.2; no longer R186.2, R187.2
- net ACC1_+12V: now also R186.1, C153.2, C154.1, D23.1 (K), D24.1 (A1), J22.1 (Pin_1), J22.2 (Pin_2)
- net ACC3_DIR: now also R201.2
- net ACC3_IMON: now also R192.1
- net ACC3_PG: now also R187.2; no longer R185.2
- net ACC3_PRESENT: now also R199.2
- net ACC3_PWR_EN: now also R188.2
- net ACC3_PWR_FLG: now also R200.2
- net ACC3_RX: now also R198.1
- net GND: now also C153.1, C154.2, C155.1, C156.1, C157.1, C158.1, C159.1, C160.1, D23.2 (A), D24.2 (A2), D26.1 (A1), D27.1 (A1), J22.3 (Pin_3), J22.5 (Pin_5), R190.1, R191.1, R194.1, R195.1, R201.1
- net at U24.1 (EN/UVLO_1), U24.11 (EN/UVLO_2): now also R185.1, R188.1, R190.2
- net at U24.10 (ITIMER_1), U24.14 (ITIMER_2): now also C157.2
- net at U24.12 (PGTH/_~{FLT_2}), U24.4 (PGTH/_~{FLT_1}): now also R186.2, R194.2
- net at U24.13 (DVDT_2), U24.7 (DVDT_1): now also C158.2
- net at U24.2 (OVLO/_OVCSEL): now also R191.2
- net at Q5.1 (G), U24.3 (PG/_AUXOFF): now also R187.1, R193.1; no longer R185.1, R186.1
- net at U24.9 (ILM): now also R192.2, R195.2
- net at Q5.3 (D): now also D25.1 (K)
- net at U25.8 (A): now also D26.2 (A2), J22.7 (Pin_7)
- net at U25.9 (B): now also D27.2 (A2), J22.8 (Pin_8)
- new net: D25.2 (A), R189.1
- new net: J22.6 (Pin_6), R196.1, R200.1
- new net: J22.4 (Pin_4), R197.1, R199.1

Commit message: init
Parts:
- added R211, R212, R213: 100, Resistor_SMD:R_0603_1608Metric, symbol Device:R_Small
- added R214: 10k, Resistor_SMD:R_0603_1608Metric, symbol Device:R_Small
- added R217: 120, Resistor_SMD:R_0603_1608Metric, symbol Device:R_Small
Connections:
- net +3.3V: now also R214.2; no longer U25.7 (SLR)
- net ACC3_DIR: now also R212.1; no longer R201.2, U25.3 (DE), U25.4 (~{RE})
- net ACC3_RX: now also R211.1; no longer R198.1, U25.2 (R)
- net ACC3_TX: now also R213.1; no longer U25.5 (D)
- net at D26.2 (A2), J22.7 (Pin_7): now also U25.9 (B), R217.2; no longer U25.8 (A)
- net at D27.2 (A2), J22.8 (Pin_8): now also U25.8 (A), R217.1; no longer U25.9 (B)
- new net: R198.1, R211.2, U25.2 (R)
- new net: R201.2, R212.2, U25.3 (DE), U25.4 (~{RE})
- new net: R213.2, U25.5 (D)
- new net: R214.1, U25.7 (SLR)

Commit message: m
Parts:
- added JP1: SolderJumper_3_Bridged12, symbol Jumper:SolderJumper_3_Bridged12
- added TP1, TP2, TP5: TestPoint, TestPoint:TestPoint_Pad_D1.0mm, symbol Connector:TestPoint
- C158: footprint Capacitor_SMD:C_0402_1005Metric -> Capacitor_SMD:C_0603_1608Metric
Connections:
- net +3.3V: now also JP1.1 (A); no longer R214.2
- net GND: now also JP1.3 (B)
- new net: JP1.2 (C), R214.2
Other:
- moved on the sheet: C160, R214
