File: hardware/Ziess-Microsope-Controller_Main_board/LIM_ENC.kicad_sch (KiCad schematic)
At the start: 52 parts, among them J10 B3B-XH-AM, J11 B4B-XH-AM, J12 B2B-XH-AM, J13 B6B-XH-AM, J14 B6B-XH-AM, J15 B3B-XH-AM, J7 B3B-XH-AM, J8 B3B-XH-AM, J9 B6B-XH-AM, U10 SN74LVC2G17DBV, U11 SN74LVC2G17DBV, U12 SN74LVC2G17DBV, U13 SN74LVC2G17DBV, U14 SN74LVC2G17DBV

Commit message: m
Parts:
- removed J12: B2B-XH-AM, Library:BM02B-GHS-TBT_1, symbol Connector_Generic:Conn_01x02
- added J12: BM03B-GHS-TBT, Library:BM03BGHSTBTLFSN, symbol Connector_Generic:Conn_01x03
- added R102, R103, R104, R106, R190, R191, R192, R193, R98: 10K, Resistor_SMD:R_0603_1608Metric, symbol Device:R_Small
- added R194, R195: 3.3k, Resistor_SMD:R_0603_1608Metric, symbol Device:R_Small
- added R196, R197: 10k, Resistor_SMD:R_0603_1608Metric, symbol Device:R_Small
- added R198, R199, R200, R201: 22, Resistor_SMD:R_0603_1608Metric, symbol Device:R_Small
- added U26, U27, U28, U29, U30: TPD4E05U06DQA, Package_SON:USON-10_2.5x1.0mm_P0.5mm, symbol Power_Protection:TPD4E05U06DQA
- C84: footprint Capacitor_SMD:C_0201_0603Metric -> Capacitor_SMD:C_0603_1608Metric
- J10, J15, J7, J8: value B3B-XH-AM -> BM03B-GHS-TBT
- J11: value B4B-XH-AM -> BM04B-GHS-TBT
- J13, J14, J9: value B6B-XH-AM -> BM06B-GHS-TBT
Connections:
- net +3.3V: now also R196.1, R197.1
- net +5VSB: now also R194.2, R195.2
- net F_LIM_1: now also R191.2; no longer J8.1 (Pin_1)
- net F_LIM_2: now also R192.2; no longer J8.2 (Pin_2)
- net GND: now also J12.3 (Pin_3), U26.3 (GND), U26.8 (GND), U27.3 (GND), U27.8 (GND), U28.3 (GND), U28.8 (GND), U29.3 (GND), U29.8 (GND), U30.3 (GND), U30.8 (GND)
- net J_LIM: now also R193.2
- net X_ENC_CLK_OUTPUT: now also R200.1; no longer U11.6 (1Y)
- net X_ENC_CS_OUTPUT: now also R201.1; no longer U11.4 (2Y)
- net X_ENC_DO_INPUT: now also R196.2
- net X_LIM_1: now also R103.2; no longer J10.1 (Pin_1)
- net X_LIM_2: now also R104.2; no longer J10.2 (Pin_2)
- net Y_ENC_CLK_OUTPUT: now also R198.1; no longer U14.6 (1Y)
- net Y_ENC_CS_OUTPUT: now also R199.1; no longer U14.4 (2Y)
- net Y_ENC_DO_INPUT: now also R197.2
- net Y_LIM_1: now also R98.2; no longer J7.1 (Pin_1)
- net Y_LIM_2: now also R102.2; no longer J7.2 (Pin_2)
- net Z_LIM_1: now also R106.2; no longer J15.1 (Pin_1)
- net Z_LIM_2: now also R190.2; no longer J15.2 (Pin_2)
- net at J11.2 (Pin_2), U12.1 (1A): now also R195.1
- net at J11.3 (Pin_3), U12.3 (2A): now also R194.1
- new net: J15.1 (Pin_1), U28.4 (D2+)
- new net: J15.2 (Pin_2), U28.5 (D2-)
- new net: R103.1, U27.1 (D1+)
- new net: J10.1 (Pin_1), U27.4 (D2+)
- new net: J10.2 (Pin_2), U27.5 (D2-)
- new net: J12.1 (Pin_1), U30.4 (D2+)
- new net: J12.2 (Pin_2), U30.5 (D2-)
- new net: R192.1, U29.2 (D1-)
- new net: R193.1, U30.1 (D1+)
- new net: R104.1, U27.2 (D1-)
- new net: J8.1 (Pin_1), U29.4 (D2+)
- new net: J8.2 (Pin_2), U29.5 (D2-)
- new net: J7.1 (Pin_1), U26.4 (D2+)
- new net: J7.2 (Pin_2), U26.5 (D2-)
- new net: R200.2, U11.6 (1Y)
- new net: R98.1, U26.1 (D1+)
- new net: R102.1, U26.2 (D1-)
- new net: R190.1, U28.2 (D1-)
- new net: R199.2, U14.4 (2Y)
- new net: R106.1, U28.1 (D1+)
- new net: R198.2, U14.6 (1Y)
- new net: R191.1, U29.1 (D1+)
- new net: R201.2, U11.4 (2Y)
Other:
- moved on the sheet: C78, C79, C80, C83, C84, C85, C86, C87, C90, C91, C92, C94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

Commit message: init
Parts:
- removed U26, U27, U28, U29, U30: TPD4E05U06DQA, Package_SON:USON-10_2.5x1.0mm_P0.5mm, symbol Power_Protection:TPD4E05U06DQA
- added D23, D24, D25, D26, D27: SP0502BAHT, Package_TO_SOT_SMD:SOT-23, symbol Power_Protection:SP0502BAHT
Connections:
- net F_LIM_1: no longer C82.2, R81.1
- net F_LIM_2: no longer C81.2, R80.1
- net GND: now also D23.3 (A), D24.3 (A), D25.3 (A), D26.3 (A), D27.3 (A)
- net J_LIM: no longer C93.2, R88.1
- net X_LIM_1: no longer C89.2, R85.1
- net X_LIM_2: no longer C88.2, R84.1
- net Y_LIM_1: no longer C80.2, R79.1
- net Y_LIM_2: no longer C79.2, R78.1
- net Z_LIM_1: no longer C97.2, R95.1
- net Z_LIM_2: no longer C96.2, R94.1
- net at J15.1 (Pin_1): now also C97.2, R106.1, R95.1, D25.1 (K)
- net at J15.2 (Pin_2): now also C96.2, R190.1, R94.1, D25.2 (K)
- net at R103.1: now also C89.2, J10.1 (Pin_1), R85.1, D24.1 (K)
- net at J10.2 (Pin_2): now also C88.2, R104.1, R84.1, D24.2 (K)
- net at J12.1 (Pin_1): now also C93.2, R193.1, R88.1, D27.1 (K)
- net at R192.1: now also C81.2, J8.2 (Pin_2), R80.1, D26.2 (K)
- net at J8.1 (Pin_1): now also C82.2, R191.1, R81.1, D26.1 (K)
- net at J7.1 (Pin_1): now also C80.2, R79.1, R98.1, D23.1 (K)
- net at J7.2 (Pin_2): now also C79.2, R102.1, R78.1, D23.2 (K)
- no-connect marks 0 -> 2
Other:
- moved on the sheet: C79, C80, C86, C87, C88, C89, J10, J11, J7, R194, R195, R78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

Commit message: m
Parts:
- renumbered C86 to C117, C87 to C118, C79 to C119, C80 to C120, C78 to C121, C83 to C122, C84 to C123, C85 to C124, C88 to C125, C89 to C126, C90 to C127, C91 to C128, C92 to C129, C96 to C130, C97 to C131, C95 to C132, C81 to C133, C82 to C134, C94 to C135, C93 to C136, D25 to D10, D26 to D11, D27 to D12, D23 to D8, D24 to D9, J7 to J12, J10 to J13, J9 to J14, J13 to J16, J8 to J17, J12 to J18, J14 to J19, R195 to R116, R194 to R117, R78 to R118, R79 to R119, R98 to R120, R102 to R121, R84 to R122, R85 to R123, R103 to R124, R196 to R125, R82 to R126, R83 to R127, R104 to R128, R200 to R129, R201 to R130, R94 to R131, R95 to R132, R106 to R133, R197 to R134, R86 to R135, R87 to R136, R190 to R137, R80 to R138, R81 to R139, R191 to R140, R192 to R141, R198 to R142, R199 to R143, R88 to R144, R193 to R145, R89 to R146, R90 to R147, R91 to R148, R92 to R149, R93 to R150, U12 to U15, U10 to U16, U11 to U17, U13 to U18, U14 to U19
Connections:
- net +5VSB: now also J11.4 (Pin_4); no longer J11.1 (Pin_1)
- net GND: now also J11.1 (Pin_1); no longer J11.4 (Pin_4)
- net at R116.1, U15.1 (1A): now also J11.3 (Pin_3); no longer J11.2 (Pin_2)
- net at R117.1, U15.3 (2A): now also J11.2 (Pin_2); no longer J11.3 (Pin_3)
Other:
- moved on the sheet: J11

Commit message: init
Connections:
- net XY_ENC_CLK: now also U17.3 (2A), U19.3 (2A); no longer U17.1 (1A), U19.1 (1A)
- net X_ENC_CS: now also U17.1 (1A); no longer U17.3 (2A)
- net Y_ENC_CS: now also U19.1 (1A); no longer U19.3 (2A)
- net at R129.2: now also U17.4 (2Y); no longer U17.6 (1Y)
- net at R143.2: now also U19.6 (1Y); no longer U19.4 (2Y)
- net at R142.2: now also U19.4 (2Y); no longer U19.6 (1Y)
- net at R130.2: now also U17.6 (1Y); no longer U17.4 (2Y)
Changed lines of the file:
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@@
 	)
 	(symbol
-		(lib_id "Library:SN74LVC2G17DBV")
-		(at 181.61 142.24 0)
-		(unit 1)
-		(body_style 1)
-		(exclude_from_sim no)
-		(in_bom yes)
-		(on_board yes)
-		(in_pos_files yes)
-		(dnp no)
-		(property "Reference" "U19"
-			(at 173.99 132.715 0)
-			(show_name no)
-			(do_not_autoplace no)
-			(effects
-				(font
-					(size 1.27 1.27)
-				)
-				(justify left)
-			)
-		)
-		(property "Value" "SN74LVC2G17DBV"
-			(at 184.785 151.13 0)
-			(show_name no)
-			(do_not_autoplace no)
-			(effects
-				(font
-					(size 1.27 1.27)
-				)
-				(justify left)
-			)
-		)
-		(property "Footprint" "Package_TO_SOT_SMD:SOT-23-6"
-			(at 181.102 163.576 0)
-			(hide yes)
-			(show_name no)
-			(do_not_autoplace no)
-			(effects
-				(font
-					(size 1.27 1.27)
-				)
-			)
-		)
-		(property "Datasheet" "https://www.ti.com/lit/ds/symlink/sn74lvc2g17.pdf"
-			(at 180.594 169.418 0)
-			(hide yes)
-			(show_name no)
-			(do_not_autoplace no)
-			(effects
-				(font
-					(size 1.27 1.27)
-				)
-			)
-		)
-		(property "Description" "Dual schmitt buffer, VCC from 1.65 to 5.5 V, SOT-23"
-			(at 181.102 166.37 0)
-			(hide yes)
-			(show_name no)
-			(do_not_autoplace no)
-			(effects
-				(font
-					(size 1.27 1.27)
-				)
-			)
-		)
-		(pin "3"
-		)
-		(pin "2"
-		)
-		(pin "5"
-		)
-		(pin "6"
-		)
-		(pin "1"
-		)
-		(pin "4"
-		)
-		(instances
-			(project "Ziess-Microsope-Controller_Main_board"
-				(path "/95dcf840-9c51-41a6-a651-184d1d08cccc/c5484051-8362-473e-a51a-d9e129cb3c37"
-					(reference "U19")
-					(unit 1)
-				)
-			)
-		)
-	)
-	(symbol
 		(lib_id "Device:R_Small")
 		(at 252.73 97.79 0)
@@
 	)
 	(symbol
+		(lib_name "SN74LVC2G17DBV_1")
+		(lib_id "Library:SN74LVC2G17DBV")
+		(at 181.61 142.24 0)
+		(unit 1)
+		(body_style 1)
+		(exclude_from_sim no)
+		(in_bom yes)
+		(on_board yes)
+		(in_pos_files yes)
+		(dnp no)
+		(property "Reference" "U19"
+			(at 173.99 133.35 0)
+			(show_name no)
+			(do_not_autoplace no)
+			(effects
+				(font
+					(size 1.27 1.27)
+				)
+				(justify left)
+			)
+		)
+		(property "Value" "SN74LVC2G17DBV"
+			(at 184.912 151.13 0)
+			(show_name no)
+			(do_not_autoplace no)
+			(effects
+				(font
+					(size 1.27 1.27)
+				)
+				(justify left)
+			)
+		)
+		(property "Footprint" "Package_TO_SOT_SMD:SOT-23-6"
+			(at 181.102 163.576 0)
+			(hide yes)
+			(show_name no)
+			(do_not_autoplace no)
+			(effects
+				(font
+					(size 1.27 1.27)
+				)
+			)
+		)
+		(property "Datasheet" "https://www.ti.com/lit/ds/symlink/sn74lvc2g17.pdf"
+			(at 180.594 169.418 0)
+			(hide yes)
+			(show_name no)
+			(do_not_autoplace no)
+			(effects
+				(font
+					(size 1.27 1.27)
+				)
+			)
+		)
+		(property "Description" "Dual schmitt buffer, VCC from 1.65 to 5.5 V, SOT-23"
+			(at 181.102 166.37 0)
+			(hide yes)
+			(show_name no)
+			(do_not_autoplace no)
+			(effects
+				(font
+					(size 1.27 1.27)
+				)
+			)
+		)
+		(pin "3"
+		)
+		(pin "2"
+		)
+		(pin "5"
+		)
+		(pin "6"
+		)
+		(pin "1"
+		)
+		(pin "4"
+		)
+		(instances
+			(project "Ziess-Microsope-Controller_Main_board"
+				(path "/95dcf840-9c51-41a6-a651-184d1d08cccc/c5484051-8362-473e-a51a-d9e129cb3c37"
+					(reference "U19")
+					(unit 1)
+				)
+			)
+		)
+	)
+	(symbol
 		(lib_id "power:+3.3V")
 		(at 27.94 153.67 0)
@@
 	)
 	(symbol
+		(lib_name "SN74LVC2G17DBV_1")
 		(lib_id "Library:SN74LVC2G17DBV")
 		(at 181.61 77.47 0)
@@
 		)
 		(property "Value" "SN74LVC2G17DBV"
-			(at 184.785 86.36 0)
+			(at 184.912 86.36 0)
 			(show_name no)
 			(do_not_autoplace no)

Commit message: init
Parts:
- removed J12, J13: BM03B-GHS-TBT, Library:BM03BGHSTBTLFSN, symbol Connector_Generic:Conn_01x03
- added J12: BM06B-GHS-TBT, Library:BM06BGHSTBTLFSN, symbol Connector_Generic:Conn_01x06
- C117, C118, C119, C120, C121, C122, C123, C124, C125, C126, C127, C128, C129, C130, C131, C132, C133, C134, C135, C136: footprint Capacitor_SMD:C_0603_1608Metric -> Capacitor_SMD:C_0402_1005Metric
- R116, R117, R118, R119, R120, R121, R122, R123, R124, R125, R126, R127, R128, R129, R130, R131, R132, R133, R134, R135, R136, R137, R138, R139, R140, R141, R142, R143, R144, R145, R146, R147, R148, R149, R150: footprint Resistor_SMD:R_0603_1608Metric -> Resistor_SMD:R_0402_1005Metric
Connections:
- net GND: now also J12.1 (Pin_1), J12.4 (Pin_4)
- net at C126.2, D9.1 (K), R123.1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: now also J12.3 (Pin_3)
- net at C125.2, D9.2 (K), R122.1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: now also J12.2 (Pin_2)
- net at C120.2, D8.1 (K), R119.1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: now also J12.6 (Pin_6)
- net at C119.2, D8.2 (K), R118.1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: now also J12.5 (Pin_5)
